File: Hardware/VGMPlayer/VGMPlayer.kicad_pcb (KiCad board)
At the start: 2 copper layers, 59 parts, among them J1 USB_B_Mini, J2 Conn_01x20_Male, J3 Conn_01x20_Male, U1 STC8951, U10 LTC6903, U11 HC-06, U2 LD1117, U3 LM386, U4 LM386, U5 OLED_128_64_I2C, U6 AUDIOJACK, U7 YM2612, U8 SN76489, U9 LTC6903, Y1 11.0592MHz

Commit message: asdasd
Parts:
- C11, C12, C14, C16, C17, C18, C2, C27, C28, C5, C6, C7: footprint Capacitor_THT:CP_Radial_D8.0mm_P2.50mm -> Capacitor_THT:CP_Axial_L18.0mm_D10.0mm_P25.00mm_Horizontal
- C15: footprint Capacitor_THT:CP_Radial_D8.0mm_P2.50mm -> Capacitor_THT:CP_Axial_L18.0mm_D10.0mm_P25.00mm_Horizontal; moved to B.Cu
- C21, C22, C23, C24: footprint Capacitor_THT:CP_Radial_D8.0mm_P2.50mm -> Capacitor_THT:C_Axial_L17.0mm_D7.0mm_P20.00mm_Horizontal
- JP1, Y1: moved to B.Cu
- moved U11 147.1 mm to (71.1, 66.0)
- moved C11 135.9 mm to (188.0, 73.7)
- moved C17 127.5 mm to (250.2, 59.7), turned to 180 degrees
- moved R13 127.0 mm to (229.9, 81.3), turned to 180 degrees
- moved C19 118.4 mm to (233.7, 81.3)
- moved R14 118.2 mm to (234.1, 95.8)
- moved C21 116.9 mm to (238.8, 74.9)
- moved C16 116.7 mm to (96.5, 52.1)
- moved C20 115.9 mm to (230.3, 95.8), turned to 180 degrees
- moved C7 114.3 mm to (143.5, 102.9)
- moved C5 106.4 mm to (143.5, 73.7)
- moved U7 104.7 mm to (99.1, 72.4)
- moved JP1 102.6 mm to (36.8, 68.6), turned to 90 degrees
- moved J1 102.5 mm to (21.6, 77.5), turned to 90 degrees
- moved C22 101.4 mm to (238.8, 87.6)
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Connections:
- net Net-(J3-Pad10) renamed EA
- C1 pad 2: Net-(C1-Pad2) -> XTAL2
- C2 pad 2: Net-(C2-Pad2) -> RST
- C3 pad 2: Net-(C3-Pad2) -> XTAL1
- J2 pad 18: Net-(J2-Pad18) -> XTAL2
- J2 pad 19: Net-(J2-Pad19) -> XTAL1
- J2 pad 9: Net-(J2-Pad9) -> RST
- J3 pad 11: Net-(J3-Pad11) -> ALE
- J3 pad 12: Net-(J3-Pad12) -> PSEN
- R1 pad 1: Net-(C2-Pad2) -> RST
- U1 pad 18: Net-(C1-Pad2) -> XTAL2
- U1 pad 19: Net-(C3-Pad2) -> XTAL1
- U1 pad 29: Net-(U1-Pad29) -> PSEN
- U1 pad 30: Net-(U1-Pad30) -> ALE
- U1 pad 9: Net-(C2-Pad2) -> RST
- Y1 pad 1: Net-(C1-Pad2) -> XTAL2
- Y1 pad 2: Net-(C3-Pad2) -> XTAL1
Routing:
- net GND: track 0.00 -> 46.2 mm
- net RST: track 0.00 -> 33.8 mm
- net VCC: track 0.00 -> 17.8 mm
- net XTAL1: track 0.00 -> 12.4 mm
- net XTAL2: track 0.00 -> 11.4 mm
- net YM_WR: track 0.00 -> 5.08 mm
- net YM_RD: track 0.00 -> 5.08 mm
- net YM_IC: track 0.00 -> 5.08 mm
- net YM_CS: track 0.00 -> 5.08 mm
- net YM_A1: track 0.00 -> 5.08 mm
- net YM_A0: track 0.00 -> 5.08 mm
- net TXD: track 0.00 -> 5.08 mm
- net RXD: track 0.00 -> 5.08 mm

Commit message: PCB
Parts:
- added JP10: Jumper_NC_Small, Jumper:SolderJumper-2_P1.3mm_Open_TrianglePad1.0x1.5mm, B.Cu at (99.6, 91.4)
- added JP11: Jumper_NC_Small, Jumper:SolderJumper-2_P1.3mm_Open_TrianglePad1.0x1.5mm, B.Cu at (99.6, 88.9)
- added JP12: Jumper_NC_Small, Jumper:SolderJumper-2_P1.3mm_Open_TrianglePad1.0x1.5mm, B.Cu at (99.6, 86.4)
- added JP13: Jumper_NC_Small, Jumper:SolderJumper-2_P1.3mm_Open_TrianglePad1.0x1.5mm, B.Cu at (99.6, 83.8)
- added JP14: Jumper_NC_Small, Jumper:SolderJumper-2_P1.3mm_Open_TrianglePad1.0x1.5mm, B.Cu at (99.6, 81.3)
- added JP15: Jumper_NC_Small, Jumper:SolderJumper-2_P1.3mm_Open_TrianglePad1.0x1.5mm, B.Cu at (99.6, 78.7)
- added JP16: Jumper_NC_Small, Jumper:SolderJumper-2_P1.3mm_Open_TrianglePad1.0x1.5mm, B.Cu at (99.6, 76.2)
- added JP2: Jumper_NC_Small, Jumper:SolderJumper-2_P1.3mm_Open_TrianglePad1.0x1.5mm, B.Cu at (90.3, 107.9)
- added JP3: Jumper_NC_Small, Jumper:SolderJumper-2_P1.3mm_Open_TrianglePad1.0x1.5mm, B.Cu at (90.3, 110.5)
- added JP4: Jumper_NC_Small, Jumper:SolderJumper-2_P1.3mm_Open_TrianglePad1.0x1.5mm, B.Cu at (90.3, 113.0)
- added JP5: Jumper_NC_Small, Jumper:SolderJumper-2_P1.3mm_Open_TrianglePad1.0x1.5mm, B.Cu at (90.3, 115.5)
- added JP6: Jumper_NC_Small, Jumper:SolderJumper-2_P1.3mm_Open_TrianglePad1.0x1.5mm, B.Cu at (90.3, 118.1)
- added JP7: Jumper_NC_Small, Jumper:SolderJumper-2_P1.3mm_Open_TrianglePad1.0x1.5mm, B.Cu at (90.3, 120.6)
- added JP8: Jumper_NC_Small, Jumper:SolderJumper-2_P1.3mm_Open_TrianglePad1.0x1.5mm, B.Cu at (90.3, 123.2)
- added JP9: Jumper_NC_Small, Jumper:SolderJumper-2_P1.3mm_Open_TrianglePad1.0x1.5mm, B.Cu at (99.6, 94.0)
- added R15: 0, Resistor_SMD:R_0805_2012Metric, F.Cu at (72.4, 62.2)
- C11, C12, C16, C2, C27, C28, C5, C6, C7: footprint Capacitor_THT:CP_Axial_L18.0mm_D10.0mm_P25.00mm_Horizontal -> Capacitor_THT:CP_Radial_D4.0mm_P1.50mm
- C14, C17, C18: footprint Capacitor_THT:CP_Axial_L18.0mm_D10.0mm_P25.00mm_Horizontal -> Capacitor_THT:CP_Radial_D8.0mm_P3.50mm
- C15: footprint Capacitor_THT:CP_Axial_L18.0mm_D10.0mm_P25.00mm_Horizontal -> Capacitor_THT:CP_Radial_D8.0mm_P3.50mm; moved to F.Cu
- C21, C22, C23, C24: footprint Capacitor_THT:C_Axial_L17.0mm_D7.0mm_P20.00mm_Horizontal -> Capacitor_THT:CP_Radial_D8.0mm_P3.50mm
- J1: value USB_B_Mini -> USB_B_Micro; footprint Connector_USB:USB_Mini-B_Lumberg_2486_01_Horizontal -> Connector_USB:USB_Micro-B_Amphenol_10103594-0001LF_Horizontal
- JP1: value SolderJumper_2_Bridged -> Jumper_NC_Small; footprint Jumper:SolderJumper-2_P1.3mm_Bridged_RoundedPad1.0x1.5mm -> Jumper:SolderJumper-2_P1.3mm_Open_TrianglePad1.0x1.5mm
- U2: value LD1117 -> 7805-VGM
- U6: value AUDIOJACK -> AUDIOJACK-VGM; footprint Connector_Audio:Jack_3.5mm_PJ31060-I_Horizontal -> Connector_Audio:Jack_Horizontal
- Y1: moved to F.Cu
- moved C2 142.9 mm to (71.1, 91.4)
- moved U6 131.1 mm to (140.5, 74.9)
- moved C17 130.0 mm to (120.8, 72.3)
- moved C18 112.9 mm to (129.8, 99.6), turned to 0 degrees
- moved C21 112.4 mm to (126.4, 72.3)
- moved U3 101.6 mm to (117.2, 78.9)
- moved C22 100.5 mm to (138.9, 99.6)
- moved C28 100.5 mm to (116.8, 122.6), turned to 270 degrees
- moved R14 99.0 mm to (138.8, 122.4)
- moved C15 97.4 mm to (133.5, 120.9), turned to 180 degrees
- moved C19 95.6 mm to (138.3, 88.0)
- moved C20 94.3 mm to (138.8, 118.6), turned to 0 degrees
- moved C14 92.7 mm to (133.2, 89.5)
- moved R13 92.0 mm to (138.3, 90.0), turned to 0 degrees
- moved U4 91.7 mm to (128.9, 106.2)
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Connections:
- J3 pad 13: SN_D7 -> P2.7
- J3 pad 14: SN_D6 -> P2.6
- J3 pad 15: SN_D5 -> P2.5
- J3 pad 16: SN_D4 -> P2.4
- J3 pad 17: SN_D3 -> P2.3
- J3 pad 18: SN_D2 -> P2.2
- J3 pad 19: SN_D1 -> P2.1
- J3 pad 20: SN_D0 -> P2.0
- JP1 pad 1: +5V -> P2.7
- JP1 pad 2: VCC -> SN_D7
- U1 pad 21: SN_D0 -> P2.0
- U1 pad 22: SN_D1 -> P2.1
- U1 pad 23: SN_D2 -> P2.2
- U1 pad 24: SN_D3 -> P2.3
- U1 pad 25: SN_D4 -> P2.4
- U1 pad 26: SN_D5 -> P2.5
- U1 pad 27: SN_D6 -> P2.6
- U1 pad 28: SN_D7 -> P2.7
- U2 pad 1: GND -> +5V
- U2 pad 2: VCC -> GND
- U2 pad 3: +5V -> VCC
- U6 pad 1: GND -> Net-(C21-Pad2)
- U6 pad 2: Net-(C21-Pad2) -> Net-(C22-Pad2)
- U6 pad 3: Net-(C22-Pad2) -> GND
Routing:
- net GND: track 46.2 -> 407.9 mm
- net VCC: track 17.8 -> 278.8 mm
- net YM_CS: track 5.08 -> 78.4 mm
- net IIC_SCK: track 0.00 -> 67.9 mm
- net SN_D0: track 0.00 -> 65.7 mm
- net IIC_SDA: track 0.00 -> 65.1 mm, vias 0 -> 2
- net SN_D1: track 0.00 -> 59.7 mm
- net YM_A1: track 5.08 -> 64.0 mm
- net SN_D2: track 0.00 -> 55.3 mm, vias 0 -> 1
- net SN_WR: track 0.00 -> 54.2 mm
- net YM_A0: track 5.08 -> 58.2 mm
- net YM_RD: track 5.08 -> 56.8 mm, vias 0 -> 1
- net SN_OUT: track 0.00 -> 50.1 mm
- net SN_D3: track 0.00 -> 49.8 mm, vias 0 -> 1
- net YM_WR: track 5.08 -> 54.4 mm, vias 0 -> 1
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- added copper zone on B.Cu, net GND
- added copper zone on F.Cu, net GND

Commit message: ewsd
Parts:
- added D1: , LED_SMD:LED_0805_2012Metric, F.Cu at (144.0, 134.1)
- added D10: , LED_SMD:LED_0805_2012Metric, F.Cu at (118.7, 134.1)
- added D11: , LED_SMD:LED_0805_2012Metric, F.Cu at (116.2, 134.1)
- added D12: , LED_SMD:LED_0805_2012Metric, F.Cu at (113.6, 134.1)
- added D13: , LED_SMD:LED_0805_2012Metric, F.Cu at (111.1, 134.1)
- added D14: , LED_SMD:LED_0805_2012Metric, F.Cu at (108.5, 134.1)
- added D15: , LED_SMD:LED_0805_2012Metric, F.Cu at (106.0, 134.1)
- added D16: , LED_SMD:LED_0805_2012Metric, F.Cu at (103.4, 134.1)
- added D17: LED, LED_SMD:LED_0805_2012Metric, F.Cu at (141.5, 151.4)
- added D18: LED, LED_SMD:LED_0805_2012Metric, F.Cu at (138.9, 151.4)
- added D19: LED, LED_SMD:LED_0805_2012Metric, F.Cu at (136.4, 151.4)
- added D2: , LED_SMD:LED_0805_2012Metric, F.Cu at (141.5, 134.1)
- added D20: LED, LED_SMD:LED_0805_2012Metric, F.Cu at (133.9, 151.4)
- added D21: LED, LED_SMD:LED_0805_2012Metric, F.Cu at (131.3, 151.4)
- added D22: LED, LED_SMD:LED_0805_2012Metric, F.Cu at (128.8, 151.4)
- added D23: LED, LED_SMD:LED_0805_2012Metric, F.Cu at (126.2, 151.4)
- added D24: LED, LED_SMD:LED_0805_2012Metric, F.Cu at (123.7, 151.4)
- added D25: LED, LED_SMD:LED_0805_2012Metric, F.Cu at (113.4, 152.3)
- added D26: LED, LED_SMD:LED_0805_2012Metric, F.Cu at (110.9, 152.3)
- added D27: LED, LED_SMD:LED_0805_2012Metric, F.Cu at (108.4, 152.3)
- added D28: LED, LED_SMD:LED_0805_2012Metric, F.Cu at (105.8, 152.3)
- added D29: LED, LED_SMD:LED_0805_2012Metric, F.Cu at (103.3, 152.3)
- added D3: , LED_SMD:LED_0805_2012Metric, F.Cu at (139.0, 134.1)
- added D30: LED, LED_SMD:LED_0805_2012Metric, F.Cu at (100.8, 152.3)
- added D31: LED, LED_SMD:LED_0805_2012Metric, F.Cu at (98.3, 152.3)
- added D32: LED, LED_SMD:LED_0805_2012Metric, F.Cu at (95.7, 152.3)
- added D4: , LED_SMD:LED_0805_2012Metric, F.Cu at (136.4, 134.1)
- added D5: , LED_SMD:LED_0805_2012Metric, F.Cu at (133.9, 134.1)
- added D6: , LED_SMD:LED_0805_2012Metric, F.Cu at (131.3, 134.1)
- added D7: , LED_SMD:LED_0805_2012Metric, F.Cu at (128.8, 134.1)
- added D8: , LED_SMD:LED_0805_2012Metric, F.Cu at (126.3, 134.1)
- added D9: , LED_SMD:LED_0805_2012Metric, F.Cu at (121.3, 134.1)
- added J4: Conn_01x20_Male, Connector_PinSocket_2.54mm:PinSocket_1x20_P2.54mm_Vertical, F.Cu at (144.0, 130.6)
- added J5: Conn_01x20_Male, Connector_PinSocket_2.54mm:PinSocket_1x20_P2.54mm_Vertical, F.Cu at (144.0, 156.0)
- added R16: , Resistor_SMD:R_0805_2012Metric, F.Cu at (144.0, 137.8)
- added R17: , Resistor_SMD:R_0805_2012Metric, F.Cu at (141.5, 137.8)
- added R18: , Resistor_SMD:R_0805_2012Metric, F.Cu at (139.0, 137.8)
- added R19: , Resistor_SMD:R_0805_2012Metric, F.Cu at (136.4, 137.8)
- added R20: , Resistor_SMD:R_0805_2012Metric, F.Cu at (133.9, 137.8)
- added R21: , Resistor_SMD:R_0805_2012Metric, F.Cu at (131.3, 137.8)
- added R22: , Resistor_SMD:R_0805_2012Metric, F.Cu at (128.8, 137.8)
- added R23: , Resistor_SMD:R_0805_2012Metric, F.Cu at (126.3, 137.8)
- added R24: , Resistor_SMD:R_0805_2012Metric, F.Cu at (121.3, 137.7)
- added R25: , Resistor_SMD:R_0805_2012Metric, F.Cu at (118.7, 137.7)
- added R26: , Resistor_SMD:R_0805_2012Metric, F.Cu at (116.2, 137.7)
- added R27: , Resistor_SMD:R_0805_2012Metric, F.Cu at (113.6, 137.7)
- added R28: , Resistor_SMD:R_0805_2012Metric, F.Cu at (111.1, 137.7)
- added R29: , Resistor_SMD:R_0805_2012Metric, F.Cu at (108.5, 137.7)
- added R30: , Resistor_SMD:R_0805_2012Metric, F.Cu at (106.0, 137.7)
- added R31: , Resistor_SMD:R_0805_2012Metric, F.Cu at (103.4, 137.7)
- added R32: 1k, Resistor_SMD:R_0805_2012Metric, F.Cu at (141.5, 147.9)
- added R33: 1k, Resistor_SMD:R_0805_2012Metric, F.Cu at (138.9, 147.9)
- added R34: 1k, Resistor_SMD:R_0805_2012Metric, F.Cu at (136.4, 147.9)
- added R35: 1k, Resistor_SMD:R_0805_2012Metric, F.Cu at (133.9, 147.9)
- added R36: 1k, Resistor_SMD:R_0805_2012Metric, F.Cu at (131.3, 147.9)
- added R37: 1k, Resistor_SMD:R_0805_2012Metric, F.Cu at (128.8, 147.9)
- added R38: 1k, Resistor_SMD:R_0805_2012Metric, F.Cu at (126.2, 147.9)
- added R39: 1k, Resistor_SMD:R_0805_2012Metric, F.Cu at (123.7, 147.9)
- added R40: 1k, Resistor_SMD:R_0805_2012Metric, F.Cu at (113.4, 148.7)
- added R41: 1k, Resistor_SMD:R_0805_2012Metric, F.Cu at (110.9, 148.7)
- added R42: 1k, Resistor_SMD:R_0805_2012Metric, F.Cu at (108.4, 148.7)
- added R43: 1k, Resistor_SMD:R_0805_2012Metric, F.Cu at (105.8, 148.7)
- added R44: 1k, Resistor_SMD:R_0805_2012Metric, F.Cu at (103.3, 148.7)
- added R45: 1k, Resistor_SMD:R_0805_2012Metric, F.Cu at (100.8, 148.7)
- added R46: 1k, Resistor_SMD:R_0805_2012Metric, F.Cu at (98.3, 148.7)
- added R47: 1k, Resistor_SMD:R_0805_2012Metric, F.Cu at (95.7, 148.7)
Routing:
- net Net-(J5-Pad1): track 0.00 -> 106.9 mm
- net Net-(D24-Pad1): track 0.00 -> 3.64 mm
- net Net-(D23-Pad1): track 0.00 -> 3.64 mm
- net Net-(D22-Pad1): track 0.00 -> 3.64 mm
- net Net-(D20-Pad1): track 0.00 -> 3.64 mm
- net Net-(D19-Pad1): track 0.00 -> 3.64 mm
- net Net-(D18-Pad1): track 0.00 -> 3.64 mm
- net Net-(D21-Pad1): track 0.00 -> 3.64 mm
- net Net-(D17-Pad1): track 0.00 -> 3.64 mm
- net Net-(D25-Pad1): track 0.00 -> 2.80 mm
- net Net-(D26-Pad1): track 0.00 -> 2.79 mm
- net Net-(D28-Pad1): track 0.00 -> 2.78 mm
- net Net-(D29-Pad1): track 0.00 -> 2.77 mm
- net Net-(D30-Pad1): track 0.00 -> 2.76 mm
- net Net-(D31-Pad1): track 0.00 -> 2.75 mm
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Other:
- board outline added: 94.5 x 99.8 mm

Commit message: Done!
Other:
- board text added: "Designed By Mac Lin"
- board text added: "VGM PLAYER V0.1"
Changed lines of the file:
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@@
   (general
     (thickness 1.6)
-    (drawings 4)
+    (drawings 6)
     (tracks 860)
     (zones 0)
@@
     )
   )
+  (gr_text "Designed By Mac Lin" (at 122.174 65.786) (layer F.SilkS)
+    (effects (font (size 1.5 1.5) (thickness 0.3)))
+  )
+  (gr_text "VGM PLAYER V0.1" (at 120.269 63.246) (layer F.SilkS)
+    (effects (font (size 1.5 1.5) (thickness 0.3)))
+  )
   (gr_line (start 147.32 60.452) (end 147.32 160.274) (layer Edge.Cuts) (width 0.15))

Commit message: asd
Parts:
- moved D14 2.42 mm to (108.4, 136.5)
- moved D17 2.42 mm to (141.4, 153.8)
- moved D19 2.42 mm to (136.3, 153.8)
- moved D20 2.42 mm to (133.7, 153.8)
- moved D21 2.42 mm to (131.2, 153.8)
- moved D25 2.42 mm to (113.3, 154.7)
- moved D29 2.42 mm to (103.2, 154.7)
- moved J5 2.42 mm to (143.9, 158.4)
- moved R29 2.42 mm to (108.4, 140.2)
- moved R32 2.42 mm to (141.4, 150.4)
- moved R34 2.42 mm to (136.3, 150.4)
- moved R35 2.42 mm to (133.7, 150.4)
- moved R36 2.42 mm to (131.2, 150.4)
- moved R40 2.42 mm to (113.3, 151.1)
- moved R44 2.42 mm to (103.2, 151.1)
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Routing:
- net GND: vias 0 -> 1
Other:
- board size 94.5 x 99.8 mm -> 94.5 x 103.1 mm

Commit message: 1
Parts:
- D1, D10, D11, D12, D13, D14, D15, D16, D2, D3, D4, D5, D6, D7, D8, D9: value (none) -> LED
- J1: value USB_B_Micro -> Barrel_Jack_Switch; footprint Connector_USB:USB_Micro-B_Amphenol_10103594-0001LF_Horizontal -> Connector_BarrelJack:BarrelJack_Horizontal
- R16, R17, R18, R19, R20, R21, R22, R23, R24, R25, R26, R27, R28, R29, R30, R31: value (none) -> 1k
- moved J1 10.8 mm to (67.6, 66.8), turned to 0 degrees
- moved C10 8.64 mm to (75.9, 62.2)
- moved C23 8.64 mm to (96.5, 64.5)
- moved C25 8.64 mm to (105.7, 65.9)
- moved C27 8.64 mm to (111.3, 64.5)
- moved R15 8.64 mm to (81.0, 62.2)
- moved U2 8.64 mm to (75.9, 68.6)
- moved U9 8.64 mm to (107.2, 69.0)
- moved U5 8.52 mm to (87.9, 70.4)
- moved JP1 1.30 mm to (90.6, 106.6)
- moved JP3 1.30 mm to (90.6, 111.7)
- moved JP8 1.30 mm to (90.6, 124.4)
- moved R1 1.30 mm to (68.8, 97.8)
- moved Y1 1.30 mm to (71.4, 117.0)
- moved C13 1.30 mm to (77.7, 76.2)
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Connections:
- J1 pad 2: Net-(J1-Pad2) -> GND
Routing:
- net GND: track 407.9 -> 0.00 mm, vias 1 -> 0
- net VCC: track 278.8 -> 0.00 mm
- net Net-(J5-Pad1): track 106.9 -> 0.00 mm
- net YM_CS: track 78.4 -> 0.00 mm
- net IIC_SCK: track 67.9 -> 0.00 mm
- net SN_D0: track 65.7 -> 0.00 mm
- net IIC_SDA: track 65.1 -> 0.00 mm, vias 2 -> 0
- net YM_A1: track 64.0 -> 0.00 mm
- net SN_D1: track 59.7 -> 0.00 mm
- net YM_A0: track 58.2 -> 0.00 mm
- net YM_RD: track 56.8 -> 0.00 mm, vias 1 -> 0
- net SN_D2: track 55.3 -> 0.00 mm, vias 1 -> 0
- net YM_WR: track 54.4 -> 0.00 mm, vias 1 -> 0
- net SN_WR: track 54.2 -> 0.00 mm
- net SN_OUT: track 50.1 -> 0.00 mm
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- removed copper zone on B.Cu, net GND
- removed copper zone on F.Cu, net GND

Commit message: 1
Parts:
- removed D1, D10, D11, D12, D13, D14, D15, D16, D17, D18, D19, D2, D20, D21, D22, D23, D24, D25, D26, D27, D28, D29, D3, D30, D31, D32, D4, D5, D6, D7, D8, D9: LED, LED_SMD:LED_0805_2012Metric
- removed J3, J5: Conn_01x20_Male, Connector_PinSocket_2.54mm:PinSocket_1x20_P2.54mm_Vertical
- removed JP1, JP10, JP11, JP12, JP13, JP14, JP15, JP16, JP2, JP3, JP4, JP5, JP6, JP7, JP8, JP9: Jumper_NC_Small, Jumper:SolderJumper-2_P1.3mm_Open_TrianglePad1.0x1.5mm
- removed R18, R19, R20, R21, R22, R23, R24, R25, R26, R27, R28, R29, R30, R31, R32, R33, R34, R35, R36, R37, R38, R39, R40, R41, R42, R43, R44, R45, R46, R47: 1k, Resistor_SMD:R_0805_2012Metric
- added C29: 10uF, Capacitor_THT:CP_Radial_D8.0mm_P3.50mm, F.Cu at (109.9, 63.4)
- added C30: 1.5nF, Capacitor_SMD:C_0805_2012Metric, F.Cu at (131.3, 76.6)
- added C31: 1.5nF, Capacitor_SMD:C_0805_2012Metric, F.Cu at (133.9, 76.6)
- added C32: 33pF, Capacitor_SMD:C_0805_2012Metric, F.Cu at (133.0, 120.4)
- added C33: 33pF, Capacitor_SMD:C_0805_2012Metric, F.Cu at (122.6, 120.3)
- added L1: L, Inductor_SMD:L_0805_2012Metric, F.Cu at (61.6, 71.0)
- added L2: L, Inductor_SMD:L_0805_2012Metric, F.Cu at (61.5, 62.7)
- added R51: 1k, Resistor_SMD:R_0805_2012Metric, F.Cu at (121.8, 123.0)
- added R52: 1k, Resistor_SMD:R_0805_2012Metric, F.Cu at (121.8, 117.6)
- added U12: 74HC04, VGM:SOP-14_4.4x8.3mm_P1.27mm, F.Cu at (127.8, 118.9)
- added U13: YM3012, Package_DIP:DIP-16_W7.62mm_Socket, F.Cu at (116.1, 81.3)
- added U14: LM386, Package_DIP:DIP-8_W7.62mm_Socket, F.Cu at (116.0, 62.7)
- added U15: LM386, Package_DIP:DIP-8_W7.62mm_Socket, F.Cu at (126.9, 62.7)
- added U16: LM386, Package_DIP:DIP-8_W7.62mm_Socket, F.Cu at (137.8, 62.7)
- added U17: LM386, Package_DIP:DIP-8_W7.62mm_Socket, F.Cu at (137.8, 73.5)
- added U18: OLED_128_64_I2C, Connector_PinSocket_2.54mm:PinSocket_1x04_P2.54mm_Vertical, F.Cu at (50.3, 62.7)
- added U19: ESP8266Module, Connector_PinSocket_2.54mm:PinSocket_1x06_P2.54mm_Vertical, F.Cu at (50.3, 90.6)
- added U20: YM2612, Package_DIP:DIP-24_W15.24mm_Socket, F.Cu at (145.3, 88.0)
- added Y2: 3.768Mhz, Crystal:Crystal_HC49-4H_Vertical, F.Cu at (138.4, 122.4)
- added Y5: 7.67Mhz, Crystal:Crystal_HC49-4H_Vertical, F.Cu at (117.0, 122.5)
- J1: value Barrel_Jack_Switch -> Conn_02x20_Odd_Even; footprint Connector_BarrelJack:BarrelJack_Horizontal -> Connector_PinSocket_2.00mm:PinSocket_2x20_P2.00mm_Vertical
- J2: value Conn_01x20_Male -> Conn_02x20_Odd_Even; footprint Connector_PinSocket_2.54mm:PinSocket_1x20_P2.54mm_Vertical -> Connector_PinSocket_2.00mm:PinSocket_2x20_P2.00mm_Vertical
- J4: value Conn_01x20_Male -> USB_B_Micro; footprint Connector_PinSocket_2.54mm:PinSocket_1x20_P2.54mm_Vertical -> Connector_USB:USB_Micro-B_Molex-105017-0001
- R15: value 0 -> 270
- U11: footprint Connector_PinSocket_2.54mm:PinSocket_1x04_P2.54mm_Vertical -> Connector_PinSocket_2.54mm:PinSocket_1x06_P2.54mm_Vertical
- U5: value OLED_128_64_I2C -> YM2151; footprint Connector_PinSocket_2.54mm:PinSocket_1x04_P2.54mm_Vertical -> Package_DIP:DIP-24_W15.24mm_Socket
- moved J4 92.2 mm to (51.7, 132.1)
- moved U1 80.1 mm to (56.6, 155.7), turned to 90 degrees
- moved R1 74.0 mm to (104.8, 162.4), turned to 0 degrees
- moved J2 70.4 mm to (61.3, 146.6), turned to 90 degrees
- moved RN1 69.7 mm to (56.7, 137.2), turned to 0 degrees
- moved C2 69.0 mm to (88.3, 159.6), turned to 270 degrees
- moved C10 68.1 mm to (72.2, 130.2), turned to 270 degrees
- moved C13 66.4 mm to (52.5, 137.7), turned to 180 degrees
- moved U2 64.6 mm to (63.3, 131.9)
- moved C16 51.1 mm to (57.6, 129.9), turned to 270 degrees
- moved R15 50.5 mm to (130.9, 70.4), turned to 180 degrees
- moved Y1 49.0 mm to (94.5, 160.3), turned to 0 degrees
- moved C1 47.8 mm to (104.8, 160.4)
- moved R13 46.0 mm to (93.8, 78.4), turned to 180 degrees
- moved C3 44.2 mm to (104.8, 158.4)
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Connections:
- net Net-(U10-Pad6) renamed SN_CLK
- net Net-(U7-Pad24) renamed YM_CLK
- C1 pad 1: GND -> GND_8051
- C1 pad 2: XTAL2 -> Net-(C1-Pad2)
- C10 pad 1: GND -> GND_8051
- C10 pad 2: +5V -> +5V_8051
- C13 pad 1: VCC -> +5V_8051
- C13 pad 2: GND -> GND_8051
- C14 pad 1: VCC -> +5V
- C14 pad 2: GND -> GNDA
- C15 pad 1: VCC -> +5V
- C15 pad 2: GND -> GNDA
- C16 pad 1: VCC -> Net-(C16-Pad1)
- C16 pad 2: GND -> GND_8051
- C17 pad 2: GND -> GNDA
- C18 pad 2: GND -> GNDA
- C2 pad 1: VCC -> +5V_8051
- C2 pad 2: RST -> Net-(C2-Pad2)
- C23 pad 1: VCC -> VDD
- C24 pad 1: VCC -> VDD
- C25 pad 2: VCC -> VDD
- C26 pad 2: VCC -> VDD
- C27 pad 1: VCC -> VDD
- C28 pad 1: VCC -> VDD
- C3 pad 1: GND -> GND_8051
- C3 pad 2: XTAL1 -> Net-(C3-Pad2)
- C4 pad 2: GND -> GNDA
- J1 pad 1: +5V -> Net-(J1-Pad1)
- J1 pad 2: GND -> +5V
- J1 pad 3: Net-(J1-Pad3) -> D0
- J2 pad 1: YM_D0 -> +3V3_8051
- J2 pad 10: RXD -> P0.1
- J2 pad 11: TXD -> P1.3
- J2 pad 12: YM_CS -> P2.7
- J2 pad 13: YM_WR -> P1.4
- J2 pad 14: YM_RD -> GND_8051
- J2 pad 15: YM_A0 -> P1.5
- J2 pad 16: YM_A1 -> P2.6
- J2 pad 17: YM_IC -> +3V3_8051
- J2 pad 18: XTAL2 -> P2.5
- J2 pad 19: XTAL1 -> P1.6
- J2 pad 2: YM_D1 -> +5V_8051
- J2 pad 20: GND -> GND_8051
- J2 pad 3: YM_D2 -> P1.0
- J2 pad 4: YM_D3 -> +5V_8051
- J2 pad 5: YM_D4 -> P1.1
- J2 pad 6: YM_D5 -> GND_8051
- J2 pad 7: YM_D6 -> P1.2
- J2 pad 8: YM_D7 -> P0.0
- J2 pad 9: RST -> GND_8051
- J4 pad 1: Net-(D1-Pad1) -> Net-(C16-Pad1)
- J4 pad 5: Net-(D5-Pad1) -> GND_8051
- J4 pad 6: Net-(D6-Pad1) -> GND_8051
- R1 pad 1: RST -> Net-(C2-Pad2)
- R1 pad 2: GND -> GND_8051
- R13 pad 2: GND -> GNDA
- R14 pad 2: GND -> GNDA
- R15 pad 1: VCC -> Net-(R15-Pad1)
- R15 pad 2: +5V -> Net-(R15-Pad2)
- R16 pad 2: Net-(J5-Pad1) -> Net-(R16-Pad2)
- R17 pad 2: Net-(J5-Pad1) -> Net-(C32-Pad1)
- R2 pad 1: GND -> GNDA
- R3 pad 1: GND -> GNDA
- R4 pad 1: GND -> GNDA
- RN1 pad 1: VCC -> +5V_8051
- RN1 pad 2: I2C_SCK -> P0.0
- RN1 pad 3: I2C_SDA -> P0.1
- RN1 pad 4: SN_WR -> P0.2
- U1 pad 1: YM_D0 -> P1.0
- U1 pad 10: RXD -> P3.0
- U1 pad 11: TXD -> P3.1
- U1 pad 12: YM_CS -> P3.2
- U1 pad 13: YM_WR -> P3.3
- U1 pad 14: YM_RD -> P3.4
- U1 pad 15: YM_A0 -> P3.5
- U1 pad 16: YM_A1 -> P3.6
- U1 pad 17: YM_IC -> P3.7
- U1 pad 18: XTAL2 -> Net-(C1-Pad2)
- U1 pad 19: XTAL1 -> Net-(C3-Pad2)
- U1 pad 2: YM_D1 -> P1.1
- U1 pad 20: GND -> GND_8051
- U1 pad 29: PSEN -> Net-(U1-Pad29)
- U1 pad 3: YM_D2 -> P1.2
- U1 pad 30: ALE -> Net-(U1-Pad30)
- U1 pad 31: VCC -> +5V_8051
- U1 pad 37: SN_WR -> P0.2
- U1 pad 38: I2C_SDA -> P0.1
- U1 pad 39: I2C_SCK -> P0.0
- U1 pad 4: YM_D3 -> P1.3
- U1 pad 40: VCC -> +5V_8051
- U1 pad 5: YM_D4 -> P1.4
- U1 pad 6: YM_D5 -> P1.5
- U1 pad 7: YM_D6 -> P1.6
- U1 pad 8: YM_D7 -> P1.7
- U1 pad 9: RST -> Net-(C2-Pad2)
- U10 pad 2: IIC_SDA -> I2C_SDA
- U10 pad 3: IIC_SCK -> I2C_SCK
- U10 pad 7: VCC -> VDD
- U10 pad 8: VCC -> VDD
- U11 pad 1: VCC -> Net-(U11-Pad1)
- U11 pad 2: GND -> VDD
- U11 pad 3: RXD -> GND
- U11 pad 4: TXD -> RXD
- U2 pad 1: +5V -> +5V_8051
- U2 pad 2: GND -> GND_8051
- U2 pad 3: VCC -> Net-(C16-Pad1)
- U3 pad 2: GND -> GNDA
- U3 pad 4: GND -> GNDA
- U3 pad 6: VCC -> +5V
- U4 pad 2: GND -> GNDA
- U4 pad 4: GND -> GNDA
- U4 pad 6: VCC -> +5V
- U5 pad 1: GND -> GND_YM2151
- U5 pad 2: VCC -> YM2151_IRQ
- U5 pad 3: I2C_SCK -> YM2151_IC
- U5 pad 4: I2C_SDA -> YM2151_A0
- U6 pad 3: GND -> GNDA
- U7 pad 19: GND -> GNDA
- U7 pad 2: YM_D0 -> D0
- U7 pad 22: VCC -> +5V
- U7 pad 23: VCC -> VDD
- U7 pad 3: YM_D1 -> D1
- U7 pad 4: YM_D2 -> D2
- U7 pad 5: YM_D3 -> D3
- U7 pad 6: YM_D4 -> D4
- U7 pad 7: YM_D5 -> D5
- U7 pad 8: YM_D6 -> D6
- U7 pad 9: YM_D7 -> D7
- U8 pad 1: SN_D5 -> D5
- U8 pad 10: SN_D0 -> D0
- U8 pad 11: SN_D1 -> D1
- U8 pad 12: SN_D2 -> D2
- U8 pad 13: SN_D3 -> D3
- U8 pad 15: SN_D4 -> D4
- U8 pad 16: VCC -> VDD
- U8 pad 2: SN_D6 -> D6
- U8 pad 3: SN_D7 -> D7
- U9 pad 2: IIC_SDA -> I2C_SDA
- U9 pad 3: IIC_SCK -> I2C_SCK
- U9 pad 7: VCC -> VDD
- U9 pad 8: VCC -> VDD
- Y1 pad 1: XTAL2 -> Net-(C1-Pad2)
- Y1 pad 2: XTAL1 -> Net-(C3-Pad2)
Other:
- board size 94.5 x 103.1 mm -> 99.4 x 103.3 mm
- board text added: "Designed By"
- board text added: "Mac Lin"
- board text removed: "Designed By Mac Lin"
