File: Hardware/VGMPlayer/VGMPlayer.kicad_pcb (KiCad board)
At the start: 2 copper layers, 99.4 x 103.3 mm, 81 parts, among them J1 Conn_02x20_Odd_Even, J2 Conn_02x20_Odd_Even, J4 USB_B_Micro, U1 STC8951, U10 LTC6903, U11 HC-06, U12 74HC04, U13 YM3012, U14 LM386, U15 LM386, U16 LM386, U17 LM386, U18 OLED_128_64_I2C, U19 ESP8266Module, U2 7805-VGM, U20 YM2612, U3 LM386, U4 LM386, U5 YM2151, U6 AUDIOJACK-VGM, U7 YM2612, U8 SN76489, U9 LTC6903, Y1 11.0592MHz, Y2 3.768Mhz, Y5 7.67Mhz

Commit message: 1
Parts:
- removed R16, R17, R51, R52: 1k, Resistor_SMD:R_0805_2012Metric
- removed U15, U16, U17: LM386, Package_DIP:DIP-8_W7.62mm_Socket
- removed Y2: 3.768Mhz, Crystal:Crystal_HC49-4H_Vertical
- removed Y5: 7.67Mhz, Crystal:Crystal_HC49-4H_Vertical
- added U21: 74HCT595, Package_DIP:DIP-16_W7.62mm, F.Cu at (59.8, 130.0)
- added U22: 74HCT595, Package_DIP:DIP-16_W7.62mm, F.Cu at (69.7, 130.0)
- added U23: 74HCT595, Package_DIP:DIP-16_W7.62mm, F.Cu at (50.0, 130.0)
- C32: value 33pF -> 10uF; footprint Capacitor_SMD:C_0805_2012Metric -> Capacitor_THT:CP_Radial_D4.0mm_P1.50mm
- C33: value 33pF -> 100nF
- J1, J2: value Conn_02x20_Odd_Even -> Conn_02x20_Counter_Clockwise; footprint Connector_PinSocket_2.00mm:PinSocket_2x20_P2.00mm_Vertical -> Package_DIP:DIP-40_W15.24mm_Socket
- U12: value 74HC04 -> 7805-VGM; footprint VGM:SOP-14_4.4x8.3mm_P1.27mm -> Package_TO_SOT_THT:TO-220-3_Vertical
- U14: value LM386 -> LM324; footprint Package_DIP:DIP-8_W7.62mm_Socket -> Package_DIP:DIP-14_W7.62mm
- moved J4 91.9 mm to (143.6, 134.4), turned to 90 degrees
- moved C13 90.7 mm to (142.8, 128.9), turned to 0 degrees
- moved U18 82.4 mm to (104.1, 125.2), turned to 90 degrees
- moved U2 82.1 mm to (144.3, 145.7), turned to 180 degrees
- moved C16 79.6 mm to (137.0, 136.2), turned to 90 degrees
- moved C10 65.5 mm to (135.4, 147.3), turned to 90 degrees
- moved U11 47.4 mm to (50.1, 121.4), turned to 90 degrees
- moved U19 34.6 mm to (50.1, 125.1), turned to 90 degrees
- moved Y1 33.4 mm to (120.5, 139.2)
- moved R1 33.4 mm to (130.8, 141.4)
- moved C1 33.4 mm to (130.7, 139.4)
- moved C3 33.4 mm to (130.7, 137.3)
- moved C2 32.0 mm to (113.1, 139.3)
- moved U14 29.4 mm to (145.3, 62.7), turned to 270 degrees
- moved U1 27.7 mm to (83.0, 147.4)
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Connections:
- net Net-(J1-Pad28) renamed PP_LATCH
- net Net-(J1-Pad32) renamed I2C_CLK
- net Net-(J1-Pad40) renamed +3V3
- C24 pad 1: VDD -> +5V
- C32 pad 1: Net-(C32-Pad1) -> Net-(C16-Pad1)
- C32 pad 2: Net-(C32-Pad2) -> GND_8051
- C33 pad 1: Net-(C33-Pad1) -> GND_8051
- C33 pad 2: Net-(C33-Pad2) -> +3V_8051
- J1 pad 10: I2C_SDA -> D5
- J1 pad 11: D3 -> D6
- J1 pad 12: SN_WR -> D7
- J1 pad 13: D4 -> YM_CS
- J1 pad 14: GND -> YM_WR
- J1 pad 15: D5 -> YM_A0
- J1 pad 16: YM_CLK_CS -> YM_A1
- J1 pad 17: Net-(J1-Pad1) -> Net-(J1-Pad17)
- J1 pad 18: SN_CLK_CS -> Net-(J1-Pad18)
- J1 pad 19: D6 -> GND
- J1 pad 2: +5V -> Net-(J1-Pad2)
- J1 pad 21: D7 -> YM_IC
- J1 pad 23: YM_CS -> Net-(J1-Pad23)
- J1 pad 25: GND -> Net-(J1-Pad25)
- J1 pad 26: Net-(J1-Pad26) -> TXD
- J1 pad 27: Net-(J1-Pad27) -> RXD
- J1 pad 29: YM_WR -> PP_DAT
- J1 pad 3: D0 -> Net-(J1-Pad3)
- J1 pad 30: GND -> PP_CLK
- J1 pad 31: YM_RD -> I2C_DAT
- J1 pad 33: YM_A0 -> SN_CLK_CS
- J1 pad 34: GND -> YM_CLK_CS
- J1 pad 35: YM_A1 -> SN_WR
- J1 pad 36: Net-(J1-Pad36) -> SPI_MOSI
- J1 pad 37: YM_IC -> SPI_CLK
- J1 pad 38: Net-(J1-Pad38) -> VDD
- J1 pad 4: +5V -> Net-(J1-Pad4)
- J1 pad 5: D1 -> D0
- J1 pad 6: GND -> D1
- J1 pad 8: I2C_SCK -> D3
- J1 pad 9: GND -> D4
- J2 pad 1: +3V3_8051 -> Net-(J2-Pad1)
- J2 pad 10: P0.1 -> P0.5
- J2 pad 11: P1.3 -> P0.6
- J2 pad 12: P2.7 -> P0.7
- J2 pad 13: P1.4 -> P2.0
- J2 pad 14: GND_8051 -> P2.1
- J2 pad 15: P1.5 -> P3.2
- J2 pad 16: P2.6 -> P3.3
- J2 pad 17: +3V3_8051 -> Net-(J2-Pad17)
- J2 pad 18: P2.5 -> +3V_8051
- J2 pad 19: P1.6 -> GND_8051
- J2 pad 2: +5V_8051 -> P2.2
- J2 pad 21: P1.7 -> P3.4
- J2 pad 22: P2.4 -> P3.5
- J2 pad 23: P3.0 -> P3.6
- J2 pad 24: P2.3 -> P3.7
- J2 pad 25: GND_8051 -> P1.0
- J2 pad 26: P2.2 -> P1.1
- J2 pad 27: Net-(J2-Pad27) -> P1.2
- J2 pad 28: Net-(J2-Pad28) -> P1.3
- J2 pad 29: P3.1 -> P1.4
- J2 pad 3: P1.0 -> P1.5
- J2 pad 30: GND_8051 -> P1.7
- J2 pad 31: P3.2 -> P2.3
- J2 pad 32: P2.1 -> P2.4
- J2 pad 33: P3.3 -> P2.5
- J2 pad 34: GND_8051 -> P2.6
- J2 pad 35: P3.4 -> P2.7
- J2 pad 36: P2.0 -> P3.0
- J2 pad 37: P3.5 -> P3.1
- J2 pad 38: P3.6 -> +5V_8051
- J2 pad 4: +5V_8051 -> P1.6
- J2 pad 40: P3.7 -> +3V_8051
- J2 pad 5: P1.1 -> P0.0
- J2 pad 6: GND_8051 -> P0.1
- J2 pad 7: P1.2 -> P0.2
- J2 pad 8: P0.0 -> P0.3
- J2 pad 9: GND_8051 -> P0.4
- U10 pad 2: I2C_SDA -> SPI_CLK
- U10 pad 3: I2C_SCK -> SPI_MOSI
- U12 pad 1: Net-(R16-Pad2) -> +3V_8051
- U12 pad 2: Net-(C32-Pad2) -> GND_8051
- U12 pad 3: Net-(C32-Pad1) -> Net-(C16-Pad1)
- U13 pad 1: +5V_YM2151 -> Net-(U13-Pad1)
- U13 pad 3: YM2151_IC -> GND_YM2151
- U13 pad 4: GND_YM2151 -> Net-(U13-Pad4)
- U13 pad 7: Net-(U13-Pad7) -> YM2151_IC
- U14 pad 1: Net-(U14-Pad1) -> Net-(U13-Pad13)
- U14 pad 4: AGND_YM2151 -> Net-(U14-Pad4)
- U14 pad 5: Net-(U13-Pad13) -> Net-(U13-Pad12)
- U14 pad 6: +5V_YM2151 -> Net-(R15-Pad1)
- U14 pad 7: Net-(U14-Pad7) -> Net-(R15-Pad1)
- U14 pad 8: Net-(U14-Pad8) -> YM2151_MOL
- U5 pad 19: Net-(U13-Pad7) -> Net-(U13-Pad6)
- U5 pad 20: Net-(U13-Pad6) -> Net-(U13-Pad5)
- U5 pad 21: Net-(U13-Pad5) -> Net-(U13-Pad4)
- U5 pad 22: +5V_YM2151 -> VDD_YM2151
- U7 pad 16: YM_RD -> VDD
- U8 pad 16: VDD -> +5V
- U9 pad 2: I2C_SDA -> SPI_CLK
- U9 pad 3: I2C_SCK -> SPI_MOSI
Other:
- outline, holes or cut-outs redrawn
- board text added: "VGM PLAYER V0.2"
- board text removed: "VGM PLAYER V0.1"
