File: Hardware/VGMPlayer/VGMPlayer.kicad_pcb (KiCad board)
At the start: 2 copper layers, 99.4 x 103.3 mm, 75 parts, among them J1 Conn_02x20_Counter_Clockwise, J2 Conn_02x20_Counter_Clockwise, J4 USB_B_Micro, U1 STC8951, U10 LTC6903, U11 HC-06, U12 7805-VGM, U13 YM3012, U14 LM324, U18 OLED_128_64_I2C, U19 ESP8266Module, U2 7805-VGM, U20 YM2612, U21 74HCT595, U22 74HCT595, U23 74HCT595, U3 LM386, U4 LM386, U5 YM2151, U6 AUDIOJACK-VGM, U7 YM2612, U8 SN76489, U9 LTC6903, Y1 11.0592MHz

Commit message: 1
Parts:
- removed C10, C33: 100nF, Capacitor_SMD:C_0805_2012Metric
- removed C13: 10nF, Capacitor_SMD:C_0805_2012Metric
- removed C16, C32: 10uF, Capacitor_THT:CP_Radial_D4.0mm_P1.50mm
- removed J2: Conn_02x20_Counter_Clockwise, Package_DIP:DIP-40_W15.24mm_Socket
- removed J4: USB_B_Micro, Connector_USB:USB_Micro-B_Molex-105017-0001
- removed R1: 10k, Resistor_SMD:R_0805_2012Metric
- removed U12: 7805-VGM, Package_TO_SOT_THT:TO-220-3_Vertical
- removed U20: YM2612, Package_DIP:DIP-24_W15.24mm_Socket
- removed U21, U22, U23: 74HCT595, Package_DIP:DIP-16_W7.62mm
- removed Y1: 11.0592MHz, Crystal:Crystal_HC49-4H_Vertical
- added D1: LED, LED_SMD:LED_0805_2012Metric, F.Cu at (113.8, 94.9)
- added D2: LED, LED_SMD:LED_0805_2012Metric, F.Cu at (117.2, 94.9)
- added D3: LED, LED_SMD:LED_0805_2012Metric, F.Cu at (120.7, 94.9)
- added D4: LED, LED_SMD:LED_0805_2012Metric, F.Cu at (104.7, 92.0)
- added D5: LED, LED_SMD:LED_0805_2012Metric, F.Cu at (126.4, 106.1)
- added D6: LED, LED_SMD:LED_0805_2012Metric, F.Cu at (126.4, 108.1)
- added D7: LED, LED_SMD:LED_0805_2012Metric, F.Cu at (129.8, 107.7)
- added D8: LED, LED_SMD:LED_0805_2012Metric, F.Cu at (133.3, 107.7)
- added RV1: 10k, Connector_PinHeader_2.54mm:PinHeader_1x03_P2.54mm_Vertical, F.Cu at (136.7, 76.5)
- added RV2: 10k, Connector_PinHeader_2.54mm:PinHeader_1x03_P2.54mm_Vertical, F.Cu at (133.1, 76.5)
- added SW1: Play/Suffle, Button_Switch_THT:SW_Tactile_Straight_KSA0Axx1LFTR, F.Cu at (143.4, 88.2)
- added SW2: Stop, Button_Switch_THT:SW_Tactile_Straight_KSA0Axx1LFTR, F.Cu at (173.4, 48.0)
- added SW3: Next/Pause, Button_Switch_THT:SW_Tactile_Straight_KSA0Axx1LFTR, F.Cu at (151.9, 69.0)
- added SW4: Prev/Resume, Button_Switch_THT:SW_Tactile_Straight_KSA0Axx1LFTR, F.Cu at (124.2, 79.2)
- C1: value 30pF -> 100uF; footprint Capacitor_SMD:C_0805_2012Metric -> Capacitor_THT:CP_Radial_D8.0mm_P3.50mm
- C2: value 10uF -> 100uF; footprint Capacitor_THT:CP_Radial_D4.0mm_P1.50mm -> Capacitor_THT:CP_Radial_D8.0mm_P3.50mm
- C3: value 30pF -> 1000uF; footprint Capacitor_SMD:C_0805_2012Metric -> Capacitor_THT:CP_Radial_D8.0mm_P3.50mm
- J1: value Conn_02x20_Counter_Clockwise -> USB_B_Mini; footprint Package_DIP:DIP-40_W15.24mm_Socket -> Connector_USB:USB_Micro-B_Wuerth_629105150521_CircularHoles
- L1, L2: value L -> 30uH
- U1: value STC8951 -> STM32F103XX
- U2: value 7805-VGM -> SDCardModule; footprint Package_TO_SOT_THT:TO-220-3_Vertical -> Connector_PinHeader_2.54mm:PinHeader_1x08_P2.54mm_Vertical
- moved U11 152.5 mm to (182.3, 45.3), turned to 0 degrees
- moved J1 140.0 mm to (189.4, 46.8)
- moved U1 124.4 mm to (30.2, 34.8), turned to 0 degrees
- moved C6 119.5 mm to (196.3, 45.7)
- moved C9 116.7 mm to (196.4, 49.0), turned to 0 degrees
- moved L2 116.5 mm to (188.0, 73.6), turned to 0 degrees
- moved C25 116.4 mm to (188.0, 69.7), turned to 0 degrees
- moved R2 113.2 mm to (196.8, 61.2), turned to 0 degrees
- moved C23 109.2 mm to (186.8, 55.9), turned to 0 degrees
- moved R14 107.6 mm to (196.8, 63.1)
- moved R9 106.3 mm to (196.8, 65.1), turned to 0 degrees
- moved L1 102.7 mm to (173.0, 89.3), turned to 0 degrees
- moved C17 102.7 mm to (195.5, 55.9)
- moved C24 101.4 mm to (171.6, 66.9), turned to 0 degrees
- moved C20 96.6 mm to (191.4, 69.7)
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Connections:
- net IRQ renamed Net-(U7-Pad13)
- C1 pad 1: GND_8051 -> VDD
- C1 pad 2: Net-(C1-Pad2) -> GND
- C2 pad 1: +5V_8051 -> +5V
- C2 pad 2: Net-(C2-Pad2) -> GNDA
- C24 pad 2: GND -> GNDA
- C25 pad 1: GND -> GNDA
- C25 pad 2: VDD -> +5V
- C26 pad 1: GND -> GNDA
- C26 pad 2: VDD -> +5V
- C27 pad 1: VDD -> +5V
- C27 pad 2: GND -> GNDA
- C28 pad 1: VDD -> +5V
- C28 pad 2: GND -> GNDA
- C29 pad 2: AGND_YM2151 -> GNDA
- C3 pad 1: GND_8051 -> +5V
- C3 pad 2: Net-(C3-Pad2) -> GNDA
- C30 pad 1: AGND_YM2151 -> GNDA
- C31 pad 1: AGND_YM2151 -> GNDA
- J1 pad 1: Net-(J1-Pad1) -> VDD
- J1 pad 5: D0 -> GND
- J1 pad 6: D1 -> GND
- R5 pad 1: Net-(C8-Pad1) -> Net-(R5-Pad1)
- R6 pad 1: Net-(C9-Pad1) -> Net-(R6-Pad1)
- R7 pad 1: Net-(C9-Pad1) -> Net-(R6-Pad1)
- R8 pad 1: Net-(C8-Pad1) -> Net-(R5-Pad1)
- RN1 pad 1: +5V_8051 -> VDD
- RN1 pad 2: P0.0 -> Net-(D1-Pad2)
- RN1 pad 3: P0.1 -> Net-(D2-Pad2)
- RN1 pad 4: P0.2 -> Net-(D3-Pad2)
- RN1 pad 5: P0.3 -> Net-(D4-Pad2)
- RN1 pad 6: P0.4 -> Net-(D5-Pad2)
- RN1 pad 7: P0.5 -> Net-(D6-Pad2)
- RN1 pad 8: P0.6 -> Net-(D7-Pad2)
- RN1 pad 9: P0.7 -> Net-(D8-Pad2)
- U1 pad 1: P1.0 -> Net-(U1-Pad1)
- U1 pad 10: P3.0 -> D5
- U1 pad 11: P3.1 -> D6
- U1 pad 12: P3.2 -> D7
- U1 pad 13: P3.3 -> YM_CS
- U1 pad 14: P3.4 -> YM_WR
- U1 pad 15: P3.5 -> YM_A0
- U1 pad 16: P3.6 -> YM_A1
- U1 pad 17: P3.7 -> Net-(U1-Pad17)
- U1 pad 18: Net-(C1-Pad2) -> Net-(U1-Pad18)
- U1 pad 19: Net-(C3-Pad2) -> GND
- U1 pad 2: P1.1 -> Net-(U1-Pad2)
- U1 pad 20: GND_8051 -> GND
- U1 pad 21: P2.0 -> YM_IC
- U1 pad 22: P2.1 -> SPI_CLK
- U1 pad 23: P2.2 -> SPI_MISO
- U1 pad 24: P2.3 -> SPI_MOSI
- U1 pad 25: P2.4 -> Play
- U1 pad 26: P2.5 -> TXD
- U1 pad 27: P2.6 -> RXD
- U1 pad 28: P2.7 -> Prev_Resume
- U1 pad 29: Net-(U1-Pad29) -> Next_Pause
- U1 pad 3: P1.2 -> Net-(U1-Pad3)
- U1 pad 30: Net-(U1-Pad30) -> Stop
- U1 pad 31: +5V_8051 -> Net-(U1-Pad31)
- U1 pad 32: P0.7 -> YM_CLK_CS
- U1 pad 33: P0.6 -> SD_CS
- U1 pad 34: P0.5 -> I2C_CLK
- U1 pad 35: P0.4 -> I2C_DAT
- U1 pad 36: P0.3 -> SN_WR
- U1 pad 37: P0.2 -> SN_CLK_CS
- U1 pad 38: P0.1 -> VDD
- U1 pad 39: P0.0 -> GND
- U1 pad 4: P1.3 -> Net-(U1-Pad4)
- U1 pad 40: +5V_8051 -> +3V3
- U1 pad 5: P1.4 -> D0
- U1 pad 6: P1.5 -> D1
- U1 pad 7: P1.6 -> D2
- U1 pad 8: P1.7 -> D3
- U1 pad 9: Net-(C2-Pad2) -> D4
- U10 pad 1: GND -> GNDA
- U10 pad 2: SPI_CLK -> SPI_MOSI
- U10 pad 3: SPI_MOSI -> SPI_CLK
- U10 pad 7: VDD -> +5V
- U10 pad 8: VDD -> +5V
- U13 pad 1: Net-(U13-Pad1) -> +5V
- U13 pad 14: Net-(U13-Pad13) -> Net-(U13-Pad14)
- U13 pad 16: AGND_YM2151 -> GNDA
- U13 pad 3: GND_YM2151 -> GND
- U13 pad 7: YM2151_IC -> YM_IC
- U13 pad 8: AGND_YM2151 -> GNDA
- U14 pad 11: Net-(U14-Pad11) -> GNDA
- U14 pad 13: YM2151_MOR -> YM_MOR
- U14 pad 14: YM2151_MOR -> YM_MOR
- U14 pad 2: Net-(U13-Pad13) -> Net-(U13-Pad14)
- U14 pad 4: Net-(U14-Pad4) -> +5V
- U14 pad 8: YM2151_MOL -> YM_MOL
- U14 pad 9: YM2151_MOL -> YM_MOL
- U18 pad 3: I2C_SCK -> I2C_CLK
- U18 pad 4: I2C_SDA -> I2C_DAT
- U2 pad 1: +5V_8051 -> GND
- U2 pad 2: GND_8051 -> SPI_MISO
- U2 pad 3: Net-(C16-Pad1) -> SPI_CLK
- U5 pad 1: GND_YM2151 -> GND
- U5 pad 10: YM2151_D0 -> D0
- U5 pad 11: GND_YM2151 -> GND
- U5 pad 12: YM2151_D1 -> D1
- U5 pad 13: YM2151_D2 -> D2
- U5 pad 14: YM2151_D3 -> D3
- U5 pad 15: YM2151_D4 -> D4
- U5 pad 16: YM2151_D5 -> D5
- U5 pad 17: YM2151_D6 -> D6
- U5 pad 18: YM2151_D7 -> D7
- U5 pad 2: YM2151_IRQ -> Net-(U5-Pad2)
- U5 pad 22: VDD_YM2151 -> VDD
- U5 pad 24: YM2151_CLK -> YM_CLK
- U5 pad 3: YM2151_IC -> YM_IC
- U5 pad 4: YM2151_A0 -> YM_A0
- U5 pad 5: YM2151_WR -> YM_WR
- U5 pad 6: YM2151_RD -> VDD
- U5 pad 7: YM2151_CS -> YM_CS
- U8 pad 6: GND -> GNDA
- U8 pad 8: GND -> GNDA
- U9 pad 1: GND -> GNDA
- U9 pad 2: SPI_CLK -> SPI_MOSI
- U9 pad 3: SPI_MOSI -> SPI_CLK
- U9 pad 7: VDD -> +5V
- U9 pad 8: VDD -> +5V
Other:
- board outline removed
- net class Default: clearance 0.25 -> 0.2
- rule pad_to_mask_clearance: 0.051 -> 0
- rule trace_clearance: 0.25 -> 0.2
- board text removed: "Designed By"
- board text removed: "Mac Lin"
- board text removed: "VGM PLAYER V0.2"

Commit message: 1
Parts:
- removed D8: LED, LED_SMD:LED_0805_2012Metric
- removed RN1: R_Network08, Resistor_THT:R_Array_SIP9
- added D0: LED, LED_SMD:LED_0805_2012Metric, F.Cu at (74.3, 69.5)
- added Q1: 9013, Package_TO_SOT_THT:TO-92, F.Cu at (31.1, 27.9)
- added Q2: S8550, Package_TO_SOT_THT:TO-92, F.Cu at (36.9, 26.8)
- added R1: 0, Resistor_SMD:R_0805_2012Metric, F.Cu at (47.2, 37.3)
- added R16: 0, Resistor_SMD:R_0805_2012Metric, F.Cu at (47.2, 52.6)
- added R17: 0, Resistor_SMD:R_0805_2012Metric, F.Cu at (47.2, 55.1)
- added R18: 330, Resistor_SMD:R_0805_2012Metric, F.Cu at (77.7, 56.1)
- added R19: 330, Resistor_SMD:R_0805_2012Metric, F.Cu at (77.7, 58.0)
- added R20: 330, Resistor_SMD:R_0805_2012Metric, F.Cu at (77.7, 59.9)
- added R21: 330, Resistor_SMD:R_0805_2012Metric, F.Cu at (77.7, 61.8)
- added R22: 330, Resistor_SMD:R_0805_2012Metric, F.Cu at (77.7, 63.8)
- added R23: 330, Resistor_SMD:R_0805_2012Metric, F.Cu at (77.7, 65.7)
- added R24: 330, Resistor_SMD:R_0805_2012Metric, F.Cu at (77.7, 67.6)
- added R25: 330, Resistor_SMD:R_0805_2012Metric, F.Cu at (77.7, 69.6)
- added R26: 47k, Resistor_SMD:R_0805_2012Metric, F.Cu at (37.0, 29.9)
- added R27: 1k, Resistor_SMD:R_0805_2012Metric, F.Cu at (34.1, 27.6)
- added R28: 4.7k, Resistor_SMD:R_0805_2012Metric, F.Cu at (30.1, 30.4)
- added SW5: PWR, Resistor_SMD:R_0805_2012Metric, F.Cu at (34.0, 90.6)
- SW1: value Play/Suffle -> Mode; footprint Button_Switch_THT:SW_Tactile_Straight_KSA0Axx1LFTR -> Resistor_SMD:R_0805_2012Metric
- SW2: value Stop -> NEXT; footprint Button_Switch_THT:SW_Tactile_Straight_KSA0Axx1LFTR -> Resistor_SMD:R_0805_2012Metric
- SW3: value Next/Pause -> PREV; footprint Button_Switch_THT:SW_Tactile_Straight_KSA0Axx1LFTR -> Resistor_SMD:R_0805_2012Metric
- SW4: value Prev/Resume -> SELECT; footprint Button_Switch_THT:SW_Tactile_Straight_KSA0Axx1LFTR -> Resistor_SMD:R_0805_2012Metric
- moved J1 167.7 mm to (22.8, 27.4), turned to 180 degrees
- moved U11 164.6 mm to (19.7, 71.0)
- moved L2 153.2 mm to (42.0, 27.3), turned to 270 degrees
- moved L1 145.0 mm to (40.7, 29.9)
- moved C25 135.4 mm to (59.4, 27.2), turned to 270 degrees
- moved SW2 128.8 mm to (51.9, 90.6)
- moved C27 123.8 mm to (56.6, 26.7), turned to 180 degrees
- moved C23 121.8 mm to (68.4, 27.1), turned to 180 degrees
- moved C31 110.7 mm to (89.4, 40.8), turned to 90 degrees
- moved C1 106.6 mm to (73.9, 27.1)
- moved C24 106.5 mm to (66.0, 81.0), turned to 180 degrees
- moved SW3 106.4 mm to (47.7, 90.6)
- moved R15 106.3 mm to (83.3, 53.1), turned to 180 degrees
- moved U9 104.6 mm to (57.2, 31.0)
- moved R2 103.9 mm to (94.1, 45.3), turned to 90 degrees
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Connections:
- D1 pad 1: D0 -> D1
- D2 pad 1: D1 -> D2
- D3 pad 1: D2 -> D3
- D4 pad 1: D3 -> D4
- D5 pad 1: D4 -> D5
- D6 pad 1: D5 -> D6
- D7 pad 1: D6 -> D7
- J1 pad 1: VDD -> Net-(J1-Pad1)
- SW1 pad 1: Play -> BUTTON_MODE
- SW2 pad 1: Stop -> BUTTON_NEXT
- SW3 pad 1: Next_Pause -> BUTTON_PREV
- SW4 pad 1: Prev_Resume -> BUTTON_SELECT
- U1 pad 25: Play -> BUTTON_SELECT
- U1 pad 28: Prev_Resume -> BUTTON_PREV
- U1 pad 29: Next_Pause -> BUTTON_NEXT
- U1 pad 30: Stop -> BUTTON_MODE
- U1 pad 31: Net-(U1-Pad31) -> PWR_HOLD
Routing:
- net GNDA: track 0.00 -> 333.8 mm
- net GND: track 0.00 -> 303.9 mm
- net +5V: track 0.00 -> 202.5 mm, vias 0 -> 1
- net VDD: track 0.00 -> 200.9 mm, vias 0 -> 1
- net SN_CLK_CS: track 0.00 -> 116.6 mm
- net D0: track 0.00 -> 110.5 mm
- net YM_A0: track 0.00 -> 105.4 mm, vias 0 -> 1
- net YM_IC: track 0.00 -> 102.5 mm, vias 0 -> 1
- net D1: track 0.00 -> 98.4 mm
- net SPI_CLK: track 0.00 -> 93.0 mm, vias 0 -> 1
- net D2: track 0.00 -> 89.4 mm, vias 0 -> 1
- net D3: track 0.00 -> 85.7 mm
- net SPI_MOSI: track 0.00 -> 84.5 mm, vias 0 -> 1
- net I2C_CLK: track 0.00 -> 83.5 mm
- net I2C_DAT: track 0.00 -> 80.8 mm
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Other:
- board outline added: 110.7 x 70.6 mm

Commit message: 1
Parts:
- added J2: SD_Card, Connector_Card:SD_TE_2041021, F.Cu at (63.2, 79.1)
- moved R18 66.5 mm to (19.1, 87.5), turned to 90 degrees
- moved D7 65.3 mm to (19.1, 91.0), turned to 90 degrees
- moved R19 63.9 mm to (21.0, 87.5), turned to 90 degrees
- moved D6 62.6 mm to (21.0, 91.0), turned to 90 degrees
- moved R20 61.3 mm to (23.0, 87.5), turned to 90 degrees
- moved D5 60.0 mm to (22.9, 91.0), turned to 90 degrees
- moved R21 58.7 mm to (24.9, 87.5), turned to 90 degrees
- moved D4 57.3 mm to (24.9, 91.0), turned to 90 degrees
- moved R22 56.2 mm to (26.8, 87.5), turned to 90 degrees
- moved D3 54.7 mm to (26.8, 91.0), turned to 90 degrees
- moved R23 53.6 mm to (28.7, 87.5), turned to 90 degrees
- moved D2 52.1 mm to (28.7, 91.0), turned to 90 degrees
- moved R24 51.1 mm to (30.7, 87.5), turned to 90 degrees
- moved SW4 50.6 mm to (106.6, 90.3)
- moved SW2 49.9 mm to (101.7, 90.3)
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Routing:
- net GNDA: track 333.8 -> 0.00 mm
- net GND: track 303.9 -> 0.00 mm
- net +5V: track 202.5 -> 0.00 mm, vias 1 -> 0
- net VDD: track 200.9 -> 0.00 mm, vias 1 -> 0
- net SN_CLK_CS: track 116.6 -> 0.00 mm
- net D0: track 110.5 -> 0.00 mm
- net YM_A0: track 105.4 -> 0.00 mm, vias 1 -> 0
- net YM_IC: track 102.5 -> 0.00 mm, vias 1 -> 0
- net D1: track 98.4 -> 0.00 mm
- net SPI_CLK: track 93.0 -> 0.00 mm, vias 1 -> 0
- net D2: track 89.4 -> 0.00 mm, vias 1 -> 0
- net D3: track 85.7 -> 0.00 mm
- net SPI_MOSI: track 84.5 -> 0.00 mm, vias 1 -> 0
- net I2C_CLK: track 83.5 -> 0.00 mm
- net I2C_DAT: track 80.8 -> 0.00 mm
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
Commit message: 1
Parts:
- moved U18 53.3 mm to (53.0, 117.7), turned to 90 degrees
- moved U6 39.2 mm to (117.9, 106.7)
- moved U3 39.0 mm to (99.3, 62.4)
- moved R13 39.0 mm to (99.4, 72.7)
- moved C19 38.9 mm to (106.7, 72.7)
- moved U4 38.8 mm to (117.7, 99.0)
- moved C20 38.8 mm to (110.2, 88.7)
- moved C21 38.8 mm to (114.4, 76.1)
- moved C15 38.8 mm to (112.6, 83.8)
- moved R14 38.8 mm to (117.7, 88.7)
- moved C18 38.5 mm to (101.3, 96.1)
- moved C22 38.5 mm to (103.1, 85.3)
- moved C14 38.5 mm to (104.7, 77.9)
- moved C17 38.0 mm to (115.5, 63.2)
- moved R18 35.5 mm to (35.5, 119.0), turned to 270 degrees
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Other:
- board size 110.7 x 70.6 mm -> 100 x 98.8 mm

Commit message: 1
Routing:
- net GNDA: track 0.00 -> 316.8 mm
- net GND: track 0.00 -> 312.6 mm
- net VDD: track 0.00 -> 272.0 mm, vias 0 -> 1
- net +5V: track 0.00 -> 229.0 mm, vias 0 -> 2
- net D1: track 0.00 -> 160.0 mm, vias 0 -> 1
- net D2: track 0.00 -> 159.4 mm, vias 0 -> 1
- net D0: track 0.00 -> 149.0 mm
- net Net-(Q1-Pad3): track 0.00 -> 144.3 mm, vias 0 -> 1
- net D7: track 0.00 -> 143.0 mm, vias 0 -> 1
- net D5: track 0.00 -> 139.1 mm, vias 0 -> 2
- net SPI_MOSI: track 0.00 -> 133.4 mm, vias 0 -> 1
- net SPI_CLK: track 0.00 -> 131.9 mm
- net D4: track 0.00 -> 128.2 mm, vias 0 -> 1
- net D6: track 0.00 -> 128.0 mm, vias 0 -> 2
- net D3: track 0.00 -> 125.3 mm, vias 0 -> 2
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- added copper zone on B.Cu, net (none)
- added copper zone on F.Cu, net (none)
- added copper zone on F.Cu, net GND

Commit message: 1
Parts:
- removed RV1, RV2: 10k, Connector_PinHeader_2.54mm:PinHeader_1x03_P2.54mm_Vertical
- removed U18: OLED_128_64_I2C, Connector_PinSocket_2.54mm:PinSocket_1x04_P2.54mm_Vertical
- added J3: LCD_PORT, Connector_PinSocket_2.54mm:PinSocket_2x15_P2.54mm_Vertical, F.Cu at (90.5, 113.5)
- added U12: R_POT_SW, Connector_Audio:VGM_VR_SW, F.Cu at (108.3, 119.1)
- SW1, SW2, SW3, SW4, SW5: footprint Resistor_SMD:R_0805_2012Metric -> Button_Switch_SMD:VGM_Button
- U6: footprint Connector_Audio:Jack_Horizontal -> Connector_Audio:VGMAudio_Jack
- moved D0 85.4 mm to (91.3, 65.7), turned to 180 degrees
- moved R25 84.7 mm to (87.8, 65.6), turned to 180 degrees
- moved D1 82.7 mm to (91.3, 67.6), turned to 180 degrees
- moved R24 82.0 mm to (87.8, 67.6), turned to 180 degrees
- moved D2 80.0 mm to (91.3, 69.5), turned to 180 degrees
- moved R23 79.3 mm to (87.8, 69.5), turned to 180 degrees
- moved D3 77.3 mm to (91.3, 71.4), turned to 180 degrees
- moved R22 76.6 mm to (87.8, 71.4), turned to 180 degrees
- moved D4 74.6 mm to (91.3, 73.4), turned to 180 degrees
- moved R21 73.9 mm to (87.8, 73.4), turned to 180 degrees
- moved D5 71.9 mm to (91.3, 75.3), turned to 180 degrees
- moved R20 71.2 mm to (87.8, 75.3), turned to 180 degrees
- moved D6 69.3 mm to (91.3, 77.2), turned to 180 degrees
- moved R19 68.5 mm to (87.8, 77.2), turned to 180 degrees
- moved D7 66.6 mm to (91.3, 79.2), turned to 180 degrees
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Connections:
- net Net-(J1-Pad1) renamed PWR_USB
- net YM_A0 renamed A0
- net YM_A1 renamed A1
- net YM_CS renamed ~YM_CS
- net YM_IC renamed ~RESET
- net YM_WR renamed ~WR
- J1 pad 5: GND -> GNDA
- J1 pad 6: GND -> GNDA
- J2 pad 1: SD_CS -> Net-(J2-Pad1)
- J2 pad 2: SPI_MOSI -> SD_CS
- J2 pad 3: GND -> SPI_MOSI
- J2 pad 4: +3V3 -> GND
- J2 pad 5: SPI_CLK -> +3V3
- J2 pad 6: GND -> SPI_CLK
- L1 pad 1: GNDA -> GND
- L1 pad 2: GND -> GNDA
- L2 pad 1: +5V -> VDD
- L2 pad 2: VDD -> +5V
- Q1 pad 2: GND -> GNDA
- Q2 pad 3: VDD -> +5V
- SW5 pad 1: GND -> GNDA
- U1 pad 35: I2C_DAT -> ~RD
- U5 pad 6: VDD -> Net-(U5-Pad6)
- U7 pad 16: VDD -> Net-(U7-Pad16)
Routing:
- net GNDA: track 316.8 -> 0.00 mm
- net GND: track 312.6 -> 0.00 mm
- net VDD: track 272.0 -> 0.00 mm, vias 1 -> 0
- net +5V: track 229.0 -> 0.00 mm, vias 2 -> 0
- net D1: track 160.0 -> 0.00 mm, vias 1 -> 0
- net D2: track 159.4 -> 0.00 mm, vias 1 -> 0
- net D0: track 149.0 -> 0.00 mm
- net Net-(Q1-Pad3): track 144.3 -> 0.00 mm, vias 1 -> 0
- net D7: track 143.0 -> 0.00 mm, vias 1 -> 0
- net D5: track 139.1 -> 0.00 mm, vias 2 -> 0
- net SPI_MOSI: track 133.4 -> 0.00 mm, vias 1 -> 0
- net SPI_CLK: track 131.9 -> 0.00 mm
- net D4: track 128.2 -> 0.00 mm, vias 1 -> 0
- net D6: track 128.0 -> 0.00 mm, vias 2 -> 0
- net D3: track 125.3 -> 0.00 mm, vias 2 -> 0
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- removed copper zone on B.Cu, net (none)
- removed copper zone on F.Cu, net (none)
- removed copper zone on F.Cu, net GND

Commit message: 1
Parts:
- moved SW5 8.94 mm to (47.3, 119.2)
- moved SW3 8.94 mm to (69.8, 119.1)
- moved SW1 8.94 mm to (60.8, 119.1)
- moved SW2 8.94 mm to (78.9, 119.1)
- moved SW4 8.94 mm to (88.0, 119.1)
- moved U12 8.15 mm to (100.1, 119.0)
- moved U6 4.68 mm to (111.0, 115.4)
- moved U2 1.22 mm to (49.6, 95.7)
Routing:
- net GNDA: track 0.00 -> 454.5 mm, vias 0 -> 1
- net +5V: track 0.00 -> 288.4 mm, vias 0 -> 1
- net GND: track 0.00 -> 286.4 mm
- net D7: track 0.00 -> 194.7 mm, vias 0 -> 1
- net VDD: track 0.00 -> 188.1 mm
- net D0: track 0.00 -> 183.7 mm, vias 0 -> 1
- net SPI_MOSI: track 0.00 -> 179.2 mm
- net ~WR: track 0.00 -> 167.9 mm, vias 0 -> 1
- net A0: track 0.00 -> 162.8 mm, vias 0 -> 1
- net D1: track 0.00 -> 161.2 mm
- net D2: track 0.00 -> 155.8 mm, vias 0 -> 1
- net D3: track 0.00 -> 145.1 mm, vias 0 -> 1
- net D4: track 0.00 -> 133.4 mm, vias 0 -> 1
- net +3V3: track 0.00 -> 133.0 mm, vias 0 -> 1
- net D5: track 0.00 -> 132.5 mm, vias 0 -> 1
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
Commit message: 1
Parts:
- added JP1: Jumper_NC_Small, Jumper:SolderJumper-2_P1.3mm_Open_RoundedPad1.0x1.5mm, F.Cu at (103.1, 111.5)
- added U15: STM32F103XX, Package_DIP:DIP-40_W15.24mm_Socket, F.Cu at (33.4, 33.9)
- moved J3 47.9 mm to (57.4, 79.0), turned to 90 degrees
- moved R25 43.0 mm to (106.4, 104.4), turned to 0 degrees
- moved D0 40.4 mm to (102.9, 104.4), turned to 0 degrees
- moved R24 39.6 mm to (106.4, 102.5), turned to 0 degrees
- moved D1 36.8 mm to (102.9, 102.5), turned to 0 degrees
- moved R23 36.2 mm to (106.4, 100.6), turned to 0 degrees
- moved D2 33.1 mm to (102.9, 100.5), turned to 0 degrees
- moved R22 32.9 mm to (106.4, 98.6), turned to 0 degrees
- moved R21 29.8 mm to (106.4, 96.7), turned to 0 degrees
- moved D3 29.5 mm to (102.9, 98.6), turned to 0 degrees
- moved R1 28.7 mm to (53.3, 65.9), turned to 0 degrees
- moved R20 26.9 mm to (106.4, 94.8), turned to 0 degrees
- moved D4 26.0 mm to (102.9, 96.7), turned to 0 degrees
- moved R19 24.3 mm to (106.4, 92.8), turned to 0 degrees
- moved D5 22.7 mm to (102.9, 94.8), turned to 0 degrees
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Connections:
- J2 pad 5: +3V3 -> Net-(J2-Pad5)
- J2 pad 6: SPI_CLK -> +3V3
- J2 pad 7: SPI_MISO -> SPI_CLK
- J2 pad 8: Net-(J2-Pad8) -> GND
- J2 pad 9: Net-(J2-Pad9) -> SPI_MISO
- U1 pad 31: PWR_HOLD -> ~VGM_CS
- U1 pad 33: SD_CS -> ~SD_CS
- U1 pad 34: I2C_CLK -> ~LCD_CS
- U2 pad 5: SD_CS -> ~SD_CS
- U5 pad 24: YM_CLK -> SN_CLK
Routing:
- net GNDA: track 454.5 -> 0.00 mm, vias 1 -> 0
- net +5V: track 288.4 -> 0.00 mm, vias 1 -> 0
- net GND: track 286.4 -> 0.00 mm
- net D7: track 194.7 -> 0.00 mm, vias 1 -> 0
- net VDD: track 188.1 -> 0.00 mm
- net D0: track 183.7 -> 0.00 mm, vias 1 -> 0
- net SPI_MOSI: track 179.2 -> 0.00 mm
- net ~WR: track 167.9 -> 0.00 mm, vias 1 -> 0
- net A0: track 162.8 -> 0.00 mm, vias 1 -> 0
- net D1: track 161.2 -> 0.00 mm
- net D2: track 155.8 -> 0.00 mm, vias 1 -> 0
- net D3: track 145.1 -> 0.00 mm, vias 1 -> 0
- net D4: track 133.4 -> 0.00 mm, vias 1 -> 0
- net +3V3: track 133.0 -> 0.00 mm, vias 1 -> 0
- net D5: track 132.5 -> 0.00 mm, vias 1 -> 0
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