File: Hardware/VGMPlayer/VGMPlayer.kicad_pcb (KiCad board)
At the start: 2 copper layers, 100 x 98.8 mm, 93 parts, among them J1 USB_B_Mini, J2 SD_Card, J3 LCD_PORT, Q1 9013, Q2 S8550, SW1 Mode, SW2 NEXT, SW3 PREV, SW4 SELECT, SW5 PWR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

Commit message: 1
Parts:
- removed JP1: Jumper_NC_Small, Jumper:SolderJumper-2_P1.3mm_Open_RoundedPad1.0x1.5mm
- removed U15: STM32F103XX, Package_DIP:DIP-40_W15.24mm_Socket
- added C10: 1000uF, Capacitor_THT:CP_Radial_D8.0mm_P3.50mm, F.Cu at (53.7, 69.0)
- added JP2: Jumper_NC_Small, Jumper:SolderJumper-2_P1.3mm_Open_RoundedPad1.0x1.5mm, F.Cu at (35.6, 58.6)
- added JP3: Jumper_NC_Small, Jumper:SolderJumper-2_P1.3mm_Open_RoundedPad1.0x1.5mm, F.Cu at (35.6, 62.3)
- added JP4: Jumper_NC_Small, Jumper:SolderJumper-2_P1.3mm_Open_RoundedPad1.0x1.5mm, F.Cu at (35.6, 66.0)
- added JP5: Jumper_NC_Small, Jumper:SolderJumper-2_P1.3mm_Open_RoundedPad1.0x1.5mm, F.Cu at (35.6, 69.6)
- moved R1 27.8 mm to (50.5, 38.2), turned to 270 degrees
- moved R16 15.6 mm to (50.0, 52.6), turned to 180 degrees
- moved R17 15.0 mm to (49.9, 55.1), turned to 180 degrees
- moved R6 12.4 mm to (95.5, 48.9), turned to 270 degrees
- moved D2 10.4 mm to (100.9, 90.3)
- moved D0 10.4 mm to (100.9, 94.2)
- moved R24 10.4 mm to (104.3, 92.3)
- moved R18 10.4 mm to (104.3, 80.7)
- moved R19 10.4 mm to (104.3, 82.6)
- moved R20 10.4 mm to (104.3, 84.5)
- moved R21 10.4 mm to (104.3, 86.5)
- moved R22 10.4 mm to (104.3, 88.4)
- moved D3 10.4 mm to (100.9, 88.4)
- moved D4 10.4 mm to (100.9, 86.4)
- moved D5 10.4 mm to (100.9, 84.5)
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Connections:
- C25 pad 2: +5V -> VDD
- C26 pad 2: +5V -> VDD
- C27 pad 1: +5V -> VDD
- C28 pad 1: +5V -> VDD
- J2 pad 11: Net-(J2-Pad11) -> GND
- R18 pad 2: VDD -> +5V
- R19 pad 2: VDD -> +5V
- R20 pad 2: VDD -> +5V
- R21 pad 2: VDD -> +5V
- R22 pad 2: VDD -> +5V
- R23 pad 2: VDD -> +5V
- R24 pad 2: VDD -> +5V
- R25 pad 2: VDD -> +5V
- U10 pad 7: +5V -> VDD
- U10 pad 8: +5V -> VDD
- U11 pad 2: VDD -> +3V3
- U12 pad 7: +5V -> Net-(U12-Pad7)
- U12 pad 8: PWR_USB -> Net-(U12-Pad8)
- U19 pad 2: VDD -> +3V3
- U5 pad 24: SN_CLK -> YM_CLK
- U9 pad 7: +5V -> VDD
- U9 pad 8: +5V -> VDD
Routing:
- net GNDA: track 0.00 -> 442.4 mm
- net GND: track 0.00 -> 330.2 mm
- net +5V: track 0.00 -> 225.4 mm
- net A0: track 0.00 -> 204.4 mm, vias 0 -> 1
- net VDD: track 0.00 -> 168.1 mm, vias 0 -> 2
- net +3V3: track 0.00 -> 148.4 mm
- net Net-(Q1-Pad3): track 0.00 -> 147.5 mm, vias 0 -> 1
- net D0: track 0.00 -> 141.1 mm
- net D2: track 0.00 -> 136.4 mm
- net D1: track 0.00 -> 133.6 mm, vias 0 -> 1
- net YM_MOL: track 0.00 -> 127.2 mm
- net SPI_CLK: track 0.00 -> 122.3 mm, vias 0 -> 2
- net Net-(R6-Pad1): track 0.00 -> 121.0 mm
- net SPI_MOSI: track 0.00 -> 120.1 mm, vias 0 -> 1
- net D4: track 0.00 -> 120.1 mm, vias 0 -> 2
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Other:
- net class POWER added: clearance 0.2, trace_width 0.4, via_dia 0.8, via_drill 0.4
- board text added: "VGM Player v0.9 Designed By Mac Lin"

Commit message: 1
Connections:
- J3 pad 4: Net-(J3-Pad4) -> +3V3
Routing:
- net +3V3: track 148.4 -> 150.9 mm

Commit message: 1
Parts:
- removed JP2, JP3, JP4, JP5: Jumper_NC_Small, Jumper:SolderJumper-2_P1.3mm_Open_RoundedPad1.0x1.5mm
- added C100: TBD, Capacitor_SMD:C_0805_2012Metric, F.Cu at (95.4, 34.5)
- added C101: TBD, Capacitor_SMD:C_0805_2012Metric, F.Cu at (81.7, 34.1)
- added R100: TBD, Resistor_SMD:R_0805_2012Metric, F.Cu at (95.3, 38.6)
- added R101: TBD, Resistor_SMD:R_0805_2012Metric, F.Cu at (85.8, 34.1)
- added R102: TBD, Resistor_SMD:R_0805_2012Metric, F.Cu at (42.6, 41.0)
- added R103: TBD, Resistor_SMD:R_0805_2012Metric, F.Cu at (42.6, 37.4)
- moved SW5 108.5 mm to (117.3, 43.5), turned to 90 degrees
- moved U12 90.0 mm to (118.0, 30.8), turned to 270 degrees
- moved U6 88.2 mm to (100.6, 27.8), turned to 0 degrees
- moved SW1 65.8 mm to (117.3, 90.3), turned to 90 degrees
- moved SW4 65.5 mm to (117.3, 60.2), turned to 90 degrees
- moved SW3 62.6 mm to (117.3, 80.3), turned to 90 degrees
- moved SW2 62.5 mm to (117.3, 70.2), turned to 90 degrees
- moved U19 47.8 mm to (56.8, 82.6), turned to 270 degrees
- moved J3 41.3 mm to (67.4, 118.9), turned to 180 degrees
- moved U11 39.2 mm to (56.7, 86.3), turned to 270 degrees
- moved R18 33.4 mm to (117.7, 111.3)
- moved D7 33.4 mm to (114.2, 111.3)
- moved R19 29.9 mm to (117.7, 109.3)
- moved D6 29.9 mm to (114.2, 109.3)
- moved R20 26.5 mm to (117.7, 107.4)
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Routing:
- net Net-(C9-Pad1): track 119.2 -> 12.9 mm
- net D1: track 133.6 -> 232.0 mm, vias 1 -> 0
- net A0: track 204.4 -> 115.8 mm, vias 1 -> 0
- net Net-(R5-Pad1): track 116.0 -> 34.8 mm, vias 0 -> 1
- net GNDA: track 442.4 -> 362.3 mm
- net Net-(R6-Pad1): track 121.0 -> 51.7 mm, vias 0 -> 1
- net D7: track 119.7 -> 186.2 mm, vias 3 -> 2
- net D6: track 117.3 -> 182.5 mm, vias 1 -> 0
- net Net-(C8-Pad1): track 95.8 -> 30.8 mm
- net D5: track 103.7 -> 168.5 mm
- net RXD: track 74.9 -> 18.4 mm
- net D3: track 111.6 -> 165.0 mm, vias 0 -> 1
- net A1: track 54.5 -> 100.8 mm
- net YM_MOL: track 127.2 -> 85.7 mm
- net D2: track 136.4 -> 173.9 mm, vias 0 -> 1
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- added copper zone on F.Cu, net (none)
- added copper zone on B.Cu, net GND
- added copper zone on F.Cu, net GND

Commit message: 1
Parts:
- added R29: TBD, Resistor_SMD:R_0805_2012Metric, F.Cu at (75.5, 116.1)
- added R30: TBD, Resistor_SMD:R_0805_2012Metric, F.Cu at (75.5, 118.1)
- moved C10 52.9 mm to (77.7, 112.0), turned to 90 degrees
- moved J3 0.76 mm to (67.4, 118.1)
Connections:
- C10 pad 1: +3V3 -> Net-(C10-Pad1)
- J3 pad 2: +3V3 -> Net-(C10-Pad1)
- J3 pad 4: +3V3 -> Net-(C10-Pad1)
Routing:
- net +5V: track 239.1 -> 309.5 mm
- net D4: track 153.4 -> 197.9 mm, vias 2 -> 1
- net SPI_CLK: track 144.3 -> 108.4 mm, vias 2 -> 1
- net SN_CLK_CS: track 94.5 -> 59.8 mm, vias 0 -> 1
- net D1: track 232.0 -> 201.3 mm, vias 0 -> 1
- net VDD: track 180.0 -> 152.3 mm, vias 0 -> 1
- net BUTTON_SELECT: track 84.9 -> 112.5 mm, vias 0 -> 1
- net SPI_MOSI: track 136.1 -> 108.8 mm
- net D3: track 165.0 -> 185.9 mm, vias 1 -> 0
- net Net-(C10-Pad1): track 0.00 -> 20.2 mm
- net GND: track 361.3 -> 341.8 mm, vias 0 -> 1
- net YM_MOR: track 76.9 -> 57.8 mm
- net Net-(R5-Pad1): track 34.8 -> 49.5 mm, vias 1 -> 0
- net A1: track 100.8 -> 87.6 mm
- net D7: track 186.2 -> 173.2 mm, vias 2 -> 1
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- added copper zone on B.Cu, net (none)
- removed copper zone on B.Cu, net GND
- removed copper zone on F.Cu, net GND
