File: Hardware/VGMPlayer/VGMPlayer.sch (KiCad schematic (older format))
At the start: 59 parts, among them J1 USB_B_Mini, J2 Conn_01x20_Male, J3 Conn_01x20_Male, U1 STC8951, U10 LTC6903, U11 HC-06, U2 LD1117, U3 LM386, U4 LM386, U5 OLED_128_64_I2C, U6 AUDIOJACK, U7 YM2612, U8 SN76489, U9 LTC6903, Y1 11.0592MHz

Commit message: asdasd
Parts:
- U1: symbol VGM:STC8951 -> VGMPlayer-rescue:STC8951-VGM
- U10, U9: symbol VGM:LTC6903 -> VGMPlayer-rescue:LTC6903-VGM
- U11: symbol VGM:HC-06 -> VGMPlayer-rescue:HC-06-VGM
- U2: symbol VGM:LD1117 -> VGMPlayer-rescue:LD1117-VGM
- U5: symbol VGM:OLED_128_64_I2C -> VGMPlayer-rescue:OLED_128_64_I2C-VGM
- U6: symbol VGM:AUDIOJACK -> VGMPlayer-rescue:AUDIOJACK-VGM
- U7: symbol VGM:YM2612 -> VGMPlayer-rescue:YM2612-VGM
- U8: symbol VGM:SN76489 -> VGMPlayer-rescue:SN76489-VGM
Connections:
- net labels added: ALE, EA, PSEN, RST, XTAL1, XTAL2
- wire segments 324 -> 337
Changed lines of the file:
@@
 $EndComp
 $Comp
-L VGM:AUDIOJACK U6
+L VGMPlayer-rescue:AUDIOJACK-VGM U6
 U 1 1 5C00BAD0
 P 7650 8750
@@
 $EndComp
 $Comp
-L VGM:LD1117 U2
+L VGMPlayer-rescue:LD1117-VGM U2
 U 1 1 5C00BB96
 P 4500 6900
@@
 $EndComp
 $Comp
-L VGM:OLED_128_64_I2C U5
+L VGMPlayer-rescue:OLED_128_64_I2C-VGM U5
 U 1 1 5C00BCE4
 P 6750 7000
@@
 $EndComp
 $Comp
-L VGM:SN76489 U8
+L VGMPlayer-rescue:SN76489-VGM U8
 U 1 1 5C00BD65
 P 9550 9700
@@
 $EndComp
 $Comp
-L VGM:YM2612 U7
+L VGMPlayer-rescue:YM2612-VGM U7
 U 1 1 5C00BE09
 P 9550 8300
@@
 	10050 9700 10450 9700
 $Comp
-L VGM:LTC6903 U9
+L VGMPlayer-rescue:LTC6903-VGM U9
 U 1 1 5C1B9B2C
 P 12450 8300
@@
 $EndComp
 $Comp
-L VGM:LTC6903 U10
+L VGMPlayer-rescue:LTC6903-VGM U10
 U 1 1 5C266C0B
 P 12450 9400
@@
 	11800 8800 11800 9400
 $Comp
-L VGM:HC-06 U11
+L VGMPlayer-rescue:HC-06-VGM U11
 U 1 1 5C125DAA
 P 14700 8900
@@
 	2950 9900 3300 9900
 $Comp
-L VGM:STC8951 U1
+L VGMPlayer-rescue:STC8951-VGM U1
 U 1 1 5C2DD3EE
 P 2700 4600
@@
 	1350 6000 1350 5900
 Wire Wire Line
-	1350 5900 2200 5900
+	1350 5900 1700 5900
 Text GLabel 1850 4100 0    50   Input ~ 0
 YM_D0
@@
 	4800 5000 4800 4100
 Wire Wire Line
-	850  5800 2200 5800
+	850  5800 1800 5800
 Connection ~ 850  6000
 Wire Wire Line
@@
 Wire Wire Line
 	3600 4100 4800 4100
+Text GLabel 3950 5200 2    50   Input ~ 0
+PSEN
+Text GLabel 3950 5100 2    50   Input ~ 0
+ALE
+Wire Wire Line
+	3950 5200 3600 5200
+Wire Wire Line
+	3950 5100 3600 5100
+Text GLabel 6950 5200 2    50   Input ~ 0
+PSEN
+Text GLabel 6950 5100 2    50   Input ~ 0
+ALE
+Text GLabel 6950 5000 2    50   Input ~ 0
+EA
+Wire Wire Line
+	6950 5000 6650 5000
+Wire Wire Line
+	6950 5100 6650 5100
+Wire Wire Line
+	6650 5200 6950 5200
+Text GLabel 1250 4900 0    50   Input ~ 0
+RST
+Wire Wire Line
+	1350 4900 1250 4900
+Text GLabel 1700 6000 3    50   Input ~ 0
+XTAL1
+Text GLabel 1800 6000 3    50   Input ~ 0
+XTAL2
+Wire Wire Line
+	1800 5800 1800 6000
+Connection ~ 1800 5800
+Wire Wire Line
+	1800 5800 2200 5800
+Wire Wire Line
+	1700 5900 1700 6000
+Connection ~ 1700 5900
+Wire Wire Line
+	1700 5900 2200 5900
+Text GLabel 5800 4900 0    50   Input ~ 0
+RST
+Wire Wire Line
+	5800 4900 6150 4900
+Text GLabel 5800 5800 0    50   Input ~ 0
+XTAL2
+Text GLabel 5800 5900 0    50   Input ~ 0
+XTAL1
+Wire Wire Line
+	6150 5800 5800 5800
+Wire Wire Line
+	5800 5900 6150 5900
 $EndSCHEMATC

Commit message: PCB
Parts:
- removed J1: USB_B_Mini, Connector_USB:USB_Mini-B_Lumberg_2486_01_Horizontal, symbol Connector:USB_B_Mini
- removed JP1: SolderJumper_2_Bridged, Jumper:SolderJumper-2_P1.3mm_Bridged_RoundedPad1.0x1.5mm, symbol Jumper:SolderJumper_2_Bridged
- removed U2: LD1117, Package_TO_SOT_THT:TO-220-3_Vertical, symbol VGMPlayer-rescue:LD1117-VGM
- added J1: USB_B_Micro, Connector_USB:USB_Micro-B_Amphenol_10103594-0001LF_Horizontal, symbol Connector:USB_B_Micro
- added JP1, JP10, JP11, JP12, JP13, JP14, JP15, JP16, JP2, JP3, JP4, JP5, JP6, JP7, JP8, JP9: Jumper_NC_Small, Jumper:SolderJumper-2_P1.3mm_Open_TrianglePad1.0x1.5mm, symbol Device:Jumper_NC_Small
- added R15: 0, Resistor_SMD:R_0805_2012Metric, symbol Device:R
- added U2: 7805-VGM, Package_TO_SOT_THT:TO-220-3_Vertical, symbol VGMPlayer-rescue:7805-VGM
- C11, C12, C16, C2, C27, C28, C5, C6, C7: footprint Capacitor_THT:CP_Axial_L18.0mm_D10.0mm_P25.00mm_Horizontal -> Capacitor_THT:CP_Radial_D4.0mm_P1.50mm
- C14, C15, C17, C18: footprint Capacitor_THT:CP_Axial_L18.0mm_D10.0mm_P25.00mm_Horizontal -> Capacitor_THT:CP_Radial_D8.0mm_P3.50mm
- C21, C22, C23, C24: footprint Capacitor_THT:C_Axial_L17.0mm_D7.0mm_P20.00mm_Horizontal -> Capacitor_THT:CP_Radial_D8.0mm_P3.50mm
- U6: value AUDIOJACK -> AUDIOJACK-VGM; footprint Connector_Audio:Jack_3.5mm_PJ31060-I_Horizontal -> Connector_Audio:Jack_Horizontal
Connections:
- net labels added: P2.0, P2.1, P2.2, P2.3, P2.4, P2.5, P2.6, P2.7
- wire segments 337 -> 371

Commit message: ewsd
Parts:
- added D1, D10, D11, D12, D13, D14, D15, D16, D17, D18, D19, D2, D20, D21, D22, D23, D24, D25, D26, D27, D28, D29, D3, D30, D31, D32, D4, D5, D6, D7, D8, D9: LED, LED_SMD:LED_0805_2012Metric, symbol Device:LED
- added J4, J5: Conn_01x20_Male, Connector_PinSocket_2.54mm:PinSocket_1x20_P2.54mm_Vertical, symbol Connector:Conn_01x20_Male
- added R16, R17, R18, R19, R20, R21, R22, R23, R24, R25, R26, R27, R28, R29, R30, R31, R32, R33, R34, R35, R36, R37, R38, R39, R40, R41, R42, R43, R44, R45, R46, R47: 1k, Resistor_SMD:R_0805_2012Metric, symbol Device:R
Connections:
- wire segments 371 -> 502

Commit message: 1
Parts:
- removed J1: USB_B_Micro, Connector_USB:USB_Micro-B_Amphenol_10103594-0001LF_Horizontal, symbol Connector:USB_B_Micro
- added C29, C30, C31, C32, C33, C34, C35, C36, C37, C38, C39, C40: 22pF, Capacitor_SMD:C_0805_2012Metric, symbol Device:C
- added J1: Barrel_Jack_Switch, Connector_BarrelJack:BarrelJack_Horizontal, symbol Connector:Barrel_Jack_Switch
- added R48, R49, R50, R51, R52, R53: 1M, Resistor_SMD:R_0805_2012Metric, symbol Device:R
- added U12: 74HC04, symbol 74xx:74HC04
- added Y2, Y3, Y4, Y5, Y6, Y7: 7.67Mhz, Crystal:Crystal_HC49-4H_Vertical, symbol Device:Crystal
Connections:
- net labels added: SN_CLK, YM_CLK
- wire segments 502 -> 561
Other:
- moved on the sheet: C23, C24, C25, C26, C27, C28, U6, U8

Commit message: 1
Parts:
- removed C29, C34, C35, C36, C37, C38, C39, C40: 22pF, Capacitor_SMD:C_0805_2012Metric, symbol Device:C
- removed D1, D10, D11, D12, D13, D14, D15, D16, D17, D18, D19, D2, D20, D21, D22, D23, D24, D25, D26, D27, D28, D29, D3, D30, D31, D32, D4, D5, D6, D7, D8, D9: LED, LED_SMD:LED_0805_2012Metric, symbol Device:LED
- removed J1: Barrel_Jack_Switch, Connector_BarrelJack:BarrelJack_Horizontal, symbol Connector:Barrel_Jack_Switch
- removed J2, J3, J4, J5: Conn_01x20_Male, Connector_PinSocket_2.54mm:PinSocket_1x20_P2.54mm_Vertical, symbol Connector:Conn_01x20_Male
- removed JP1, JP10, JP11, JP12, JP13, JP14, JP15, JP16, JP2, JP3, JP4, JP5, JP6, JP7, JP8, JP9: Jumper_NC_Small, Jumper:SolderJumper-2_P1.3mm_Open_TrianglePad1.0x1.5mm, symbol Device:Jumper_NC_Small
- removed R18, R19, R20, R21, R22, R23, R24, R25, R26, R27, R28, R29, R30, R31, R32, R33, R34, R35, R36, R37, R38, R39, R40, R41, R42, R43, R44, R45, R46, R47: 1k, Resistor_SMD:R_0805_2012Metric, symbol Device:R
- removed R48, R49, R50, R53: 1M, Resistor_SMD:R_0805_2012Metric, symbol Device:R
- removed U11: HC-06, Connector_PinSocket_2.54mm:PinSocket_1x04_P2.54mm_Vertical, symbol VGMPlayer-rescue:HC-06-VGM
- removed U5: OLED_128_64_I2C, Connector_PinSocket_2.54mm:PinSocket_1x04_P2.54mm_Vertical, symbol VGMPlayer-rescue:OLED_128_64_I2C-VGM
- removed Y3, Y4, Y6, Y7: 7.67Mhz, Crystal:Crystal_HC49-4H_Vertical, symbol Device:Crystal
- added C29: 10uF, Capacitor_THT:CP_Radial_D8.0mm_P3.50mm, symbol Device:CP1
- added J1, J2: Conn_02x20_Odd_Even, Connector_PinSocket_2.00mm:PinSocket_2x20_P2.00mm_Vertical, symbol Connector_Generic:Conn_02x20_Odd_Even
- added J4: USB_B_Micro, Connector_USB:USB_Micro-B_Molex-105017-0001, symbol Connector:USB_B_Micro
- added L1, L2: L, Inductor_SMD:L_0805_2012Metric, symbol Device:L
- added U11: HC-06, Connector_PinSocket_2.54mm:PinSocket_1x06_P2.54mm_Vertical, symbol VGMPlayer-rescue:HC-06
- added unit 7 of U12
- added U13: YM3012, Package_DIP:DIP-16_W7.62mm_Socket, symbol VGMPlayer-rescue:YM3012
- added U14, U15, U16, U17: LM386, Package_DIP:DIP-8_W7.62mm_Socket, symbol Amplifier_Audio:LM386
- added U18: OLED_128_64_I2C, Connector_PinSocket_2.54mm:PinSocket_1x04_P2.54mm_Vertical, symbol VGMPlayer-rescue:OLED_128_64_I2C-VGM
- added U19: ESP8266Module, Connector_PinSocket_2.54mm:PinSocket_1x06_P2.54mm_Vertical, symbol VGMPlayer-rescue:ESP8266Module
- added U20: YM2612, Package_DIP:DIP-24_W15.24mm_Socket, symbol VGMPlayer-rescue:YM2612-VGM
- added U5: YM2151, Package_DIP:DIP-24_W15.24mm_Socket, symbol VGMPlayer-rescue:YM2151
- C30, C31: value 22pF -> 1.5nF
- C32, C33: value 22pF -> 33pF
- R15: value 0 -> 270
- R51, R52: value 1M -> 1k
- U12: footprint (none) -> VGM:SOP-14_4.4x8.3mm_P1.27mm
- Y2: value 7.67Mhz -> 3.768Mhz
Connections:
- net labels added: +3V3_8051, +5V_8051, +5V_YM2151, AGND_YM2151, D0, D1, D2, D3, D4, D5, D6, D7, GNDA, GND_8051, GND_YM2151, P0.0, P0.1, P0.2, P1.0, P1.1, P1.2, P1.3, P1.4, P1.5, P1.6, P1.7, P3.0, P3.1, P3.2, P3.3, P3.4, P3.5, P3.6, P3.7, VDD, VDD_YM2151, YM2151_A0, YM2151_A1, YM2151_CLK, YM2151_CS, YM2151_D0, YM2151_D1, YM2151_D2, YM2151_D3, YM2151_D4, YM2151_D5, YM2151_D6, YM2151_D7, YM2151_IC, YM2151_IRQ, YM2151_MOL, YM2151_MOR, YM2151_RD, YM2151_WR
- net labels removed: ALE, EA, IIC_SCK, IIC_SDA, PSEN, RST, SN_D0, SN_D1, SN_D2, SN_D3, SN_D4, SN_D5, SN_D6, SN_D7, VCC, XTAL1, XTAL2, YM_D0, YM_D1, YM_D2, YM_D3, YM_D4, YM_D5, YM_D6, YM_D7
- wire segments 561 -> 572
Other:
- moved on the sheet: C1, C10, C11, C12, C13, C14, C15, C16, C17, C18, C19, C2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

Commit message: 1
Parts:
- removed C32: 33pF, Capacitor_SMD:C_0805_2012Metric, symbol Device:C
- removed J1, J2: Conn_02x20_Odd_Even, Connector_PinSocket_2.00mm:PinSocket_2x20_P2.00mm_Vertical, symbol Connector_Generic:Conn_02x20_Odd_Even
- removed R16, R17, R51, R52: 1k, Resistor_SMD:R_0805_2012Metric, symbol Device:R
- removed U12: 74HC04, VGM:SOP-14_4.4x8.3mm_P1.27mm, symbol 74xx:74HC04
- removed U14, U15, U16, U17: LM386, Package_DIP:DIP-8_W7.62mm_Socket, symbol Amplifier_Audio:LM386
- removed Y2: 3.768Mhz, Crystal:Crystal_HC49-4H_Vertical, symbol Device:Crystal
- removed Y5: 7.67Mhz, Crystal:Crystal_HC49-4H_Vertical, symbol Device:Crystal
- added C32: 10uF, Capacitor_THT:CP_Radial_D4.0mm_P1.50mm, symbol Device:CP1
- added J1, J2: Conn_02x20_Counter_Clockwise, Package_DIP:DIP-40_W15.24mm_Socket, symbol Connector_Generic:Conn_02x20_Counter_Clockwise
- added U12: 7805-VGM, Package_TO_SOT_THT:TO-220-3_Vertical, symbol VGMPlayer-rescue:7805-VGM
- added U14: LM324, Package_DIP:DIP-14_W7.62mm, symbol Amplifier_Operational:LM324
- added U21, U22, U23: 74HCT595, Package_DIP:DIP-16_W7.62mm, symbol 74xx:74HCT595
- C33: value 33pF -> 100nF
Connections:
- net labels added: +3.3V, +3V_8051, I2C_CLK, I2C_DAT, PP_CLK, PP_CLK1, PP_DAT, PP_DAT1, PP_LATCH, PP_LATCH1, SPI_CLK, SPI_MOSI
- net labels removed: +3V3_8051, YM_RD
- wire segments 572 -> 553
Other:
- moved on the sheet: C1, C13, C2, C23, C24, C25, C26, C27, C28, C3, L1, R1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

Commit message: 1
Parts:
- removed U21, U22, U23: 74HCT595, Package_DIP:DIP-16_W7.62mm, symbol 74xx:74HCT595
Connections:
- net I2C_CLK: now also J1.25 (Pin_25); no longer J1.32 (Pin_32)
- net I2C_DAT: now also J1.24 (Pin_24); no longer J1.31 (Pin_31)
- net SN_WR: now also J1.22 (Pin_22); no longer J1.35 (Pin_35)
- new net SD_CS: J1.32 (Pin_32)
- new net SPI_MISO: J1.35 (Pin_35)
- new net TBD_CS: J1.31 (Pin_31)
Other:
- moved on the sheet: J2, U18

Commit message: 1
Parts:
- removed C1, C3: 30pF, Capacitor_SMD:C_0805_2012Metric, symbol Device:C
- removed C10, C33: 100nF, Capacitor_SMD:C_0805_2012Metric, symbol Device:C
- removed C13: 10nF, Capacitor_SMD:C_0805_2012Metric, symbol Device:C
- removed C16, C32: 10uF, Capacitor_THT:CP_Radial_D4.0mm_P1.50mm, symbol Device:CP1
- removed J1, J2: Conn_02x20_Counter_Clockwise, Package_DIP:DIP-40_W15.24mm_Socket, symbol Connector_Generic:Conn_02x20_Counter_Clockwise
- removed J4: USB_B_Micro, Connector_USB:USB_Micro-B_Molex-105017-0001, symbol Connector:USB_B_Micro
- removed R1: 10k, Resistor_SMD:R_0805_2012Metric, symbol Device:R
- removed U1: STC8951, Package_DIP:DIP-40_W15.24mm_Socket, symbol VGMPlayer-rescue:STC8951-VGM
- removed U12, U2: 7805-VGM, Package_TO_SOT_THT:TO-220-3_Vertical, symbol VGMPlayer-rescue:7805-VGM
- removed U20: YM2612, Package_DIP:DIP-24_W15.24mm_Socket, symbol VGMPlayer-rescue:YM2612-VGM
- removed Y1: 11.0592MHz, Crystal:Crystal_HC49-4H_Vertical, symbol Device:Crystal
- added C1: 100uF, Capacitor_THT:CP_Radial_D8.0mm_P3.50mm, symbol Device:CP1
- added C3: 1000uF, Capacitor_THT:CP_Radial_D8.0mm_P3.50mm, symbol Device:CP1
- added D1, D2, D3, D4, D5, D6, D7, D8: LED, symbol Device:LED
- added J1: USB_B_Mini, Connector_USB:USB_Micro-B_Wuerth_629105150521_CircularHoles, symbol Connector:USB_B_Mini
- added J2: SD_Card, Connector_Card:SD_TE_2041021, symbol VGMPlayer-rescue:SD_Card
- added RV1, RV2: 10k, Varistor:RV_Disc_D7mm_W3.4mm_P5mm, symbol Device:R_POT_US
- added SW1: Play/Suffle, symbol Switch:SW_Push
- added SW2: Stop, symbol Switch:SW_Push
- added SW3: Next/Pause, symbol Switch:SW_Push
- added SW4: Prev/Resume, symbol Switch:SW_Push
- added U1: STM32F103XX, Package_DIP:DIP-40_W25.4mm_Socket, symbol VGMPlayer-rescue:STM32F103XX
- C2: value 10uF -> 100uF; footprint Capacitor_THT:CP_Radial_D4.0mm_P1.50mm -> Capacitor_THT:CP_Radial_D8.0mm_P3.50mm
- L1, L2: value L -> 30uH
- U14: footprint (none) -> Package_DIP:DIP-14_W7.62mm
Connections:
- net AGND_YM2151 is gone; now on net GNDA: C29.2, C30.1, C31.1, U13.16 (AGND), U13.8 (AGND)
- net GND_YM2151 is gone; now on net GND: U13.3 (DGND), U5.1 (GND), U5.11 (GND)
- net I2C_SCK is gone; now on net I2C_CLK: U18.3 (SCK)
- net I2C_SDA is gone; now on net I2C_DAT: U18.4 (SDA)
- net VDD_YM2151 is gone; now on net VDD: U5.22 (VDD)
- net YM2151_A0 is gone; now on net YM_A0: U5.4 (A0)
- net YM2151_CLK is gone; now on net YM_CLK: U5.24 (PhiM)
- net YM2151_CS is gone; now on net YM_CS: U5.7 (/CS)
- net YM2151_D0 is gone; now on net D0: U5.10 (D0)
- net YM2151_D1 is gone; now on net D1: U5.12 (D1)
- net YM2151_D2 is gone; now on net D2: U5.13 (D2)
- net YM2151_D3 is gone; now on net D3: U5.14 (D3)
- net YM2151_D4 is gone; now on net D4: U5.15 (D4)
- net YM2151_D5 is gone; now on net D5: U5.16 (D5)
- net YM2151_D6 is gone; now on net D6: U5.17 (D6)
- net YM2151_D7 is gone; now on net D7: U5.18 (D7)
- net YM2151_IC is gone; now on net YM_IC: U13.7 (/IC), U5.3 (/IC)
- net YM2151_MOL is gone; now on net YM_MOL: U14.8, U14.9 (-)
- net YM2151_MOR is gone; now on net YM_MOR: U14.13 (-), U14.14
- net YM2151_RD is gone; now on net VDD: U5.6 (/RD)
- net YM2151_WR is gone; now on net YM_WR: U5.5 (/WR)
- net +3V3: now also J2.4 (VDD), U1.40 (3.3V)
- net +5V: now also C2.1, C25.2, C26.2, C27.1, C28.1, U10.7 (OE), U10.8 (VCC), U13.1 (VDD), U14.4 (V+), U9.7 (OE), U9.8 (VCC), C3.1
- net D0: now also D1.1 (K), U1.5 (A0)
- net D1: now also D2.1 (K), U1.6 (A1)
- net D2: now also D3.1 (K), U1.7 (A2)
- net D3: now also D4.1 (K), U1.8 (A3)
- net D4: now also D5.1 (K), U1.9 (A4)
- net D5: now also D6.1 (K), U1.10 (A5)
- net D6: now also D7.1 (K), U1.11 (A6)
- net D7: now also D8.1 (K), U1.12 (A7)
- net GND: now also C1.2, J1.5 (GND), J1.6 (Shield), J2.3 (VSS), J2.6 (VSS), SW1.2, SW2.2, SW3.2, SW4.2, U1.19 (GND), U1.20 (GND), U1.39 (GND); no longer C24.2, C25.1, C26.1, C27.2, C28.2, U10.1 (GND), U8.6 (/OE), U8.8 (GND), U9.1 (GND)
- net GNDA: now also C2.2, C24.2, C25.1, C26.1, C27.2, C28.2, U10.1 (GND), U14.11 (V-), U8.6 (/OE), U8.8 (GND), U9.1 (GND), C3.2, RV1.3, RV2.3
- net I2C_CLK: now also U1.24 (B15)
- net I2C_DAT: now also U1.23 (B14)
- net RXD: now also U1.26 (A9)
- net SD_CS: now also J2.1 (CD/DAT3), U1.32 (B4)
- net SN_CLK_CS: now also U1.33 (B5)
- net SN_WR: now also U1.22 (B13)
- net SPI_CLK: now also U10.3 (SCK), U9.3 (SCK), J2.5 (CLK), U1.37 (B9); no longer U10.2 (SDI), U9.2 (SDI)
- net SPI_MISO: now also J2.7 (DAT0), U1.35 (B7)
- net SPI_MOSI: now also U10.2 (SDI), U9.2 (SDI), J2.2 (CMD), U1.36 (B8); no longer U10.3 (SCK), U9.3 (SCK)
- net TBD_CS: now also U1.31 (B3)
- net TXD: now also U1.25 (A8)
- net VDD: now also RN1.1 (common), C1.1, J1.1 (VBUS), U1.38 (5V); no longer C25.2, C26.2, C27.1, C28.1, U10.7 (OE), U10.8 (VCC), U9.7 (OE), U9.8 (VCC)
- net YM_A0: now also U1.15 (B10)
- net YM_A1: now also U1.16 (B11)
- net YM_CLK_CS: now also U1.34 (B6)
- net YM_CS: now also U1.13 (B0)
- net YM_IC: now also U1.21 (B12)
- net YM_WR: now also U1.14 (B1)
- net at R5.1, R8.1: now also RV2.1; no longer C8.1, R9.2
- net at R6.1, R7.1: now also RV1.1; no longer C9.1, R10.2
- net at U13.13 (MP), U14.1: no longer U13.14 (BC), U14.2 (-)
- removed net +5V_8051: C2.1, RN1.1 (common)
- net IRQ: no longer names the net of U7.13 (IRQ)
- net P0.0: no longer names the net of RN1.2 (R1)
- net P0.0: now also D1.2 (A)
- net P0.1: no longer names the net of RN1.3 (R2)
- net P0.1: now also D2.2 (A)
- net P0.2: no longer names the net of RN1.4 (R3)
- net P0.2: now also D3.2 (A)
- net P0.3: no longer names the net of RN1.5 (R4)
- net P0.3: now also D4.2 (A)
- net P0.4: no longer names the net of RN1.6 (R5)
- net P0.4: now also D5.2 (A)
- net P0.5: no longer names the net of RN1.7 (R6)
- net P0.5: now also D6.2 (A)
- net P0.6: no longer names the net of RN1.8 (R7)
- net P0.6: now also D7.2 (A)
- net P0.7: no longer names the net of RN1.9 (R8)
- net P0.7: now also D8.2 (A)
- net YM2151_IRQ: no longer names the net of U5.2 (/IRQ)
- new net: C8.1, R9.2, RV2.2
- new net: C9.1, R10.2, RV1.2
- new net: U13.14 (BC), U14.2 (-)
- new net Next_Pause: SW3.1, U1.28 (A11)
- new net Play: SW1.1, U1.30 (A15)
- new net Prev_Resume: SW4.1, U1.27 (A10)
- new net Stop: SW2.1, U1.29 (A12)
Other:
- moved on the sheet: C11, C12, C15, C18, C23, C24, C25, C26, C27, C28, C29, C30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
