File: Hardware/VGMPlayer/VGMPlayer.sch (KiCad schematic (older format))
At the start: 75 parts, among them J1 USB_B_Mini, J2 SD_Card, SW1 Play/Suffle, SW2 Stop, SW3 Next/Pause, SW4 Prev/Resume, U1 STM32F103XX, U10 LTC6903, U11 HC-06, U13 YM3012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

Commit message: 1
Parts:
- removed J2: SD_Card, Connector_Card:SD_TE_2041021, symbol VGMPlayer-rescue:SD_Card
- added U2: SDCardModule, Connector_PinHeader_2.54mm:PinHeader_1x08_P2.54mm_Vertical, symbol VGMPlayer-rescue:SDCardModule
- D1, D2, D3, D4, D5, D6, D7, D8: footprint (none) -> LED_SMD:LED_0805_2012Metric
- RV1, RV2: footprint Varistor:RV_Disc_D7mm_W3.4mm_P5mm -> Connector_PinHeader_2.54mm:PinHeader_1x03_P2.54mm_Vertical
- SW1, SW2, SW3, SW4: footprint (none) -> Button_Switch_THT:SW_Tactile_Straight_KSA0Axx1LFTR
- U1: footprint Package_DIP:DIP-40_W25.4mm_Socket -> Package_DIP:DIP-40_W15.24mm_Socket
Connections:
- net +3V3: now also U2.7 (3v3)
- net GND: now also U2.1 (GND), U2.8 (GND)
- net I2C_CLK: now also U1.34 (B6); no longer U1.24 (B15)
- net I2C_DAT: now also U1.35 (B7); no longer U1.23 (B14)
- net Next_Pause: now also U1.29 (A12); no longer U1.28 (A11)
- net Play: now also U1.25 (A8); no longer U1.30 (A15)
- net Prev_Resume: now also U1.28 (A11); no longer U1.27 (A10)
- net RXD: now also U1.27 (A10); no longer U1.26 (A9)
- net SD_CS: now also U1.33 (B5), U2.5 (CS); no longer U1.32 (B4)
- net SN_CLK_CS: now also U1.37 (B9); no longer U1.33 (B5)
- net SN_WR: now also U1.36 (B8); no longer U1.22 (B13)
- net SPI_CLK: now also U1.22 (B13), U2.3 (SCK); no longer U1.37 (B9)
- net SPI_MISO: now also U1.23 (B14), U2.2 (MISO); no longer U1.35 (B7)
- net SPI_MOSI: now also U1.24 (B15), U2.4 (MOSI); no longer U1.36 (B8)
- net Stop: now also U1.30 (A15); no longer U1.29 (A12)
- net TXD: now also U1.26 (A9); no longer U1.25 (A8)
- net YM_CLK_CS: now also U1.32 (B4); no longer U1.34 (B6)
- net TBD_CS: no longer names the net of U1.31 (B3)
Changed lines of the file:
@@
 Text GLabel 2300 2250 0    50   Input ~ 0
 YM_A1
-Text GLabel 4050 1250 2    50   Input ~ 0
+Text GLabel 4050 2450 2    50   Input ~ 0
 SPI_MISO
+Text GLabel 4050 2550 2    50   Input ~ 0
+SPI_CLK
+Text GLabel 4050 2350 2    50   Input ~ 0
+SPI_MOSI
+Text GLabel 4050 1550 2    50   Input ~ 0
+YM_CLK_CS
 Text GLabel 4050 1050 2    50   Input ~ 0
-SPI_CLK
-Text GLabel 4050 1150 2    50   Input ~ 0
-SPI_MOSI
-Text GLabel 4050 1350 2    50   Input ~ 0
-YM_CLK_CS
-Text GLabel 4050 1450 2    50   Input ~ 0
 SN_CLK_CS
 $Comp
@@
 Wire Wire Line
 	7100 4100 7100 4200
-Text GLabel 4050 1550 2    50   Input ~ 0
+Text GLabel 4050 1450 2    50   Input ~ 0
 SD_CS
-Text GLabel 4050 1650 2    50   Input ~ 0
-TBD_CS
-Text GLabel 4050 2550 2    50   Input ~ 0
+Text GLabel 4050 1150 2    50   Input ~ 0
 SN_WR
 Wire Wire Line
@@
 F 0 "U1" H 2700 700 50  0000 C CNN
 F 1 "STM32F103XX" H 3050 700 50  0000 C CNN
-F 2 "Package_DIP:DIP-40_W25.4mm_Socket" H 3100 700 50  0001 C CNN
+F 2 "Package_DIP:DIP-40_W15.24mm_Socket" H 3100 700 50  0001 C CNN
 F 3 "" H 3100 700 50  0001 C CNN
 	1    3100 650
@@
 Wire Wire Line
 	4100 950  3850 950
-Text GLabel 4050 2350 2    50   Input ~ 0
+Text GLabel 4050 1350 2    50   Input ~ 0
 I2C_CLK
-Text GLabel 4050 2450 2    50   Output ~ 0
+Text GLabel 4050 1250 2    50   Output ~ 0
 I2C_DAT
-Text GLabel 4050 2150 2    50   Input ~ 0
+Text GLabel 4050 2050 2    50   Input ~ 0
 RXD
-Text GLabel 4050 2250 2    50   Output ~ 0
+Text GLabel 4050 2150 2    50   Output ~ 0
 TXD
 $Comp
@@
 F 0 "RV1" H 9982 6546 50  0000 R CNN
 F 1 "10k" H 9982 6455 50  0000 R CNN
-F 2 "Varistor:RV_Disc_D7mm_W3.4mm_P5mm" H 10050 6500 50  0001 C CNN
+F 2 "Connector_PinHeader_2.54mm:PinHeader_1x03_P2.54mm_Vertical" H 10050 6500 50  0001 C CNN
 F 3 "~" H 10050 6500 50  0001 C CNN
 	1    10050 6500
@@
 F 0 "RV2" H 9982 5046 50  0000 R CNN
 F 1 "10k" H 9982 4955 50  0000 R CNN
-F 2 "Varistor:RV_Disc_D7mm_W3.4mm_P5mm" H 10050 5000 50  0001 C CNN
+F 2 "Connector_PinHeader_2.54mm:PinHeader_1x03_P2.54mm_Vertical" H 10050 5000 50  0001 C CNN
 F 3 "~" H 10050 5000 50  0001 C CNN
 	1    10050 5000
@@
 Wire Wire Line
 	10050 5150 10050 5200
-$Comp
-L VGMPlayer-rescue:SD_Card J2
-U 1 1 5F3D5C10
-P 13150 1300
-F 0 "J2" H 13750 750 50  0000 L CNN
-F 1 "SD_Card" H 13350 750 50  0000 L CNN
-F 2 "Connector_Card:SD_TE_2041021" H 13150 1300 50  0001 C CNN
-F 3 "http://portal.fciconnect.com/Comergent//fci/drawing/10067847.pdf" H 13150 1300 50  0001 C CNN
-	1    13150 1300
-	-1   0    0    1
-$EndComp
 Wire Notes Line
 	15200 550  18600 550
@@
 Wire Notes Line
 	18600 2900 15200 2900
-Text GLabel 14500 1000 2    50   Input ~ 0
+Text GLabel 14350 1600 2    50   Input ~ 0
 SPI_MISO
-Text GLabel 14500 1500 2    50   Input ~ 0
+Text GLabel 14350 1400 2    50   Input ~ 0
 SPI_MOSI
-Text GLabel 14500 1200 2    50   Input ~ 0
+Text GLabel 14350 1500 2    50   Input ~ 0
 SPI_CLK
-Text GLabel 14500 1600 2    50   Input ~ 0
+Text GLabel 14350 1300 2    50   Input ~ 0
 SD_CS
 $Comp
 L power:GND #PWR027
 U 1 1 5F546118
-P 14150 1800
-F 0 "#PWR027" H 14150 1550 50  0001 C CNN
-F 1 "GND" H 14000 1750 50  0000 C CNN
-F 2 "" H 14150 1800 50  0001 C CNN
-F 3 "" H 14150 1800 50  0001 C CNN
-	1    14150 1800
+P 14000 1800
+F 0 "#PWR027" H 14000 1550 50  0001 C CNN
+F 1 "GND" H 14100 1800 50  0000 C CNN
+F 2 "" H 14000 1800 50  0001 C CNN
+F 3 "" H 14000 1800 50  0001 C CNN
+	1    14000 1800
 	1    0    0    -1
 $EndComp
@@
 L power:+3.3V #PWR028
 U 1 1 5F56EE7E
-P 14250 750
-F 0 "#PWR028" H 14250 600 50  0001 C CNN
-F 1 "+3.3V" H 14100 850 50  0000 C CNN
-F 2 "" H 14250 750 50  0001 C CNN
-F 3 "" H 14250 750 50  0001 C CNN
-	1    14250 750
-	1    0    0    -1
-$EndComp
-Wire Wire Line
-	14050 1400 14150 1400
-Wire Wire Line
-	14150 1400 14150 1100
-Wire Wire Line
-	14500 1200 14050 1200
-Wire Wire Line
-	14500 1600 14050 1600
-Wire Wire Line
-	14050 1500 14500 1500
-Wire Wire Line
-	14050 1000 14500 1000
-Wire Wire Line
-	14050 1300 14250 1300
-Connection ~ 14150 1400
-Wire Wire Line
-	14150 1100 14050 1100
-Wire Wire Line
-	14250 750  14250 1300
-Wire Wire Line
-	14150 1800 14150 1400
+P 14100 750
+F 0 "#PWR028" H 14100 600 50  0001 C CNN
+F 1 "+3.3V" H 13950 850 50  0000 C CNN
+F 2 "" H 14100 750 50  0001 C CNN
+F 3 "" H 14100 750 50  0001 C CNN
+	1    14100 750
+	1    0    0    -1
+$EndComp
+Wire Wire Line
+	13900 1700 14000 1700
+Wire Wire Line
+	14350 1500 13900 1500
+Wire Wire Line
+	14350 1300 13900 1300
+Wire Wire Line
+	13900 1400 14350 1400
+Wire Wire Line
+	13900 1600 14350 1600
+Wire Wire Line
+	13900 1100 14100 1100
+Wire Wire Line
+	14000 1000 13900 1000
+Wire Wire Line
+	14100 750  14100 1100
+Wire Wire Line
+	14000 1800 14000 1700
 Wire Wire Line
 	11650 6250 11900 6250
@@
 F 0 "SW1" H 18050 1685 50  0000 C CNN
 F 1 "Play/Suffle" H 18050 1594 50  0000 C CNN
-F 2 "" H 18050 1600 50  0001 C CNN
+F 2 "Button_Switch_THT:SW_Tactile_Straight_KSA0Axx1LFTR" H 18050 1600 50  0001 C CNN
 F 3 "" H 18050 1600 50  0001 C CNN
 	1    18050 1400
@@
 F 0 "SW2" H 18050 2085 50  0000 C CNN
 F 1 "Stop" H 18050 1994 50  0000 C CNN
-F 2 "" H 18050 2000 50  0001 C CNN
+F 2 "Button_Switch_THT:SW_Tactile_Straight_KSA0Axx1LFTR" H 18050 2000 50  0001 C CNN
 F 3 "" H 18050 2000 50  0001 C CNN
 	1    18050 1800
@@
 F 0 "SW3" H 18050 2485 50  0000 C CNN
 F 1 "Next/Pause" H 18050 2394 50  0000 C CNN
-F 2 "" H 18050 2400 50  0001 C CNN
+F 2 "Button_Switch_THT:SW_Tactile_Straight_KSA0Axx1LFTR" H 18050 2400 50  0001 C CNN
 F 3 "" H 18050 2400 50  0001 C CNN
 	1    18050 2200
@@
 F 0 "SW4" H 18050 2885 50  0000 C CNN
 F 1 "Prev/Resume" H 18050 2794 50  0000 C CNN
-F 2 "" H 18050 2800 50  0001 C CNN
+F 2 "Button_Switch_THT:SW_Tactile_Straight_KSA0Axx1LFTR" H 18050 2800 50  0001 C CNN
 F 3 "" H 18050 2800 50  0001 C CNN
 	1    18050 2600
@@
 Wire Wire Line
 	17850 2600 17750 2600
+Text GLabel 4050 2250 2    50   Input ~ 0
+Play
 Text GLabel 4050 1750 2    50   Input ~ 0
-Play
+Stop
 Text GLabel 4050 1850 2    50   Input ~ 0
-Stop
+Next_Pause
 Text GLabel 4050 1950 2    50   Input ~ 0
-Next_Pause
-Text GLabel 4050 2050 2    50   Input ~ 0
 Prev_Resume
 Wire Wire Line
@@
 F 0 "D1" H 15900 2000 50  0000 C CNN
 F 1 "LED" H 15950 2100 50  0001 C CNN
-F 2 "" H 15800 2050 50  0001 C CNN
+F 2 "LED_SMD:LED_0805_2012Metric" H 15800 2050 50  0001 C CNN
 F 3 "~" H 15800 2050 50  0001 C CNN
 	1    15800 2050
@@
 F 0 "D2" H 15900 2100 50  0000 C CNN
 F 1 "LED" H 15950 2200 50  0001 C CNN
-F 2 "" H 15800 2150 50  0001 C CNN
+F 2 "LED_SMD:LED_0805_2012Metric" H 15800 2150 50  0001 C CNN
 F 3 "~" H 15800 2150 50  0001 C CNN
 	1    15800 2150
@@
 F 0 "D3" H 15900 2200 50  0000 C CNN
 F 1 "LED" H 15950 2300 50  0001 C CNN
-F 2 "" H 15800 2250 50  0001 C CNN
+F 2 "LED_SMD:LED_0805_2012Metric" H 15800 2250 50  0001 C CNN
 F 3 "~" H 15800 2250 50  0001 C CNN
 	1    15800 2250
@@
 F 0 "D4" H 15900 2300 50  0000 C CNN
 F 1 "LED" H 15950 2400 50  0001 C CNN
-F 2 "" H 15800 2350 50  0001 C CNN
+F 2 "LED_SMD:LED_0805_2012Metric" H 15800 2350 50  0001 C CNN
 F 3 "~" H 15800 2350 50  0001 C CNN
 	1    15800 2350
@@
 F 0 "D5" H 15900 2400 50  0000 C CNN
 F 1 "LED" H 15950 2500 50  0001 C CNN
-F 2 "" H 15800 2450 50  0001 C CNN
+F 2 "LED_SMD:LED_0805_2012Metric" H 15800 2450 50  0001 C CNN
 F 3 "~" H 15800 2450 50  0001 C CNN
 	1    15800 2450
@@
 F 0 "D6" H 15900 2500 50  0000 C CNN
 F 1 "LED" H 15950 2600 50  0001 C CNN
-F 2 "" H 15800 2550 50  0001 C CNN
+F 2 "LED_SMD:LED_0805_2012Metric" H 15800 2550 50  0001 C CNN
 F 3 "~" H 15800 2550 50  0001 C CNN
 	1    15800 2550
@@
 F 0 "D7" H 15900 2600 50  0000 C CNN
 F 1 "LED" H 15950 2700 50  0001 C CNN
-F 2 "" H 15800 2650 50  0001 C CNN
+F 2 "LED_SMD:LED_0805_2012Metric" H 15800 2650 50  0001 C CNN
 F 3 "~" H 15800 2650 50  0001 C CNN
 	1    15800 2650
@@
 F 0 "D8" H 15900 2700 50  0000 C CNN
 F 1 "LED" H 15950 2800 50  0001 C CNN
-F 2 "" H 15800 2750 50  0001 C CNN
+F 2 "LED_SMD:LED_0805_2012Metric" H 15800 2750 50  0001 C CNN
 F 3 "~" H 15800 2750 50  0001 C CNN
 	1    15800 2750
@@
 Wire Wire Line
 	16750 2050 15950 2050
+$Comp
+L VGMPlayer-rescue:SDCardModule U2
+U 1 1 5C3D4BB0
+P 12800 1300
+F 0 "U2" H 13056 1915 50  0000 C CNN
+F 1 "SDCardModule" H 13056 1824 50  0000 C CNN
+F 2 "Connector_PinHeader_2.54mm:PinHeader_1x08_P2.54mm_Vertical" H 13050 700 50  0001 C CNN
+F 3 "" H 13050 700 50  0001 C CNN
+	1    12800 1300
+	1    0    0    -1
+$EndComp
+Connection ~ 14000 1700
+Wire Wire Line
+	14000 1000 14000 1700
 $EndSCHEMATC

Commit message: 1
Connections:
- net TBD0: now reaches U1.31 (B3)
- net Next_Pause renamed NEXT_PAUSE
- net Play renamed PLAY
- net Prev_Resume renamed PREV_RESUME
- net Stop renamed STOP
Changed lines of the file:
@@
 Connection ~ 18400 1800
 Text GLabel 17750 1400 0    50   Input ~ 0
-Play
+PLAY
 Text GLabel 17750 1800 0    50   Input ~ 0
-Stop
+STOP
 Text GLabel 17750 2200 0    50   Input ~ 0
-Next_Pause
+NEXT_PAUSE
 Text GLabel 17750 2600 0    50   Input ~ 0
-Prev_Resume
+PREV_RESUME
 Wire Wire Line
 	17850 1400 17750 1400
@@
 	17850 2600 17750 2600
 Text GLabel 4050 2250 2    50   Input ~ 0
-Play
+PLAY
 Text GLabel 4050 1750 2    50   Input ~ 0
-Stop
+STOP
 Text GLabel 4050 1850 2    50   Input ~ 0
-Next_Pause
+NEXT_PAUSE
 Text GLabel 4050 1950 2    50   Input ~ 0
-Prev_Resume
+PREV_RESUME
 Wire Wire Line
 	3850 2450 4050 2450
@@
 Wire Wire Line
 	14000 1000 14000 1700
+Text GLabel 4050 1650 2    50   Input ~ 0
+TBD0
 $EndSCHEMATC

Commit message: 1
Parts:
- removed RN1: R_Network08, Resistor_THT:R_Array_SIP9, symbol Device:R_Network08
- added R1, R16, R17: 0, Resistor_SMD:R_0805_2012Metric, symbol Device:R
- added R18, R19, R20, R21, R22, R23, R24, R25: 330, Resistor_SMD:R_0805_2012Metric, symbol Device:R
- SW1: value Play/Suffle -> Mode
- SW2: value Stop -> NEXT
- SW3: value Next/Pause -> PREV
- SW4: value Prev/Resume -> SELECT
Connections:
- net VDD: now also R18.2, R19.2, R20.2, R21.2, R22.2, R23.2, R24.2, R25.2
- net at U5.2 (/IRQ): now also R1.1
- net at U5.8 (CT1): now also R16.1
- net at U5.9 (CT2): now also R17.1
- net at D1.2 (A): now also R25.1
- net at D2.2 (A): now also R24.1
- net at D3.2 (A): now also R23.1
- net at D4.2 (A): now also R22.1
- net at D5.2 (A): now also R21.1
- net at D6.2 (A): now also R20.1
- net at D7.2 (A): now also R19.1
- net at D8.2 (A): now also R18.1
- net NEXT_PAUSE renamed NEXT
- net NEXT: now also SW2.1; no longer SW3.1
- net PLAY renamed MODE
- net MODE: now also U1.30 (A15); no longer U1.25 (A8)
- net PREV_RESUME renamed PREV
- net PREV: now also SW3.1; no longer SW4.1
- removed net STOP: SW2.1, U1.30 (A15)
- new net SELECT: SW4.1, U1.25 (A8)
Changed lines of the file:
@@
 Wire Wire Line
 	7000 800  7450 800
-Text GLabel 10400 2200 2    50   Input ~ 0
+Text GLabel 10400 2200 2    50   Output ~ 0
 SN_CLK
 Wire Wire Line
 	10400 2200 10250 2200
-Text GLabel 7150 2450 2    50   Input ~ 0
+Text GLabel 7150 2450 2    50   Output ~ 0
 YM_CLK
 Wire Wire Line
@@
 P 18050 1400
 F 0 "SW1" H 18050 1685 50  0000 C CNN
-F 1 "Play/Suffle" H 18050 1594 50  0000 C CNN
+F 1 "Mode" H 18050 1594 50  0000 C CNN
 F 2 "Button_Switch_THT:SW_Tactile_Straight_KSA0Axx1LFTR" H 18050 1600 50  0001 C CNN
 F 3 "" H 18050 1600 50  0001 C CNN
@@
 P 18050 1800
 F 0 "SW2" H 18050 2085 50  0000 C CNN
-F 1 "Stop" H 18050 1994 50  0000 C CNN
+F 1 "NEXT" H 18050 1994 50  0000 C CNN
 F 2 "Button_Switch_THT:SW_Tactile_Straight_KSA0Axx1LFTR" H 18050 2000 50  0001 C CNN
 F 3 "" H 18050 2000 50  0001 C CNN
@@
 P 18050 2200
 F 0 "SW3" H 18050 2485 50  0000 C CNN
-F 1 "Next/Pause" H 18050 2394 50  0000 C CNN
+F 1 "PREV" H 18050 2394 50  0000 C CNN
 F 2 "Button_Switch_THT:SW_Tactile_Straight_KSA0Axx1LFTR" H 18050 2400 50  0001 C CNN
 F 3 "" H 18050 2400 50  0001 C CNN
@@
 P 18050 2600
 F 0 "SW4" H 18050 2885 50  0000 C CNN
-F 1 "Prev/Resume" H 18050 2794 50  0000 C CNN
+F 1 "SELECT" H 18050 2794 50  0000 C CNN
 F 2 "Button_Switch_THT:SW_Tactile_Straight_KSA0Axx1LFTR" H 18050 2800 50  0001 C CNN
 F 3 "" H 18050 2800 50  0001 C CNN
@@
 Connection ~ 18400 1800
 Text GLabel 17750 1400 0    50   Input ~ 0
-PLAY
+MODE
 Text GLabel 17750 1800 0    50   Input ~ 0
-STOP
+NEXT
 Text GLabel 17750 2200 0    50   Input ~ 0
-NEXT_PAUSE
+PREV
 Text GLabel 17750 2600 0    50   Input ~ 0
-PREV_RESUME
+SELECT
 Wire Wire Line
 	17850 1400 17750 1400
@@
 	17850 2600 17750 2600
 Text GLabel 4050 2250 2    50   Input ~ 0
-PLAY
+SELECT
 Text GLabel 4050 1750 2    50   Input ~ 0
-STOP
+MODE
 Text GLabel 4050 1850 2    50   Input ~ 0
-NEXT_PAUSE
+NEXT
 Text GLabel 4050 1950 2    50   Input ~ 0
-PREV_RESUME
+PREV
 Wire Wire Line
 	3850 2450 4050 2450
@@
 	15650 2750 15550 2750
 $Comp
-L Device:R_Network08 RN1
-U 1 1 625295AF
-P 16350 1750
-F 0 "RN1" H 16730 1796 50  0000 L CNN
-F 1 "R_Network08" H 16200 1950 50  0000 L CNN
-F 2 "Resistor_THT:R_Array_SIP9" V 16825 1750 50  0001 C CNN
-F 3 "http://www.vishay.com/docs/31509/csc.pdf" H 16350 1750 50  0001 C CNN
-	1    16350 1750
-	-1   0    0    -1
-$EndComp
-$Comp
 L power:VDD #PWR029
 U 1 1 6269EDA4
-P 16750 1500
-F 0 "#PWR029" H 16750 1350 50  0001 C CNN
-F 1 "VDD" H 16850 1550 50  0000 C CNN
-F 2 "" H 16750 1500 50  0001 C CNN
-F 3 "" H 16750 1500 50  0001 C CNN
-	1    16750 1500
-	1    0    0    -1
-$EndComp
-Wire Wire Line
-	16750 1500 16750 1550
+P 16750 1400
+F 0 "#PWR029" H 16750 1250 50  0001 C CNN
+F 1 "VDD" H 16850 1450 50  0000 C CNN
+F 2 "" H 16750 1400 50  0001 C CNN
+F 3 "" H 16750 1400 50  0001 C CNN
+	1    16750 1400
+	1    0    0    -1
+$EndComp
 Wire Wire Line
 	16050 1950 16050 2750
@@
 Text GLabel 4050 1650 2    50   Input ~ 0
 TBD0
+$Comp
+L Device:R R17
+U 1 1 5C3D6397
+P 1050 4600
+F 0 "R17" V 1000 4450 50  0000 C CNN
+F 1 "0" V 1000 4750 50  0000 C CNN
+F 2 "Resistor_SMD:R_0805_2012Metric" V 980 4600 50  0001 C CNN
+F 3 "~" H 1050 4600 50  0001 C CNN
+	1    1050 4600
+	0    1    1    0
+$EndComp
+Wire Wire Line
+	1200 4600 1400 4600
+$Comp
+L Device:R R1
+U 1 1 5C46AD72
+P 1050 3900
+F 0 "R1" V 1000 3750 50  0000 C CNN
+F 1 "0" V 1000 4050 50  0000 C CNN
+F 2 "Resistor_SMD:R_0805_2012Metric" V 980 3900 50  0001 C CNN
+F 3 "~" H 1050 3900 50  0001 C CNN
+	1    1050 3900
+	0    1    1    0
+$EndComp
+Wire Wire Line
+	1200 3900 1400 3900
+$Comp
+L Device:R R16
+U 1 1 5C49CC6D
+P 1050 4500
+F 0 "R16" V 1000 4350 50  0000 C CNN
+F 1 "0" V 1000 4650 50  0000 C CNN
+F 2 "Resistor_SMD:R_0805_2012Metric" V 980 4500 50  0001 C CNN
+F 3 "~" H 1050 4500 50  0001 C CNN
+	1    1050 4500
+	0    1    1    0
+$EndComp
+Wire Wire Line
+	1200 4500 1400 4500
+$Comp
+L Device:R R18
+U 1 1 5C4D12AC
+P 16050 1800
+F 0 "R18" V 16100 1950 50  0000 C CNN
+F 1 "330" V 16100 1600 50  0000 C CNN
+F 2 "Resistor_SMD:R_0805_2012Metric" V 15980 1800 50  0001 C CNN
+F 3 "~" H 16050 1800 50  0001 C CNN
+	1    16050 1800
+	-1   0    0    1
+$EndComp
+$Comp
+L Device:R R19
+U 1 1 5C568BBF
+P 16150 1800
+F 0 "R19" V 16200 1950 50  0000 C CNN
+F 1 "330" V 16200 1600 50  0000 C CNN
+F 2 "Resistor_SMD:R_0805_2012Metric" V 16080 1800 50  0001 C CNN
+F 3 "~" H 16150 1800 50  0001 C CNN
+	1    16150 1800
+	-1   0    0    1
+$EndComp
+$Comp
+L Device:R R20
+U 1 1 5C59B12E
+P 16250 1800
+F 0 "R20" V 16300 1950 50  0000 C CNN
+F 1 "330" V 16300 1600 50  0000 C CNN
+F 2 "Resistor_SMD:R_0805_2012Metric" V 16180 1800 50  0001 C CNN
+F 3 "~" H 16250 1800 50  0001 C CNN
+	1    16250 1800
+	-1   0    0    1
+$EndComp
+$Comp
+L Device:R R21
+U 1 1 5C59B135
+P 16350 1800
+F 0 "R21" V 16400 1950 50  0000 C CNN
+F 1 "330" V 16400 1600 50  0000 C CNN
+F 2 "Resistor_SMD:R_0805_2012Metric" V 16280 1800 50  0001 C CNN
+F 3 "~" H 16350 1800 50  0001 C CNN
+	1    16350 1800
+	-1   0    0    1
+$EndComp
+$Comp
+L Device:R R22
+U 1 1 5C5CD6DE
+P 16450 1800
+F 0 "R22" V 16500 1950 50  0000 C CNN
+F 1 "330" V 16500 1600 50  0000 C CNN
+F 2 "Resistor_SMD:R_0805_2012Metric" V 16380 1800 50  0001 C CNN
+F 3 "~" H 16450 1800 50  0001 C CNN
+	1    16450 1800
+	-1   0    0    1
+$EndComp
+$Comp
+L Device:R R23
+U 1 1 5C5CD6E5
+P 16550 1800
+F 0 "R23" V 16600 1950 50  0000 C CNN
+F 1 "330" V 16600 1600 50  0000 C CNN
+F 2 "Resistor_SMD:R_0805_2012Metric" V 16480 1800 50  0001 C CNN
+F 3 "~" H 16550 1800 50  0001 C CNN
+	1    16550 1800
+	-1   0    0    1
+$EndComp
+$Comp
+L Device:R R24
+U 1 1 5C5CD6EC
+P 16650 1800
+F 0 "R24" V 16700 1950 50  0000 C CNN
+F 1 "330" V 16700 1600 50  0000 C CNN
+F 2 "Resistor_SMD:R_0805_2012Metric" V 16580 1800 50  0001 C CNN
+F 3 "~" H 16650 1800 50  0001 C CNN
+	1    16650 1800
+	-1   0    0    1
+$EndComp
+$Comp
+L Device:R R25
+U 1 1 5C5CD6F3
+P 16750 1800
+F 0 "R25" V 16800 1950 50  0000 C CNN
+F 1 "330" V 16800 1600 50  0000 C CNN
+F 2 "Resistor_SMD:R_0805_2012Metric" V 16680 1800 50  0001 C CNN
+F 3 "~" H 16750 1800 50  0001 C CNN
+	1    16750 1800
+	-1   0    0    1
+$EndComp
+Wire Wire Line
+	16050 1650 16050 1500
+Wire Wire Line
+	16050 1500 16150 1500
+Wire Wire Line
+	16150 1500 16150 1650
+Wire Wire Line
+	16150 1500 16250 1500
+Wire Wire Line
+	16650 1500 16650 1650
+Connection ~ 16150 1500
+Wire Wire Line
+	16750 1400 16750 1500
+Wire Wire Line
+	16750 1500 16650 1500
+Connection ~ 16750 1500
+Wire Wire Line
+	16750 1500 16750 1650
+Connection ~ 16650 1500
+Wire Wire Line
+	16550 1500 16550 1650
+Connection ~ 16550 1500
+Wire Wire Line
+	16550 1500 16650 1500
+Wire Wire Line
+	16450 1500 16450 1650
+Connection ~ 16450 1500
+Wire Wire Line
+	16450 1500 16550 1500
+Wire Wire Line
+	16350 1500 16350 1650
+Connection ~ 16350 1500
+Wire Wire Line
+	16350 1500 16450 1500
+Wire Wire Line
+	16250 1500 16250 1650
+Connection ~ 16250 1500
+Wire Wire Line
+	16250 1500 16350 1500
 $EndSCHEMATC

Commit message: 1
Parts:
- added Q2, Q?: S8550, TO-92, symbol Transistor_BJT:S8550
- added Q?: 9013, symbol Device:Q_NPN_BEC
- added R26, R?: 47k, Resistor_SMD:R_0805_2012Metric, symbol Device:R
- added R27: 330, Resistor_SMD:R_0805_2012Metric, symbol Device:R
- added SW5: PWR, Button_Switch_THT:SW_Tactile_Straight_KSA0Axx1LFTR, symbol Switch:SW_Push
Connections:
- net GND: now also Q?.2 (E), Q?.3 (C), SW5.1
- net VDD: now also Q2.3 (C); no longer J1.1 (VBUS)
- net MODE renamed BUTTON_MODE
- net NEXT renamed BUTTON_NEXT
- net PREV renamed BUTTON_PREV
- net SELECT renamed BUTTON_SELECT
- net TBD0 renamed PWR_HOLD
- net PWR_HOLD: now also R?.2
- new net: Q?.1 (B), R?.1
- new net: J1.1 (VBUS), Q2.1 (E), R26.2
- new net: Q2.2 (B), R27.2
- new net: Q?.2 (B), Q?.3 (C), R26.1
- new net: Q?.1 (E), R27.1, SW5.2
Other:
- moved on the sheet: C23, C24, C25, C26, C27, C28, D1, D2, D3, D4, D5, D6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
