File: Hardware/VGMPlayer/VGMPlayer.sch (KiCad schematic (older format))
At the start: 102 parts, among them J1 USB_B_Mini, Q2 S8550, SW1 Mode, SW2 NEXT, SW3 PREV, SW4 SELECT, SW5 PWR, U1 STM32F103XX, U10 LTC6903, U11 HC-06, U13 YM3012, U14 LM324, U18 OLED_128_64_I2C, U19 ESP8266Module, U2 SDCardModule, U3 LM386, U4 LM386, U5 YM2151, U6 AUDIOJACK-VGM, U7 YM2612, U8 SN76489, U9 LTC6903

Commit message: 1
Parts:
- removed C? (x2): 0.47uF, Capacitor_SMD:C_0805_2012Metric, symbol Device:C
- removed C? (x2): 1uF, Capacitor_THT:CP_Radial_D8.0mm_P3.50mm, symbol Device:CP1
- removed C?: 470uF, Capacitor_THT:CP_Radial_D8.0mm_P3.50mm, symbol Device:CP1
- removed C?: 0.1uF, Capacitor_SMD:C_0805_2012Metric, symbol Device:C
- removed R? (x2): 10k, Resistor_SMD:R_0805_2012Metric, symbol Device:R
- removed U?: PAM8403, symbol VGMPlayer-rescue:PAM8403
- removed U?: R_POT_SW, symbol VGMPlayer-rescue:R_POT_SW
- removed U?: AUDIOJACK-VGM, Connector_Audio:Jack_Horizontal, symbol VGMPlayer-rescue:AUDIOJACK-VGM
- Q1: renamed from Q?; footprint (none) -> Package_TO_SOT_THT:TO-92
- Q2: footprint TO-92 -> Package_TO_SOT_THT:TO-92
- SW1, SW2, SW3, SW4, SW5: footprint Button_Switch_THT:SW_Tactile_Straight_KSA0Axx1LFTR -> Resistor_SMD:R_0805_2012Metric
- gave numbers to parts that had none: 1
- renumbered D1 to D0, D2 to D1, D3 to D2, D4 to D3, D5 to D4, D6 to D5, D7 to D6, D8 to D7

Commit message: 1
Parts:
- added J2: SD_Card, Connector_Card:SD_TE_2041021, symbol VGMPlayer-rescue:SD_Card
Changed lines of the file:
@@
 	0    1    1    0
 $EndComp
+$Comp
+L VGMPlayer-rescue:SD_Card J2
+U 1 1 5C3FE198
+P 16400 -150
+F 0 "J2" H 16400 -815 50  0000 C CNN
+F 1 "SD_Card" H 16400 -724 50  0000 C CNN
+F 2 "Connector_Card:SD_TE_2041021" H 16400 -150 50  0001 C CNN
+F 3 "http://portal.fciconnect.com/Comergent//fci/drawing/10067847.pdf" H 16400 -150 50  0001 C CNN
+	1    16400 -150
+	-1   0    0    1
+$EndComp
+Text GLabel 17650 -450 2    50   Input ~ 0
+SPI_MISO
+Text GLabel 17600 50   2    50   Input ~ 0
+SPI_MOSI
+Text GLabel 17650 -250 2    50   Input ~ 0
+SPI_CLK
+Text GLabel 17600 150  2    50   Input ~ 0
+SD_CS
+Wire Wire Line
+	17600 150  17300 150
+Wire Wire Line
+	17600 50   17300 50
+Wire Wire Line
+	17650 -450 17300 -450
+Wire Wire Line
+	17650 -250 17300 -250
+Wire Wire Line
+	17300 -350 17400 -350
+Wire Wire Line
+	17400 -350 17400 -50
+Wire Wire Line
+	17400 -50  17300 -50
+$Comp
+L power:GND #PWR0101
+U 1 1 5C6ABA25
+P 17400 300
+F 0 "#PWR0101" H 17400 50  50  0001 C CNN
+F 1 "GND" H 17500 300 50  0000 C CNN
+F 2 "" H 17400 300 50  0001 C CNN
+F 3 "" H 17400 300 50  0001 C CNN
+	1    17400 300
+	1    0    0    -1
+$EndComp
+Wire Wire Line
+	17400 -50  17400 300
+Connection ~ 17400 -50
+$Comp
+L power:+3.3V #PWR0102
+U 1 1 5C71FFAB
+P 17500 -700
+F 0 "#PWR0102" H 17500 -850 50  0001 C CNN
+F 1 "+3.3V" H 17350 -600 50  0000 C CNN
+F 2 "" H 17500 -700 50  0001 C CNN
+F 3 "" H 17500 -700 50  0001 C CNN
+	1    17500 -700
+	1    0    0    -1
+$EndComp
+Wire Wire Line
+	17500 -150 17300 -150
+Wire Wire Line
+	17500 -700 17500 -150
 $EndSCHEMATC

Commit message: 1
Parts:
- added C10, C13: 0.47uF, Capacitor_SMD:C_0805_2012Metric, symbol Device:C
- added C16, C32, C34: 1uF, Capacitor_SMD:C_0805_2012Metric, symbol Device:C
- added C33: 470uF, Capacitor_THT:CP_Radial_D8.0mm_P3.50mm, symbol Device:CP1
- added R29, R30: 1k, Resistor_SMD:R_0805_2012Metric, symbol Device:R
- added U12: PAM8403, symbol VGMPlayer-rescue:PAM8403
- added U15: AUDIOJACK-VGM, Connector_Audio:Jack_Horizontal, symbol VGMPlayer-rescue:AUDIOJACK-VGM
Connections:
- net +5V: now also C16.2, C32.2, C33.1, C34.2, U12.12 (~SHDN), U12.13 (PVDD), U12.4 (PVDD), U12.5 (~MUTE), U12.6 (AVDD)
- net GNDA: now also C16.1, C32.1, C33.2, C34.1, U12.11 (GND), U12.14 (-OUT_R), U12.15 (PGND), U12.2 (PGND), U12.3 (-OUT_L), U15.3 (S)
- new net: U12.1 (+OUT_L), U15.1 (T)
- new net: R30.2, U12.10 (IN_R)
- new net: U12.16 (+OUT_R), U15.2 (R)
- new net: R29.2, U12.7 (IN_L)
- new net: C10.1, R29.1
- new net: C13.1, R30.1

Commit message: 1
Parts:
- removed C10, C13: 0.47uF, Capacitor_SMD:C_0805_2012Metric, symbol Device:C
- removed C16, C32, C34: 1uF, Capacitor_SMD:C_0805_2012Metric, symbol Device:C
- removed C33: 470uF, Capacitor_THT:CP_Radial_D8.0mm_P3.50mm, symbol Device:CP1
- removed R29, R30: 1k, Resistor_SMD:R_0805_2012Metric, symbol Device:R
- removed RV1, RV2: 10k, Connector_PinHeader_2.54mm:PinHeader_1x03_P2.54mm_Vertical, symbol Device:R_POT_US
- removed U12: PAM8403, symbol VGMPlayer-rescue:PAM8403
- removed U15: AUDIOJACK-VGM, Connector_Audio:Jack_Horizontal, symbol VGMPlayer-rescue:AUDIOJACK-VGM
- removed U18: OLED_128_64_I2C, Connector_PinSocket_2.54mm:PinSocket_1x04_P2.54mm_Vertical, symbol VGMPlayer-rescue:OLED_128_64_I2C-VGM
- added J3: LCD_PORT, Connector_PinSocket_2.54mm:PinSocket_2x15_P2.54mm_Vertical, symbol Connector_Generic:Conn_02x15_Odd_Even
- added U?: R_POT_SW, Connector_Audio:VGM_VR_SW, symbol VGMPlayer-rescue:R_POT_SW
- SW1, SW2, SW3, SW4, SW5: footprint Resistor_SMD:R_0805_2012Metric -> Button_Switch_SMD:VGM_Button
- U6: footprint Connector_Audio:Jack_Horizontal -> Connector_Audio:VGMAudio_Jack
Connections:
- net +3V3: now also J2.5 (CLK), J3.2 (Pin_2)
- net +5V: now also L2.2, Q2.3 (C), U?.7; no longer L2.1
- net D0: now also J3.26 (Pin_26)
- net D1: now also J3.23 (Pin_23)
- net D2: now also J3.24 (Pin_24)
- net D3: now also J3.21 (Pin_21)
- net D4: now also J3.22 (Pin_22)
- net D5: now also J3.19 (Pin_19)
- net D6: now also J3.20 (Pin_20)
- net D7: now also J3.17 (Pin_17)
- net GND: now also J2.4 (VDD), L1.1, J3.1 (Pin_1); no longer J1.5 (GND), J1.6 (Shield), L1.2, Q1.2 (E), SW5.1
- net GNDA: now also J1.5 (GND), J1.6 (Shield), L1.2, Q1.2 (E), SW5.1, U?.3, U?.6; no longer L1.1
- net SD_CS: now also J2.2 (CMD)
- net SPI_CLK: now also J2.6 (VSS)
- net SPI_MISO: now also J2.7 (DAT0)
- net SPI_MOSI: now also J2.3 (VSS)
- net VDD: now also L2.1; no longer L2.2, Q2.3 (C), U5.6 (/RD), U7.16 (/RD)
- net at R5.1, R8.1: now also U?.1
- net at C8.1, R9.2: now also U?.2
- net at R6.1, R7.1: now also U?.4
- net at C9.1, R10.2: now also U?.5
- net PWR_USB: now reaches J1.1 (VBUS), Q2.1 (E), R26.2
- net PWR_USB: now also U?.8
- net I2C_DAT renamed ~RD
- net ~RD: now also J3.28 (Pin_28)
- net YM_A0 renamed A0
- net A0: now also J3.30 (Pin_30)
- net YM_A1 renamed A1
- net YM_CS renamed ~YM_CS
- net YM_IC renamed ~RESET
- net ~RESET: now also J3.25 (Pin_25)
- net YM_WR renamed ~WR
- net ~WR: now also J3.27 (Pin_27)
- new net ~LCD_CS: J3.29 (Pin_29)
Other:
- moved on the sheet: D0, D1, D2, D3, D4, D5, D6, D7, J2, R18, R19, R20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

Commit message: 1
Parts:
- gave numbers to parts that had none: 1
Changed lines of the file:
@@
 	21200 1350 21100 1350
 $Comp
-L VGMPlayer-rescue:R_POT_SW U?
+L VGMPlayer-rescue:R_POT_SW U12
 U 1 1 5D145187
 P 10800 6000
-F 0 "U?" H 9962 5846 50  0000 R CNN
+F 0 "U12" H 9962 5846 50  0000 R CNN
 F 1 "R_POT_SW" V 9900 7000 50  0000 R CNN
 F 2 "Connector_Audio:VGM_VR_SW" H 10800 6000 50  0001 C CNN
@@
 	10050 6650 10050 6750
 $Comp
-L power:GNDA #PWR?
+L power:GNDA #PWR0105
 U 1 1 5D3A5019
 P 10050 6750
-F 0 "#PWR?" H 10050 6500 50  0001 C CNN
+F 0 "#PWR0105" H 10050 6500 50  0001 C CNN
 F 1 "GNDA" H 10200 6750 50  0000 C CNN
 F 2 "" H 10050 6750 50  0001 C CNN
@@
 	10050 7000 10050 7050
 $Comp
-L power:+5V #PWR?
+L power:+5V #PWR0106
 U 1 1 5DECAE47
 P 10050 7000
-F 0 "#PWR?" H 10050 6850 50  0001 C CNN
+F 0 "#PWR0106" H 10050 6850 50  0001 C CNN
 F 1 "+5V" H 9900 7050 50  0000 C CNN
 F 2 "" H 10050 7000 50  0001 C CNN

Commit message: 1
Parts:
- added JP1: Jumper_NC_Small, Jumper:SolderJumper-2_P1.3mm_Open_RoundedPad1.0x1.5mm, symbol Device:Jumper_NC_Small
- added U?: STM32F103XX, Package_DIP:DIP-40_W15.24mm_Socket, symbol VGMPlayer-rescue:STM32F103XX
Connections:
- net +3V3: now also J2.6 (VSS); no longer J2.5 (CLK)
- net +5V: now also JP1.1
- net GND: now also J2.8 (DAT1), U?.19 (GND), U?.20 (GND), U?.39 (GND)
- net PWR_USB: now also JP1.2
- net SN_CLK: now also U5.24 (PhiM)
- net SPI_CLK: now also J2.7 (DAT0), U?.21 (B12), U?.22 (B13); no longer J2.6 (VSS)
- net SPI_MISO: now also J2.9 (DAT2), U?.23 (B14); no longer J2.7 (DAT0)
- net SPI_MOSI: now also U?.24 (B15)
- net VDD: now also U?.38 (5V)
- net YM_CLK: no longer U5.24 (PhiM)
Changed lines of the file:
@@
 	1    0    0    -1
 $EndComp
-Text GLabel 2550 3800 2    50   Input ~ 0
-YM_CLK
 $Comp
 L power:VDD #PWR043
@@
 	-1   0    0    1
 $EndComp
-Text GLabel 17700 -900 2    50   Input ~ 0
+Text GLabel 17700 -1100 2    50   Input ~ 0
 SPI_MISO
 Text GLabel 17650 -500 2    50   Input ~ 0
 SPI_MOSI
-Text GLabel 17700 -800 2    50   Input ~ 0
+Text GLabel 17700 -900 2    50   Input ~ 0
 SPI_CLK
 Text GLabel 17650 -400 2    50   Input ~ 0
@@
 	17650 -500 17350 -500
 Wire Wire Line
+	17700 -1100 17350 -1100
+Wire Wire Line
 	17700 -900 17350 -900
-Wire Wire Line
-	17700 -800 17350 -800
 Wire Wire Line
 	17450 -600 17350 -600
@@
 $EndComp
 Wire Wire Line
-	17550 -700 17350 -700
-Wire Wire Line
-	17550 -1300 17550 -700
+	17550 -800 17350 -800
 $Comp
 L Connector_Generic:Conn_02x15_Odd_Even J3
@@
 Wire Wire Line
 	2450 3550 2450 4000
-Wire Wire Line
-	3000 1850 2850 1850
-Connection ~ 2850 1850
 Text GLabel 1700 750  0    50   Input ~ 0
 PWR_USB
@@
 	1    0    0    -1
 $EndComp
+$Comp
+L Device:Jumper_NC_Small JP1
+U 1 1 5C4C3F82
+P 10350 7200
+F 0 "JP1" V 10304 7274 50  0000 L CNN
+F 1 "Jumper_NC_Small" V 10395 7274 50  0000 L CNN
+F 2 "Jumper:SolderJumper-2_P1.3mm_Open_RoundedPad1.0x1.5mm" H 10350 7200 50  0001 C CNN
+F 3 "~" H 10350 7200 50  0001 C CNN
+	1    10350 7200
+	0    1    1    0
+$EndComp
+Wire Wire Line
+	10050 7050 10350 7050
+Wire Wire Line
+	10350 7050 10350 7100
+Connection ~ 10050 7050
+Wire Wire Line
+	10350 7300 10350 7450
+Wire Wire Line
+	10350 7450 10050 7450
+Connection ~ 10050 7450
+Wire Wire Line
+	17550 -1300 17550 -800
+Wire Wire Line
+	17450 -600 17450 -1000
+Wire Wire Line
+	17450 -1000 17350 -1000
+Connection ~ 17450 -600
+Text GLabel 17250 6150 2    50   Input ~ 0
+SPI_MISO
+Text GLabel 17250 6250 2    50   Input ~ 0
+SPI_CLK
+Text GLabel 17250 6050 2    50   Input ~ 0
+SPI_MOSI
+$Comp
+L power:GND #PWR?
+U 1 1 5C67B3E5
+P 15500 6500
+F 0 "#PWR?" H 15500 6250 50  0001 C CNN
+F 1 "GND" H 15350 6450 50  0000 C CNN
+F 2 "" H 15500 6500 50  0001 C CNN
+F 3 "" H 15500 6500 50  0001 C CNN
+	1    15500 6500
+	1    0    0    -1
+$EndComp
+Wire Wire Line
+	17050 4550 17150 4550
+Wire Wire Line
+	17150 4550 17150 6500
+$Comp
+L power:VDD #PWR?
+U 1 1 5C67B3ED
+P 17300 4400
+F 0 "#PWR?" H 17300 4250 50  0001 C CNN
+F 1 "VDD" H 17200 4500 50  0000 C CNN
+F 2 "" H 17300 4400 50  0001 C CNN
+F 3 "" H 17300 4400 50  0001 C CNN
+	1    17300 4400
+	-1   0    0    -1
+$EndComp
+Wire Wire Line
+	15500 6250 15500 6350
+Wire Wire Line
+	15500 6350 15650 6350
+Wire Wire Line
+	15500 6350 15500 6500
+Connection ~ 15500 6350
+Wire Wire Line
+	17050 6350 17250 6350
+Wire Wire Line
+	17250 6250 17050 6250
+Wire Wire Line
+	17250 6050 17050 6050
+$Comp
+L VGMPlayer-rescue:STM32F103XX U?
+U 1 1 5C67B41B
+P 16300 4350
+F 0 "U?" H 15900 4400 50  0000 C CNN
+F 1 "STM32F103XX" H 16250 4400 50  0000 C CNN
+F 2 "Package_DIP:DIP-40_W15.24mm_Socket" H 16300 4400 50  0001 C CNN
+F 3 "" H 16300 4400 50  0001 C CNN
+	1    16300 4350
+	1    0    0    -1
+$EndComp
+Connection ~ 15500 6500
+Wire Wire Line
+	15650 6250 15500 6250
+Wire Wire Line
+	15500 6500 17150 6500
+Wire Wire Line
+	17300 4400 17300 4650
+Wire Wire Line
+	17300 4650 17050 4650
+Wire Wire Line
+	17050 6150 17250 6150
+Text GLabel 17250 6350 2    50   Input ~ 0
+SPI_CLK
+Text GLabel 15400 4250 0    50   Input ~ 0
+YM_MOL
+Text GLabel 15350 5850 0    50   Input ~ 0
+YM_MOR
+Text GLabel 2550 3800 2    50   Input ~ 0
+SN_CLK
 $EndSCHEMATC

Commit message: 1
Parts:
- gave numbers to parts that had none: 1
Connections:
- net I2C_CLK is gone; now on net ~LCD_CS: U1.34 (B6)
- net PWR_HOLD: no longer U1.31 (B3)
- net SD_CS: no longer U1.33 (B5), U2.5 (CS)
- net SPI_CLK: no longer U15.21 (B12)
- net YM_MOL: now also U15.28 (A11)
- net YM_MOR: now also U15.27 (A10)
- new net ~SD_CS: U1.33 (B5), U2.5 (CS)
- new net ~VGM_CS: U1.31 (B3), U15.21 (B12)
Other:
- moved on the sheet: U15
Changed lines of the file:
@@
 	7100 4100 7100 4200
 Text GLabel 6850 1450 2    50   Input ~ 0
-SD_CS
+~SD_CS
 Text GLabel 6850 1150 2    50   Input ~ 0
 SN_WR
@@
 	6900 950  6650 950
 Text GLabel 6850 1350 2    50   Input ~ 0
-I2C_CLK
+~LCD_CS
 Text GLabel 6850 1250 2    50   Output ~ 0
 ~RD
@@
 SPI_CLK
 Text GLabel 17800 1300 2    50   Input ~ 0
-SD_CS
+~SD_CS
 $Comp
 L power:GND #PWR027
@@
 	17450 1000 17450 1700
 Text GLabel 6850 1650 2    50   Input ~ 0
-PWR_HOLD
+~VGM_CS
 Wire Wire Line
 	1200 4600 1400 4600
@@
 	17450 -1000 17350 -1000
 Connection ~ 17450 -600
-Text GLabel 17250 6150 2    50   Input ~ 0
+Text GLabel 16850 5200 2    50   Input ~ 0
 SPI_MISO
-Text GLabel 17250 6250 2    50   Input ~ 0
+Text GLabel 16850 5300 2    50   Input ~ 0
 SPI_CLK
-Text GLabel 17250 6050 2    50   Input ~ 0
+Text GLabel 16850 5100 2    50   Input ~ 0
 SPI_MOSI
 $Comp
-L power:GND #PWR?
+L power:GND #PWR0107
 U 1 1 5C67B3E5
-P 15500 6500
-F 0 "#PWR?" H 15500 6250 50  0001 C CNN
-F 1 "GND" H 15350 6450 50  0000 C CNN
-F 2 "" H 15500 6500 50  0001 C CNN
-F 3 "" H 15500 6500 50  0001 C CNN
-	1    15500 6500
-	1    0    0    -1
-$EndComp
-Wire Wire Line
-	17050 4550 17150 4550
-Wire Wire Line
-	17150 4550 17150 6500
-$Comp
-L power:VDD #PWR?
+P 15100 5550
+F 0 "#PWR0107" H 15100 5300 50  0001 C CNN
+F 1 "GND" H 14950 5500 50  0000 C CNN
+F 2 "" H 15100 5550 50  0001 C CNN
+F 3 "" H 15100 5550 50  0001 C CNN
+	1    15100 5550
+	1    0    0    -1
+$EndComp
+Wire Wire Line
+	16650 3600 16750 3600
+Wire Wire Line
+	16750 3600 16750 5550
+$Comp
+L power:VDD #PWR0108
 U 1 1 5C67B3ED
-P 17300 4400
-F 0 "#PWR?" H 17300 4250 50  0001 C CNN
-F 1 "VDD" H 17200 4500 50  0000 C CNN
-F 2 "" H 17300 4400 50  0001 C CNN
-F 3 "" H 17300 4400 50  0001 C CNN
-	1    17300 4400
+P 16900 3450
+F 0 "#PWR0108" H 16900 3300 50  0001 C CNN
+F 1 "VDD" H 16800 3550 50  0000 C CNN
+F 2 "" H 16900 3450 50  0001 C CNN
+F 3 "" H 16900 3450 50  0001 C CNN
+	1    16900 3450
 	-1   0    0    -1
 $EndComp
 Wire Wire Line
-	15500 6250 15500 6350
-Wire Wire Line
-	15500 6350 15650 6350
-Wire Wire Line
-	15500 6350 15500 6500
-Connection ~ 15500 6350
-Wire Wire Line
-	17050 6350 17250 6350
-Wire Wire Line
-	17250 6250 17050 6250
-Wire Wire Line
-	17250 6050 17050 6050
-$Comp
-L VGMPlayer-rescue:STM32F103XX U?
+	15100 5300 15100 5400
+Wire Wire Line
+	15100 5400 15250 5400
+Wire Wire Line
+	15100 5400 15100 5550
+Connection ~ 15100 5400
+Wire Wire Line
+	16650 5400 16850 5400
+Wire Wire Line
+	16850 5300 16650 5300
+Wire Wire Line
+	16850 5100 16650 5100
+$Comp
+L VGMPlayer-rescue:STM32F103XX U15
 U 1 1 5C67B41B
-P 16300 4350
-F 0 "U?" H 15900 4400 50  0000 C CNN
-F 1 "STM32F103XX" H 16250 4400 50  0000 C CNN
-F 2 "Package_DIP:DIP-40_W15.24mm_Socket" H 16300 4400 50  0001 C CNN
-F 3 "" H 16300 4400 50  0001 C CNN
-	1    16300 4350
-	1    0    0    -1
-$EndComp
-Connection ~ 15500 6500
-Wire Wire Line
-	15650 6250 15500 6250
-Wire Wire Line
-	15500 6500 17150 6500
-Wire Wire Line
-	17300 4400 17300 4650
-Wire Wire Line
-	17300 4650 17050 4650
-Wire Wire Line
-	17050 6150 17250 6150
-Text GLabel 17250 6350 2    50   Input ~ 0
-SPI_CLK
-Text GLabel 15400 4250 0    50   Input ~ 0
+P 15900 3400
+F 0 "U15" H 15500 3450 50  0000 C CNN
+F 1 "STM32F103XX" H 15850 3450 50  0000 C CNN
+F 2 "Package_DIP:DIP-40_W15.24mm_Socket" H 15900 3450 50  0001 C CNN
+F 3 "" H 15900 3450 50  0001 C CNN
+	1    15900 3400
+	1    0    0    -1
+$EndComp
+Connection ~ 15100 5550
+Wire Wire Line
+	15250 5300 15100 5300
+Wire Wire Line
+	15100 5550 16750 5550
+Wire Wire Line
+	16900 3450 16900 3700
+Wire Wire Line
+	16900 3700 16650 3700
+Wire Wire Line
+	16650 5200 16850 5200
+Text GLabel 16850 5400 2    50   Input ~ 0
+~VGM_CS
+Text GLabel 16850 4700 2    50   Input ~ 0
 YM_MOL
-Text GLabel 15350 5850 0    50   Input ~ 0
+Text GLabel 16850 4800 2    50   Input ~ 0
 YM_MOR
 Text GLabel 2550 3800 2    50   Input ~ 0
 SN_CLK
+Wire Wire Line
+	16850 4700 16650 4700
+Wire Wire Line
+	16650 4800 16850 4800
 $EndSCHEMATC

Commit message: 1
Parts:
- removed JP1: Jumper_NC_Small, Jumper:SolderJumper-2_P1.3mm_Open_RoundedPad1.0x1.5mm, symbol Device:Jumper_NC_Small
- removed U15: STM32F103XX, Package_DIP:DIP-40_W15.24mm_Socket, symbol VGMPlayer-rescue:STM32F103XX
- added C10: 1000uF, Capacitor_THT:CP_Radial_D8.0mm_P3.50mm, symbol Device:CP1
- added JP2, JP3, JP4, JP5: Jumper_NC_Small, Jumper:SolderJumper-2_P1.3mm_Open_RoundedPad1.0x1.5mm, symbol Device:Jumper_NC_Small
Connections:
- net +3V3: now also U11.2 (VCC), U19.2 (VCC), C10.1
- net +5V: now also R18.2, R19.2, R20.2, R21.2, R22.2, R23.2, R24.2, R25.2; no longer C25.2, C26.2, C27.1, C28.1, U10.7 (OE), U10.8 (VCC), U12.7, U9.7 (OE), U9.8 (VCC)
- net D6: now also JP2.2
- net D7: now also JP3.2
- net GND: now also J2.11 (SHELL1), C10.2
- net PWR_USB: no longer U12.8
- net SN_CLK: no longer U5.24 (PhiM)
- net VDD: now also C25.2, C26.2, C27.1, C28.1, U10.7 (OE), U10.8 (VCC), U9.7 (OE), U9.8 (VCC); no longer R18.2, R19.2, R20.2, R21.2, R22.2, R23.2, R24.2, R25.2, U11.2 (VCC), U19.2 (VCC)
- net YM_CLK: now also U5.24 (PhiM)
- net YM_MOL: now also JP2.1, JP4.1
- net YM_MOR: now also JP3.1, JP5.1
- net ~WR: now also JP5.2
- net ~YM_CS: now also JP4.2
Other:
- moved on the sheet: U1
