File: noCPU/noCPU/noCPU.sch (KiCad schematic (older format))
At the start: 38 parts, among them SW1 1, U1 74AHC1G08, U1 LM555

Commit message: 1
Parts:
- added U? (x2): 74173, symbol 74xx_IEEE:74173
- added U?: 74HC245, symbol 74xx:74HC245
Connections:
- net BUS_D0: now also U?.14 (P0), U?.18 (B0)
- net BUS_D1: now also U?.13 (P1), U?.17 (B1)
- net BUS_D2: now also U?.12 (P2), U?.16 (B2)
- net BUS_D3: now also U?.11 (P3), U?.15 (B3)
- net BUS_D4: now also U?.14 (B4), U?.14 (P0)
- net BUS_D5: now also U?.13 (B5), U?.13 (P1)
- net BUS_D6: now also U?.12 (B6), U?.12 (P2)
- net BUS_D7: now also U?.11 (B7), U?.11 (P3)
- net CLK_SOURCE: no longer U1.1
- net GND: now also U?.1 (~M), U?.1 (~M), U?.10 (GND), U?.2 (~N), U?.2 (~N), U?.8 (GND), U?.8 (GND)
- net MASTER_CLK: now also U?.7 (CK), U?.7 (CK)
- net VCC: now also U?.16 (VCC), U?.16 (VCC)
- net ~ENABLE: now also U?.19 (CE)
- net ~LOAD: now also U?.10 (~G2), U?.10 (~G2), U?.9 (~G1), U?.9 (~G1)
- new net: U?.2 (A0), U?.3 (Q0)
- new net: U?.3 (A1), U?.4 (Q1)
- new net: U?.4 (A2), U?.5 (Q2)
- new net: U?.5 (A3), U?.6 (Q3)
- new net: U?.3 (Q0), U?.6 (A4)
- new net: U?.4 (Q1), U?.7 (A5)
- new net: U?.5 (Q2), U?.8 (A6)
- new net: U?.6 (Q3), U?.9 (A7)
- new net: U?.1 (A->B), U?.20 (VCC)
Other:
- note added: "Register A"
- note added: "Register B\n"

Commit message: 1
Parts:
- removed U? (x2): 74173, symbol 74xx_IEEE:74173
- removed U?: 74HC245, symbol 74xx:74HC245
- added U10, U11: 74HC86, symbol 74xx:74HC86
- added unit 2 of U11
- added unit 3 of U11
- added unit 4 of U11
- added U? (x4): 74173, symbol 74xx_IEEE:74173
- added U? (x3): 74HC245, symbol 74xx:74HC245
- added U? (x2): 74LS283, symbol 74xx:74LS283
- added U?: 628128, symbol Memory_RAM:628128
- gave numbers to parts that had none: 24
Connections:
- net BUS_D0: now also U?.13 (Q0), U?.14 (P0), U?.14 (P0), U?.18 (B0), U?.18 (B0), U?.18 (B0)
- net BUS_D1: now also U?.13 (P1), U?.13 (P1), U?.14 (Q1), U?.17 (B1), U?.17 (B1), U?.17 (B1)
- net BUS_D2: now also U?.12 (P2), U?.12 (P2), U?.15 (Q2), U?.16 (B2), U?.16 (B2), U?.16 (B2)
- net BUS_D3: now also U?.11 (P3), U?.11 (P3), U?.15 (B3), U?.15 (B3), U?.15 (B3), U?.17 (Q3)
- net BUS_D4: now also U?.14 (B4), U?.14 (B4), U?.14 (B4), U?.14 (P0), U?.14 (P0), U?.18 (Q4)
- net BUS_D5: now also U?.13 (B5), U?.13 (B5), U?.13 (B5), U?.13 (P1), U?.13 (P1), U?.19 (Q5)
- net BUS_D6: now also U?.12 (B6), U?.12 (B6), U?.12 (B6), U?.12 (P2), U?.12 (P2), U?.20 (Q6)
- net BUS_D7: now also U?.11 (B7), U?.11 (B7), U?.11 (B7), U?.11 (P3), U?.11 (P3), U?.21 (Q7)
- net CLK_SOURCE: now also U1.1
- net GND: now also U?.1 (~M), U?.1 (~M), U?.1 (~M), U?.1 (~M), U?.10 (GND), U?.10 (GND), U?.10 (GND), U?.16 (GND), U?.2 (~N), U?.2 (~N), U?.2 (~N), U?.2 (~N), U?.22 (CS1), U?.8 (GND), U?.8 (GND), U?.8 (GND), U?.8 (GND), U?.8 (GND), U?.8 (GND)
- net MASTER_CLK: now also U?.7 (CK), U?.7 (CK), U?.7 (CK), U?.7 (CK)
- net VCC: now also U11.1 (A->B), U11.20 (VCC), U?.1 (A->B), U?.1 (A->B), U?.16 (VCC), U?.16 (VCC), U?.16 (VCC), U?.16 (VCC), U?.16 (VCC), U?.16 (VCC), U?.20 (VCC), U?.20 (VCC), U?.30 (CS2), U?.32 (VCC)
- net REGA_D0: now reaches U11.2 (A0), U7.3 (Q0)
- net REGA_D0: now also U?.2 (A0), U?.3 (Q0), U?.5 (A1)
- net REGA_D1: now reaches U11.3 (A1), U7.4 (Q1)
- net REGA_D1: now also U?.3 (A1), U?.3 (A2), U?.4 (Q1)
- net REGA_D2: now reaches U11.4 (A2), U7.5 (Q2)
- net REGA_D2: now also U?.14 (A3), U?.4 (A2), U?.5 (Q2)
- net REGA_D3: now reaches U11.5 (A3), U7.6 (Q3)
- net REGA_D3: now also U?.12 (A4), U?.5 (A3), U?.6 (Q3)
- net REGA_D4: now reaches U11.6 (A4), U8.3 (Q0)
- net REGA_D4: now also U?.3 (Q0), U?.5 (A1), U?.6 (A4)
- net REGA_D5: now reaches U11.7 (A5), U8.4 (Q1)
- net REGA_D5: now also U?.3 (A2), U?.4 (Q1), U?.7 (A5)
- net REGA_D6: now reaches U11.8 (A6), U8.5 (Q2)
- net REGA_D6: now also U?.14 (A3), U?.5 (Q2), U?.8 (A6)
- net REGA_D7: now reaches U11.9 (A7), U8.6 (Q3)
- net REGA_D7: now also U?.12 (A4), U?.6 (Q3), U?.9 (A7)
- net ~ENABLE renamed ~AO
- net ~AO: now also U?.19 (CE)
- net ~LOAD renamed ~AI
- net ~AI: now also U?.10 (~G2), U?.10 (~G2), U?.9 (~G1), U?.9 (~G1)
- new net: U?.1 (A->B), U?.20 (VCC)
- new net: U?.1 (S2), U?.3 (A1)
- new net: U?.10 (S4), U?.5 (A3)
- new net: U10.11, U?.11 (B4)
- new net: U?.13 (S3), U?.4 (A2)
- new net: U10.8, U?.15 (B3)
- new net: U10.6, U?.2 (B2)
- new net: U?.2 (A0), U?.4 (S1)
- new net: U10.3, U?.6 (B1)
- new net: U?.7 (C0), U?.9 (C4)
- new net: U?.1 (S2), U?.7 (A5)
- new net: U?.10 (S4), U?.9 (A7)
- new net: U11.11, U?.11 (B4)
- new net: U?.13 (S3), U?.8 (A6)
- new net: U11.8, U?.15 (B3)
- new net: U11.6, U?.2 (B2)
- new net: U?.4 (S1), U?.6 (A4)
- new net: U11.3, U?.6 (B1)
- new net REGB_D0: U10.1, U?.2 (A0), U?.3 (Q0)
- new net REGB_D1: U10.4, U?.3 (A1), U?.4 (Q1)
- new net REGB_D2: U10.9, U?.4 (A2), U?.5 (Q2)
- new net REGB_D3: U10.12, U?.5 (A3), U?.6 (Q3)
- new net REGB_D4: U11.1, U?.3 (Q0), U?.6 (A4)
- new net REGB_D5: U11.4, U?.4 (Q1), U?.7 (A5)
- new net REGB_D6: U11.9, U?.5 (Q2), U?.8 (A6)
- new net REGB_D7: U11.12, U?.6 (Q3), U?.9 (A7)
- new net RI: U?.29 (WR)
- new net RO: U?.24 (OE)
- new net SO: U?.19 (CE)
- new net SU: U10.10, U10.13, U10.2, U10.5, U11.10, U11.13, U11.2, U11.5, U?.7 (C0)
- new net ~BI: U?.10 (~G2), U?.10 (~G2), U?.9 (~G1), U?.9 (~G1)
- new net ~BO: U?.19 (CE)
Other:
- note added: "ALU"
- note added: "CLOCK\n"
- note added: "Memory Address Register\n"
- note added: "Register B"
- note removed: "Register B\n"
- moved on the sheet: C3, C4, C5, C6, C7, D2, D3, D4, D5, R1, R10, R2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

Commit message: 1
Parts:
- removed U11, U? (x3): 74HC245, symbol 74xx:74HC245
- removed U7, U8, U? (x4): 74173, symbol 74xx_IEEE:74173
- removed U? (x2): 74LS283, symbol 74xx:74LS283
- removed U?: 628128, symbol Memory_RAM:628128
- added D? (x6): LED, LED_SMD:LED_0805_2012Metric, symbol Device:LED
- added R? (x4): 330, Resistor_SMD:R_0805_2012Metric, symbol Device:R
- added R? (x2): 1k, Resistor_SMD:R_0805_2012Metric, symbol Device:R
- added SW?: SW_DIP_x08, symbol Switch:SW_DIP_x08
- added SW?: SW_SPDT, symbol Switch:SW_SPDT
- added U10, U11, U12, U9, U? (x6): 74HC173, symbol NOCPU:74HC173
- added U4, U5, U6, U? (x3): 74HC245, symbol NOCPU:74HC245
- added U7, U8: 74HC283, symbol NOCPU:74HC283
- added U?: 62256, symbol NOCPU:62256
- added U? (x2): 74HC157, symbol NOCPU:74HC157
- added U? (x2): 74HC161, symbol NOCPU:74HC161
- renumbered C4 to C3, C5 to C4, C6 to C5, C7 to C6, C3 to C7, R4 to R1, R5 to R2, R6 to R3, R1 to R4, R7 to R5, R2 to R6, R3 to R7, U10 to U13, U11 to U14, U1 to U15, U2 to U16, U3 to U17, U4 to U18, U1 to U19, U1 to U20, U5 to U21, U6 to U22, U1 to U23
Connections:
- net BUS_D0: now also U10.14 (D0), U4.18 (B0), U5.18 (B0), U6.18 (B0), U9.14 (D0), U?.11 (IO0), U?.14 (D0), U?.14 (D0), U?.14 (D0), U?.18 (B0), U?.18 (B0), U?.18 (B0), U?.3 (D0)
- net BUS_D1: now also U10.13 (D1), U4.17 (B1), U5.17 (B1), U6.17 (B1), U9.13 (D1), U?.12 (IO1), U?.13 (D1), U?.13 (D1), U?.13 (D1), U?.17 (B1), U?.17 (B1), U?.17 (B1), U?.4 (D1)
- net BUS_D2: now also U10.12 (D2), U4.16 (B2), U5.16 (B2), U6.16 (B2), U9.12 (D2), U?.12 (D2), U?.12 (D2), U?.12 (D2), U?.13 (IO2), U?.16 (B2), U?.16 (B2), U?.16 (B2), U?.5 (D2)
- net BUS_D3: now also U10.11 (D3), U4.15 (B3), U5.15 (B3), U6.15 (B3), U9.11 (D3), U?.11 (D3), U?.11 (D3), U?.11 (D3), U?.15 (B3), U?.15 (B3), U?.15 (B3), U?.15 (IO3), U?.6 (D3)
- net BUS_D4: now also U11.14 (D0), U12.14 (D0), U4.14 (B4), U5.14 (B4), U6.14 (B4), U?.14 (B4), U?.14 (B4), U?.14 (B4), U?.14 (D0), U?.14 (D0), U?.14 (D0), U?.16 (IO4), U?.3 (D0)
- net BUS_D5: now also U11.13 (D1), U12.13 (D1), U4.13 (B5), U5.13 (B5), U6.13 (B5), U?.13 (B5), U?.13 (B5), U?.13 (B5), U?.13 (D1), U?.13 (D1), U?.13 (D1), U?.17 (IO5), U?.4 (D1)
- net BUS_D6: now also U11.12 (D2), U12.12 (D2), U4.12 (B6), U5.12 (B6), U6.12 (B6), U?.12 (B6), U?.12 (B6), U?.12 (B6), U?.12 (D2), U?.12 (D2), U?.12 (D2), U?.18 (IO6), U?.5 (D2)
- net BUS_D7: now also U11.11 (D3), U12.11 (D3), U4.11 (B7), U5.11 (B7), U6.11 (B7), U?.11 (B7), U?.11 (B7), U?.11 (B7), U?.11 (D3), U?.11 (D3), U?.11 (D3), U?.19 (IO7), U?.6 (D3)
- net GND: now also D?.1 (K), D?.1 (K), D?.1 (K), D?.1 (K), SW?.1, SW?.2, SW?.2 (B), SW?.3, SW?.4, SW?.5, SW?.6, SW?.7, SW?.8, U10.1 (~OE1), U10.15 (R), U10.2 (~OE2), U10.8 (GND), U11.1 (~OE1), U11.15 (R), U11.2 (~OE2), U11.8 (GND), U12.1 (~OE1), U12.15 (R), U12.2 (~OE2), U12.8 (GND), U4.10 (GND), U5.10 (GND), U6.10 (GND), U7.8 (GND), U8.8 (GND), U9.1 (~OE1), U9.15 (R), U9.2 (~OE2), U9.8 (GND), U?.1 (~OE1), U?.1 (~OE1), U?.1 (~OE1), U?.1 (~OE1), U?.1 (~OE1), U?.1 (~OE1), U?.10 (A14), U?.10 (GND), U?.10 (GND), U?.10 (GND), U?.15 (E), U?.15 (E), U?.15 (R), U?.15 (R), U?.15 (R), U?.15 (R), U?.15 (R), U?.15 (R), U?.2 (~OE2), U?.2 (~OE2), U?.2 (~OE2), U?.2 (~OE2), U?.2 (~OE2), U?.2 (~OE2), U?.20 (~CE), U?.28 (VCC), U?.4 (A8), U?.5 (A9), U?.6 (A10), U?.7 (A11), U?.8 (A12), U?.8 (GND), U?.8 (GND), U?.8 (GND), U?.8 (GND), U?.8 (GND), U?.8 (GND), U?.8 (GND), U?.8 (GND), U?.8 (GND), U?.8 (GND), U?.9 (A13)
- net MASTER_CLK: now also U10.7 (CK), U11.7 (CK), U12.7 (CK), U9.7 (CK), U?.2 (CP), U?.2 (CP), U?.7 (CK), U?.7 (CK), U?.7 (CK), U?.7 (CK), U?.7 (CK), U?.7 (CK)
- net REGA_D0: now also U4.2 (A0), U7.5 (A1), U9.3 (Q0)
- net REGA_D1: now also U4.3 (A1), U7.3 (A2), U9.4 (Q1)
- net REGA_D2: now also U4.4 (A2), U7.14 (A3), U9.5 (Q2)
- net REGA_D3: now also U4.5 (A3), U7.12 (A4), U9.6 (Q3)
- net REGA_D4: now also U11.3 (Q0), U4.6 (A4), U8.5 (A1)
- net REGA_D5: now also U11.4 (Q1), U4.7 (A5), U8.3 (A2)
- net REGA_D6: now also U11.5 (Q2), U4.8 (A6), U8.14 (A3)
- net REGA_D7: now also U11.6 (Q3), U4.9 (A7), U8.12 (A4)
- net REGB_D0: now also U10.3 (Q0), U6.2 (A0)
- net REGB_D1: now also U10.4 (Q1), U6.3 (A1)
- net REGB_D2: now also U10.5 (Q2), U6.4 (A2)
- net REGB_D3: now also U10.6 (Q3), U6.5 (A3)
- net REGB_D4: now also U12.3 (Q0), U6.6 (A4)
- net REGB_D5: now also U12.4 (Q1), U6.7 (A5)
- net REGB_D6: now also U12.5 (Q2), U6.8 (A6)
- net REGB_D7: now also U12.6 (Q3), U6.9 (A7)
- net SO: now also U5.19 (CE)
- net SU: now also U7.7 (C0)
- net VCC: now also R?.1, R?.1, U10.16 (VCC), U11.16 (VCC), U12.16 (VCC), U4.1 (A->B), U4.20 (VCC), U5.1 (A->B), U5.20 (VCC), U6.1 (A->B), U6.20 (VCC), U7.16 (VCC), U8.16 (VCC), U9.16 (VCC), U?.1 (A->B), U?.1 (A->B), U?.1 (A->B), U?.1 (~MR), U?.1 (~MR), U?.14 (GND), U?.16 (VCC), U?.16 (VCC), U?.16 (VCC), U?.16 (VCC), U?.16 (VCC), U?.16 (VCC), U?.16 (VCC), U?.16 (VCC), U?.16 (VCC), U?.16 (VCC), U?.20 (VCC), U?.20 (VCC), U?.20 (VCC)
- net ~AI: now also U11.10 (~E2), U11.9 (~E1), U9.10 (~E2), U9.9 (~E1)
- net ~AO: now also U4.19 (CE)
- net ~BI: now also U10.10 (~E2), U10.9 (~E1), U12.10 (~E2), U12.9 (~E1)
- net ~BO: now also U6.19 (CE), U?.19 (CE)
- net at U13.11: now also U7.11 (B4)
- net at U13.8: now also U7.15 (B3)
- net at U13.6: now also U7.2 (B2)
- net at U13.3: now also U7.6 (B1)
- net at U14.11: now also U8.11 (B4)
- net at U14.8: now also U8.15 (B3)
- net at U14.6: now also U8.2 (B2)
- net at U14.3: now also U8.6 (B1)
- new net: U5.3 (A1), U7.1 (S2)
- new net: U5.5 (A3), U7.10 (S4)
- new net: U5.4 (A2), U7.13 (S3)
- new net: U5.2 (A0), U7.4 (S1)
- new net: U7.9 (C4), U8.7 (C0)
- new net: U5.7 (A5), U8.1 (S2)
- new net: U5.9 (A7), U8.10 (S4)
- new net: U5.8 (A6), U8.13 (S3)
- new net: U5.6 (A4), U8.4 (S1)
- new net: D?.2 (A), R?.2 (x5)
- new net: U?.2 (I0a), U?.3 (Q0) (x2)
- new net: U?.4 (Q1), U?.5 (I0b)
- new net: U?.14 (I0c), U?.5 (Q2) (x2)
- new net: U?.11 (I0d), U?.6 (Q3) (x2)
- new net: SW?.16, U?.10 (I1d), U?.4 (Q1), U?.5 (I0b)
- new net: SW?.10, U?.6 (I1b)
- new net: SW?.11, U?.13 (I1c)
- new net: SW?.12, U?.10 (I1d)
- new net: SW?.13, U?.3 (I1a)
- new net: SW?.14, U?.6 (I1b)
- new net: SW?.15, U?.13 (I1c)
- new net: SW?.9, U?.3 (I1a)
- new net: D?.2 (A), R?.2, U?.1 (S), U?.1 (S)
- new net: U?.11 (Q3), U?.5 (A3)
- new net: U?.12 (Q2), U?.4 (A2)
- new net: U?.13 (Q1), U?.3 (A1)
- new net: U?.14 (Q0), U?.2 (A0)
- new net: U?.10 (CET), U?.15 (TC), U?.7 (CEP)
- new net: U?.14 (Q0), U?.6 (A4)
- new net: U?.13 (Q1), U?.7 (A5)
- new net: U?.12 (Q2), U?.8 (A6)
- new net: U?.11 (Q3), U?.9 (A7)
- new net: D?.1 (K), SW?.1 (A)
- new net: D?.1 (K), SW?.3 (C)
- new net CE: U?.10 (CET), U?.7 (CEP)
- new net J: U?.9 (~PE), U?.9 (~PE)
- new net MAR0: U?.21 (A0), U?.4 (Za)
- new net MAR1: U?.23 (A1), U?.7 (Zb)
- new net MAR2: U?.12 (Zc), U?.24 (A2)
- new net MAR3: U?.25 (A3), U?.9 (Zd)
- new net MAR4: U?.26 (A4), U?.4 (Za)
- new net MAR5: U?.1 (A5), U?.7 (Zb)
- new net MAR6: U?.12 (Zc), U?.2 (A6)
- new net MAR7: U?.3 (A7), U?.9 (Zd)
- new net REGI_D0: U?.2 (A0), U?.3 (Q0)
- new net REGI_D1: U?.3 (A1), U?.4 (Q1)
- new net REGI_D2: U?.4 (A2), U?.5 (Q2)
- new net REGI_D3: U?.5 (A3), U?.6 (Q3)
- new net REGI_D4: U?.3 (Q0), U?.6 (A4)
- new net REGI_D5: U?.4 (Q1), U?.7 (A5)
- new net REGI_D6: U?.5 (Q2), U?.8 (A6)
- new net REGI_D7: U?.6 (Q3), U?.9 (A7)
- new net REGO_D0: U?.2 (A0), U?.3 (Q0)
- new net REGO_D1: U?.3 (A1), U?.4 (Q1)
- new net REGO_D2: U?.4 (A2), U?.5 (Q2)
- new net REGO_D3: U?.5 (A3), U?.6 (Q3)
- new net REGO_D4: U?.3 (Q0), U?.6 (A4)
- new net REGO_D5: U?.4 (Q1), U?.7 (A5)
- new net REGO_D6: U?.5 (Q2), U?.8 (A6)
- new net REGO_D7: U?.6 (Q3), U?.9 (A7)
- new net ~CO: U?.19 (CE)
- new net ~II: U?.10 (~E2), U?.10 (~E2), U?.9 (~E1), U?.9 (~E1)
- new net ~IO: U?.19 (CE)
- new net ~MI: U?.10 (~E2), U?.10 (~E2), U?.9 (~E1), U?.9 (~E1)
- new net ~OI: U?.10 (~E2), U?.10 (~E2), U?.9 (~E1), U?.9 (~E1)
- new net ~RI: U?.27 (~WE)
- new net ~RO: U?.22 (~OE)
Other:
- note added: "IO Register\n"
- note added: "Instruction Register\n"
- note added: "Memory\n"
- note added: "Program Counter\n\n"
- moved on the sheet: U13A, U13B, U13C, U13D, U14A, U14B, U14C, U14D

Commit message: 1
Parts:
- added C?: 1uF, Capacitor_THT:CP_Radial_D8.0mm_P3.50mm, symbol Device:CP1
- added C?: 0.1uF, Capacitor_SMD:C_0805_2012Metric, symbol Device:C
- added D? (x8): LED, LED_SMD:LED_0805_2012Metric, symbol Device:LED
- added R? (x8): 330, Resistor_SMD:R_0805_2012Metric, symbol Device:R
- added R? (x2): 1k, Resistor_SMD:R_0805_2012Metric, symbol Device:R
- added RV?: 100k, symbol Device:R_POT
- added U?: LM555, symbol Timer:LM555
- added U?: 74HC161, symbol NOCPU:74HC161
- added U? (x4): MAN71A, Display_7Segment:MAN71A, symbol Display_Character:MAN71A
Connections:
- net BUS_D0: now also R?.1
- net BUS_D1: now also R?.1
- net BUS_D2: now also R?.1
- net BUS_D3: now also R?.1
- net BUS_D4: now also R?.1
- net BUS_D5: now also R?.1
- net BUS_D6: now also R?.1
- net BUS_D7: now also R?.1
- net GND: now also C?.2, C?.2, D?.1 (K), D?.1 (K), D?.1 (K), D?.1 (K), D?.1 (K), D?.1 (K), D?.1 (K), D?.1 (K), U?.1 (GND), U?.8 (GND)
- net VCC: now also R?.1, U?.1 (~MR), U?.14 (CA), U?.14 (CA), U?.14 (CA), U?.14 (CA), U?.16 (VCC), U?.3 (CA), U?.3 (CA), U?.3 (CA), U?.3 (CA), U?.4 (R), U?.8 (VCC), U?.9 (~PE)
- net ~BO: no longer U?.19 (CE)
- net ~OI: no longer U?.10 (~E2), U?.10 (~E2), U?.9 (~E1), U?.9 (~E1)
- new net: D?.2 (A), R?.2 (x8)
- new net: C?.1, R?.2, U?.2 (TR), U?.6 (THR)
- new net: U?.2 (CP), U?.3 (Q)
- new net: C?.1, U?.5 (CV)
- new net: R?.2, RV?.2, U?.7 (DIS)
- new net: R?.1, RV?.3
- new net: U?.10 (CET), U?.3 (D0), U?.4 (D1), U?.5 (D2), U?.6 (D3), U?.7 (CEP)
- new net ~PI: U?.10 (~E2), U?.10 (~E2), U?.9 (~E1), U?.9 (~E1)
- new net ~PO: U?.19 (CE)
Other:
- moved on the sheet: D?, R?, SW?, U?

Commit message: 1
Parts:
- removed C1: CP1, Capacitor_THT:CP_Radial_D8.0mm_P3.50mm, symbol Device:CP1
- removed C2: 1uF, Capacitor_SMD:C_0805_2012Metric, symbol Device:C
- removed SW1: 1, Resistor_SMD:R_0805_2012Metric, symbol Switch:SW_DIP_x01
- removed U? (x4): MAN71A, Display_7Segment:MAN71A, symbol Display_Character:MAN71A
- added D10, D11, D12, D13, D14, D15, D18, D19, D2, D20, D21, D22, D23, D24, D25, D26, D3, D39, D4, D40, D41, D42, D43, D44, D45, D46, D47, D48, D49, D5, D50, D51, D52, D53, D54, D55, D56, D57, D58, D6, D7, D8, D9: LED, LED_SMD:LED_0805_2012Metric, symbol Device:LED
- added R1, R10, R11, R13, R14, R16, R17, R18, R19, R2, R20, R21, R22, R23, R24, R25, R26, R3, R39, R4, R40, R41, R42, R43, R44, R45, R46, R47, R48, R49, R5, R50, R51, R52, R53, R54, R55, R56, R57, R58, R6, R7, R8, R9: 330, Resistor_SMD:R_0805_2012Metric, symbol Device:R
- added U10: 74LS138, Package_DIP:DIP-18_W7.62mm, symbol 74xx:74LS138
- added U11, U36, U8: 62256, Package_DIP:DIP-28_W15.24mm, symbol NOCPU:62256
- added U13, U19, U24, U32: MAN71A, Display_7Segment:MAN71A, symbol Display_Character:MAN71A
- added U7: 74HC161, Package_DIP:DIP-16_W7.62mm, symbol NOCPU:74HC161
- RV1: renamed from RV?; footprint (none) -> Connector_PinHeader_2.54mm:PinHeader_1x03_P2.54mm_Horizontal
- RV2: renamed from RV1; footprint (none) -> Connector_PinHeader_2.54mm:PinHeader_1x03_P2.54mm_Horizontal
- SW1, SW2: renamed from SW?; footprint (none) -> Package_DIP:DIP-4_W7.62mm
- SW3: footprint (none) -> Package_DIP:DIP-4_W7.62mm
- SW4: renamed from SW2; footprint Resistor_SMD:R_0805_2012Metric -> Package_DIP:DIP-4_W7.62mm
- U1, U2, U23, U27, U28, U3, U31, U35, U4, U5, U9: renamed from U?; footprint (none) -> Package_DIP:DIP-16_W7.62mm
- U12, U14, U18: renamed from U?; footprint (none) -> Package_DIP:DIP-20_W7.62mm
- U15: renamed from U4; footprint (none) -> Package_DIP:DIP-20_W7.62mm
- U16: renamed from U5; footprint (none) -> Package_DIP:DIP-20_W7.62mm
- U17: renamed from U6; footprint (none) -> Package_DIP:DIP-20_W7.62mm
- U20: renamed from U7; footprint (none) -> Package_DIP:DIP-16_W7.62mm
- U21: renamed from U8; footprint (none) -> Package_DIP:DIP-16_W7.62mm
- U22: renamed from U?; footprint (none) -> Package_DIP:DIP-8_W7.62mm
- U25: renamed from U9; footprint (none) -> Package_DIP:DIP-16_W7.62mm
- U26: renamed from U10; footprint (none) -> Package_DIP:DIP-16_W7.62mm
- U29: renamed from U11; footprint (none) -> Package_DIP:DIP-16_W7.62mm
- U30: renamed from U12; footprint (none) -> Package_DIP:DIP-16_W7.62mm
- U33: renamed from U13; footprint (none) -> Package_DIP:DIP-14_W7.62mm
- U34: renamed from U14; footprint (none) -> Package_DIP:DIP-14_W7.62mm
- U37: renamed from U23; footprint (none) -> Package_DIP:DIP-14_W7.62mm
- U38: renamed from U22; footprint (none) -> Package_DIP:DIP-14_W7.62mm
- U39: renamed from U21; footprint (none) -> Package_DIP:DIP-14_W7.62mm
- U40: renamed from U19; footprint (none) -> Package_DIP:DIP-14_W7.62mm
- U41: renamed from U20; footprint (none) -> Package_DIP:DIP-14_W7.62mm
- U42: renamed from U18; footprint (none) -> Package_DIP:DIP-14_W7.62mm
- U43: renamed from U15; footprint (none) -> Package_DIP:DIP-8_W7.62mm
- U44: renamed from U16; footprint (none) -> Package_DIP:DIP-8_W7.62mm
- U45: renamed from U17; footprint (none) -> Package_DIP:DIP-8_W7.62mm
- U6: renamed from U?; footprint (none) -> Package_DIP:DIP-28_W15.24mm
- gave numbers to parts that had none: 32
- renumbered C7 to C3, C6 to C4, C4 to C6, C3 to C7, D5 to D59, D2 to D60, D3 to D61, D4 to D62, R10 to R61, R7 to R62, R8 to R63, R9 to R64, R6 to R65, R4 to R66, R5 to R67, R3 to R68, R1 to R69, R2 to R70
Connections:
- net GND: now also D1.1 (K), U6.14 (GND), D19.1 (K), D2.1 (K), D20.1 (K), D21.1 (K), D22.1 (K), D23.1 (K), D24.1 (K), D25.1 (K), D26.1 (K), D3.1 (K), D39.1 (K), D4.1 (K), D40.1 (K), D41.1 (K), D42.1 (K), D43.1 (K), D44.1 (K), D45.1 (K), D46.1 (K), D47.1 (K), D48.1 (K), D49.1 (K), D5.1 (K), D50.1 (K), D51.1 (K), D52.1 (K), D53.1 (K), D54.1 (K), D55.1 (K), D56.1 (K), D57.1 (K), D58.1 (K), D6.1 (K), D7.1 (K), D8.1 (K), U10.4 (E1), U10.5 (E2), U10.8 (GND), U11.10 (A14), U11.14 (GND), U11.20 (~CE), U11.22 (~OE), U11.8 (A12), U11.9 (A13), U36.10 (A14), U36.14 (GND), U36.20 (~CE), U36.22 (~OE), U36.6 (A10), U36.7 (A11), U36.8 (A12), U36.9 (A13), U7.3 (D0), U7.4 (D1), U7.5 (D2), U7.6 (D3), U7.8 (GND), U8.10 (A14), U8.14 (GND), U8.20 (~CE), U8.22 (~OE), U8.8 (A12), U8.9 (A13); no longer U6.28 (VCC)
- net HLT: now also U8.19 (IO7)
- net J: now also U11.12 (IO1)
- net MAR0: now also R8.1
- net MAR1: now also R7.1
- net MAR2: now also R6.1
- net MAR3: now also R5.1
- net MAR4: now also R4.1
- net MAR5: now also R3.1
- net MAR6: now also R2.1
- net MAR7: now also R1.1
- net MASTER_CLK: now also U7.2 (CP)
- net REGA_D0: now also R35.1
- net REGA_D1: now also R36.1
- net REGA_D2: now also R37.1
- net REGA_D3: now also R38.1
- net REGA_D4: now also R39.1
- net REGA_D5: now also R40.1
- net REGA_D6: now also R41.1
- net REGA_D7: now also R42.1
- net REGB_D0: now also R43.1
- net REGB_D1: now also R44.1
- net REGB_D2: now also R45.1
- net REGB_D3: now also R46.1
- net REGB_D4: now also R47.1
- net REGB_D5: now also R48.1
- net REGB_D6: now also R49.1
- net REGB_D7: now also R50.1
- net REGI_D0: now also R16.1, U11.26 (A4), U8.26 (A4)
- net REGI_D1: now also R17.1, U11.1 (A5), U8.1 (A5)
- net REGI_D2: now also R18.1, U11.2 (A6), U8.2 (A6)
- net REGI_D3: now also R19.1, U11.3 (A7), U8.3 (A7)
- net REGI_D4: now also R20.1, U11.4 (A8), U8.4 (A8)
- net REGI_D5: now also R21.1, U11.5 (A9), U8.5 (A9)
- net REGI_D6: now also R22.1, U11.6 (A10), U8.6 (A10)
- net REGI_D7: now also R23.1, U11.7 (A11), U8.7 (A11)
- net REGO_D0: now also R51.1, U36.21 (A0)
- net REGO_D1: now also R52.1, U36.23 (A1)
- net REGO_D2: now also R53.1, U36.24 (A2)
- net REGO_D3: now also R54.1, U36.25 (A3)
- net REGO_D4: now also R55.1, U36.26 (A4)
- net REGO_D5: now also R56.1, U36.1 (A5)
- net REGO_D6: now also R57.1, U36.2 (A6)
- net REGO_D7: now also R58.1, U36.3 (A7)
- net SU: now also U11.18 (IO6)
- net VCC: now also U6.28 (VCC), R10.1, R11.1, R13.1, R14.1, R24.1, R25.1, R26.1, R9.1, U10.16 (VCC), U10.6 (E3), U11.27 (~WE), U11.28 (VCC), U13.14 (CA), U13.3 (CA), U19.14 (CA), U19.3 (CA), U24.14 (CA), U24.3 (CA), U32.14 (CA), U32.3 (CA), U36.27 (~WE), U36.28 (VCC), U7.1 (~MR), U7.10 (CET), U7.16 (VCC), U7.7 (CEP), U7.9 (~PE), U8.27 (~WE), U8.28 (VCC); no longer U6.14 (GND)
- net ~AI: now also U8.12 (IO1)
- net ~AO: now also U8.11 (IO0)
- net ~BI: now also U11.17 (IO5)
- net ~BO: now also U11.11 (IO0)
- net ~CE: now also U11.13 (IO2)
- net ~CO: now also U11.15 (IO3)
- net ~II: now also U8.13 (IO2)
- net ~IO: now also U8.15 (IO3)
- net ~MI: now also U8.18 (IO6)
- net ~OI: now also U11.16 (IO4)
- net ~RI: now also U8.17 (IO5)
- net ~RO: now also U8.16 (IO4)
- net ~SO: now also U11.19 (IO7)
- net at D1.2 (A): now also R1.2
- net at U1.4 (Q1), U4.5 (I0b): no longer SW1.16, U4.10 (I1d)
- net at U35.13 (Q1): now also U36.5 (A9)
- net at U35.14 (Q0): now also U36.4 (A8)
- new net: SW1.16, U4.10 (I1d)
- new net: U10.1 (A0), U11.21 (A0), U7.14 (Q0), U8.21 (A0)
- new net: U10.2 (A1), U11.23 (A1), U7.13 (Q1), U8.23 (A1)
- new net: U10.3 (A2), U11.24 (A2), U7.12 (Q2), U8.24 (A2)
- new net: U11.25 (A3), U7.11 (Q3), U8.25 (A3)
- new net: D39.2 (A), R39.2
- new net: D40.2 (A), R40.2
- new net: D41.2 (A), R41.2
- new net: D42.2 (A), R42.2
- new net: D51.2 (A), R51.2
- new net: D52.2 (A), R52.2
- new net: D53.2 (A), R53.2
- new net: D54.2 (A), R54.2
- new net: D55.2 (A), R55.2
- new net: D56.2 (A), R56.2
- new net: D57.2 (A), R57.2
- new net: D58.2 (A), R58.2
- new net: D8.2 (A), R8.2
- new net: D7.2 (A), R7.2
- new net: D6.2 (A), R6.2
- new net: D5.2 (A), R5.2
- new net: D4.2 (A), R4.2
- new net: D3.2 (A), R3.2
- new net: D2.2 (A), R2.2
- new net: D11.1 (K), U10.10 (O5)
- new net: D12.1 (K), U10.11 (O4)
- new net: D13.1 (K), U10.12 (O3)
- new net: D14.1 (K), U10.13 (O2)
- new net: D15.1 (K), U10.14 (O1)
- new net: D18.1 (K), U10.15 (O0)
- new net: D9.1 (K), U10.7 (O7)
- new net: D10.1 (K), U10.9 (O6)
- new net: D19.2 (A), R16.2
- new net: D20.2 (A), R17.2
- new net: D21.2 (A), R18.2
- new net: D22.2 (A), R19.2
- new net: D23.2 (A), R20.2
- new net: D24.2 (A), R21.2
- new net: D25.2 (A), R22.2
- new net: D26.2 (A), R23.2
- new net: D9.2 (A), R9.2
- new net: D10.2 (A), R10.2
- new net: D11.2 (A), R11.2
- new net: D12.2 (A), R13.2
- new net: D13.2 (A), R14.2
- new net: D14.2 (A), R24.2
- new net: D15.2 (A), R25.2
- new net: D18.2 (A), R26.2
- new net: D43.2 (A), R43.2
- new net: D44.2 (A), R44.2
- new net: D45.2 (A), R45.2
- new net: D46.2 (A), R46.2
- new net: D47.2 (A), R47.2
- new net: D48.2 (A), R48.2
- new net: D49.2 (A), R49.2
- new net: D50.2 (A), R50.2
- new net SEG0: U13.1 (A), U19.1 (A), U24.1 (A), U32.1 (A), U36.11 (IO0)
- new net SEG1: U13.13 (B), U19.13 (B), U24.13 (B), U32.13 (B), U36.12 (IO1)
- new net SEG2: U13.10 (C), U19.10 (C), U24.10 (C), U32.10 (C), U36.13 (IO2)
- new net SEG3: U13.8 (D), U19.8 (D), U24.8 (D), U32.8 (D), U36.15 (IO3)
- new net SEG4: U13.7 (E), U19.7 (E), U24.7 (E), U32.7 (E), U36.16 (IO4)
- new net SEG5: U13.2 (F), U19.2 (F), U24.2 (F), U32.2 (F), U36.17 (IO5)
- new net SEG6: U13.11 (G), U19.11 (G), U24.11 (G), U32.11 (G), U36.18 (IO6)
- new net SEG7: U13.9 (D.P.), U19.9 (D.P.), U24.9 (D.P.), U32.9 (D.P.), U36.19 (IO7)
Other:
- note added: "Instruction Decoder\n"
- moved on the sheet: C1, C2, C3, C4, C5, C6, C7, D16, D17, D27, D28, D29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

Commit message: 1
Parts:
- removed D1, D2, D3, D4, D5, D6, D7, D8: LED, LED_SMD:LED_0805_2012Metric, symbol Device:LED
- added D10, D11, D12, D13, D14, D15, D16, D33, D34, D35, D36, D37, D38, D39, D40, D65, D66, D67, D68, D69, D70, D71, D72, D73, D74, D75, D76, D77, D78, D79, D80, D81, D82, D9: LED, LED_SMD:LED_0805_2012Metric, symbol Device:LED
- added R25, R26, R71, R72, R73, R74, R75, R76, R77, R78, R79, R80, R81, R82, R83, R84, R85, R86, R87, R88, R89, R90, R91, R92, R93, R94: 330, Resistor_SMD:R_0805_2012Metric, symbol Device:R
- RV1: footprint Connector_PinHeader_2.54mm:PinHeader_1x03_P2.54mm_Horizontal -> Connector_PinHeader_2.54mm:PinHeader_1x03_P2.54mm_Vertical
- SW1: footprint Package_DIP:DIP-4_W7.62mm -> Package_DIP:DIP-16_W7.62mm
- SW2, SW3: footprint Package_DIP:DIP-4_W7.62mm -> Connector_PinSocket_2.54mm:PinSocket_1x03_P2.54mm_Vertical
- renumbered D35 to D1, D16 to D100, D17 to D101, D59 to D102, D60 to D103, D61 to D104, D62 to D105, D43 to D17, D44 to D18, D45 to D19, D36 to D2, D46 to D20, D47 to D21, D48 to D22, D49 to D23, D50 to D24, D51 to D25, D52 to D26, D53 to D27, D54 to D28, D55 to D29, D37 to D3, D56 to D30, D57 to D31, D58 to D32, D38 to D4, D19 to D41, D20 to D42, D21 to D43, D22 to D44, D23 to D45, D24 to D46, D25 to D47, D26 to D48, D9 to D49, D39 to D5, D10 to D50, D11 to D51, D12 to D52, D13 to D53, D14 to D54, D15 to D55, D18 to D56, D27 to D57, D28 to D58, D29 to D59, D40 to D6, D30 to D60, D31 to D61, D32 to D62, D33 to D63, D34 to D64, D41 to D7, D42 to D8, R15 to R100, R12 to R101, R13 to R12, R14 to R13, R24 to R14, R25 to R15, R26 to R16, R16 to R17, R17 to R18, R18 to R19, R19 to R20, R20 to R21, R21 to R22, R22 to R23, R23 to R24
Connections:
- net GND: now also D10.1 (K), D11.1 (K), D12.1 (K), D13.1 (K), D14.1 (K), D15.1 (K), D16.1 (K), D33.1 (K), D34.1 (K), D35.1 (K), D36.1 (K), D37.1 (K), D38.1 (K), D39.1 (K), D40.1 (K), D65.1 (K), D66.1 (K), D67.1 (K), D68.1 (K), D69.1 (K), D70.1 (K), D71.1 (K), D72.1 (K), D73.1 (K), D74.1 (K), D75.1 (K), D76.1 (K), D77.1 (K), D78.1 (K), D79.1 (K), D80.1 (K), D9.1 (K)
- net HLT: now also R79.1
- net J: now also R93.1; no longer U11.12 (IO1)
- net MAR0: now also R1.1, U4.9 (Zd), U6.3 (A7); no longer R8.1, U6.21 (A0), U9.4 (Za)
- net MAR1: now also R2.1, U4.12 (Zc), U6.2 (A6); no longer R7.1, U6.23 (A1), U9.7 (Zb)
- net MAR2: now also R3.1, U4.7 (Zb), U6.1 (A5); no longer R6.1, U6.24 (A2), U9.12 (Zc)
- net MAR3: now also R4.1, U4.4 (Za), U6.26 (A4); no longer R5.1, U6.25 (A3), U9.9 (Zd)
- net MAR4: now also R5.1, U6.25 (A3), U9.9 (Zd); no longer R4.1, U4.4 (Za), U6.26 (A4)
- net MAR5: now also R6.1, U6.24 (A2), U9.12 (Zc); no longer R3.1, U4.7 (Zb), U6.1 (A5)
- net MAR6: now also R7.1, U6.23 (A1), U9.7 (Zb); no longer R2.1, U4.12 (Zc), U6.2 (A6)
- net MAR7: now also R8.1, U6.21 (A0), U9.4 (Za); no longer R1.1, U4.9 (Zd), U6.3 (A7)
- net SU: now also R88.1
- net ~AI: now also R85.1
- net ~AO: now also R86.1
- net ~BI: now also R89.1
- net ~BO: now also R94.1; no longer U11.11 (IO0)
- net ~CE: now also R92.1; no longer U11.13 (IO2)
- net ~CO: now also R91.1
- net ~II: now also R84.1
- net ~IO: now also R83.1
- net ~MI: now also R80.1
- net ~OI: now also R90.1
- net ~RI: now also R81.1
- net ~RO: now also R82.1
- net ~SO: now also R87.1
- net ALU_D1: now reaches U16.3 (A1), U20.1 (S2)
- net ALU_D1: now also R72.1
- net ALU_D3: now reaches U16.5 (A3), U20.10 (S4)
- net ALU_D3: now also R74.1
- net ALU_D2: now reaches U16.4 (A2), U20.13 (S3)
- net ALU_D2: now also R73.1
- net ALU_D0: now reaches U16.2 (A0), U20.4 (S1)
- net ALU_D0: now also R71.1
- net ALU_D5: now reaches U16.7 (A5), U21.1 (S2)
- net ALU_D5: now also R76.1
- net ALU_D7: now reaches U16.9 (A7), U21.10 (S4)
- net ALU_D7: now also R78.1
- net ALU_D6: now reaches U16.8 (A6), U21.13 (S3)
- net ALU_D6: now also R77.1
- net ALU_D4: now reaches U16.6 (A4), U21.4 (S1)
- net ALU_D4: now also R75.1
- net at R8.2: now also D40.2 (A)
- net at R7.2: now also D39.2 (A)
- net at R6.2: now also D38.2 (A)
- net at R5.2: now also D37.2 (A)
- net at R4.2: now also D36.2 (A)
- net at R3.2: now also D35.2 (A)
- net at R2.2: now also D34.2 (A)
- net at R1.2: now also D33.2 (A)
- new net: D9.2 (A), R71.2
- new net: D10.2 (A), R72.2
- new net: D11.2 (A), R73.2
- new net: D12.2 (A), R74.2
- new net: D13.2 (A), R75.2
- new net: D14.2 (A), R76.2
- new net: D15.2 (A), R77.2
- new net: D16.2 (A), R78.2
- new net: D72.2 (A), R86.2
- new net: D70.2 (A), R84.2
- new net: D71.2 (A), R85.2
- new net: D69.2 (A), R83.2
- new net: D68.2 (A), R82.2
- new net: D67.2 (A), R81.2
- new net: D66.2 (A), R80.2
- new net: D65.2 (A), R79.2
- new net: D80.2 (A), R94.2
- new net: D78.2 (A), R92.2
- new net: D79.2 (A), R93.2
- new net: D77.2 (A), R91.2
- new net: D76.2 (A), R90.2
- new net: D75.2 (A), R89.2
- new net: D74.2 (A), R88.2
- new net: D73.2 (A), R87.2
- new net: D82.2 (A), R26.2
- new net: D81.2 (A), R25.2
- new net: D81.1 (K), D82.1 (K)
Other:
- moved on the sheet: D57, D58, D59, D60, D61, D62, D63, D64, R27, R28, R29, R30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
