File: noCPU/noCPU/noCPU.kicad_pcb (KiCad board)
At the start: 2 copper layers, 242 parts, among them SW1 SW_DIP_x08, SW2 SW_SPDT, SW3 SW_SPDT, SW4 SW_Push, U1 74HC173, U10 74LS138, U11 62256, U12 74HC245, U13 MAN71A, U14 74HC245, U15 74HC245, U16 74HC245, U17 74HC245, U18 74HC245, U19 MAN71A, U2 74HC173, U20 74HC283, U21 74HC283, U22 LM555, U23 74HC161, U24 MAN71A, U25 74HC173, U26 74HC173, U27 74HC173, U28 74HC161, U29 74HC173, U3 74HC173, U30 74HC173, U31 74HC173, U32 MAN71A, U33 74HC86, U34 74HC86, U35 74HC161, U36 62256, U37 74AHC1G08, U38 74AHC1G32, U39 74AHC1G04, U4 74HC157, U40 74AHC1G08, U41 74AHC1G08, U42 74AHC1G04, U43 LM555, U44 LM555, U45 LM555, U5 74HC173, U6 62256, U7 74HC161, U8 62256, U9 74HC157

Commit message: 1
Parts:
- moved U6 36.1 mm to (46.5, 61.2), turned to 90 degrees
- moved SW3 17.6 mm to (220.7, 111.0)
- moved D74 1.55 mm to (65.4, 183.4)
- moved D70 1.55 mm to (57.3, 183.4)
- moved D71 1.55 mm to (59.3, 183.4)
- moved D72 1.55 mm to (61.3, 183.4)
- moved D73 1.55 mm to (63.4, 183.4)
- moved D75 1.55 mm to (67.4, 183.4)
- moved D76 1.55 mm to (69.5, 183.4)
- moved D77 1.55 mm to (71.5, 183.4)
- moved D78 1.55 mm to (73.5, 183.4)
- moved D79 1.55 mm to (75.6, 183.4)
- moved D80 1.55 mm to (77.6, 183.4)
- moved D65 1.55 mm to (47.1, 183.4)
- moved D66 1.55 mm to (49.2, 183.4)
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